File: cores/exterm/sch/exterm.kicad_sch (KiCad schematic)
At the start: 20 parts

Commit message: wip ram objects
Parts:
- removed E7: Z80CPU, symbol CPU:Z80CPU
- added B10, B11, B8, B9: 74LS157, symbol jt74:74LS157
- added B5: 74LS174, symbol jt74:74LS174
- added C4, C5: 74LS245, symbol jt74:74LS245
- added C8: MB8464A-10L-LL, symbol fujitsu:MB8464A-10L-LL
- added E13, E14, E15, E16: HM6116P-3, symbol arcade:HM6116P-3
- added E8: Z80CPU, symbol CPU:Z80CPU
Connections:
- net VCC: now also C8.28 (VCC), E13.24 (VCC), E14.24 (VCC), E15.24 (VCC), E16.24 (VCC), E8.11 (VCC)
- net VSS: now also C8.14 (VSS), E13.12 (VSS), E14.12 (VSS), E15.12 (VSS), E16.12 (VSS), E8.29 (GND)
- net DBB2: now reaches E12.11 (B7)
- net DBB2: now also A15.14 (D5), E13.11 (D2), E14.11 (D2); no longer A15.13 (D4)
- net DBB3: now reaches E12.12 (B6)
- net DBB3: now also A15.13 (D4), E13.13 (D3), E14.13 (D3); no longer A15.14 (D5)
- net DBB4: now reaches A15.11 (D3), E12.13 (B5)
- net DBB4: now also E13.14 (D4), E14.14 (D4)
- net DBB5: now reaches A15.6 (D2), E12.14 (B4)
- net DBB5: now also E13.15 (D5), E14.15 (D5)
- net DBB6: now reaches E12.15 (B3)
- net DBB6: now also E13.16 (D6), E14.16 (D6)
- net DBB7: now reaches E12.16 (B2)
- net DBB7: now also E13.17 (D7), E14.17 (D7)
- net DBB0: now reaches A15.4 (D1), E12.17 (B1)
- net DBB0: now also E13.9 (D0), E14.9 (D0)
- net DBB1: now reaches A15.3 (D0), E12.18 (B0)
- net DBB1: now also E13.10 (D1), E14.10 (D1)
- net DB2: now reaches A16.3 (D0), E11.11 (B7)
- net DB2: now also E15.11 (D2), E16.11 (D2)
- net DB3: now reaches A16.4 (D1), E11.12 (B6)
- net DB3: now also E15.13 (D3), E16.13 (D3)
- net DB4: now reaches A16.7 (D2), E11.13 (B5)
- net DB4: now also E15.14 (D4), E16.14 (D4)
- net DB5: now reaches A16.8 (D3), E11.14 (B4)
- net DB5: now also E15.15 (D5), E16.15 (D5)
- net DB6: now reaches A16.13 (D4), E11.15 (B3)
- net DB6: now also E15.16 (D6), E16.16 (D6)
- net DB7: now reaches A16.18 (D7), E11.16 (B2)
- net DB7: now also E15.17 (D7), E16.17 (D7)
- net DB0: now reaches A16.14 (D5), E11.17 (B1)
- net DB0: now also E15.9 (D0), E16.9 (D0)
- net DB1: now reaches A16.17 (D6), E11.18 (B0)
- net DB1: now also E15.10 (D1), E16.10 (D1)
- net GFX_A0: now reaches B17.15 (A0)
- net GFX_A0: now also E13.8 (A0), E14.8 (A0), E15.8 (A0), E16.8 (A0)
- net GFX_A1: now reaches B17.16 (A1)
- net GFX_A1: now also E13.7 (A1), E14.7 (A1), E15.7 (A1), E16.7 (A1)
- net GFX_A2: now reaches B17.17 (A2)
- net GFX_A2: now also E13.6 (A2), E14.6 (A2), E15.6 (A2), E16.6 (A2)
- net GFX_A3: now reaches B17.18 (A3)
- net GFX_A3: now also E13.5 (A3), E14.5 (A3), E15.5 (A3), E16.5 (A3)
- net GFX_A4: now reaches B17.19 (A4)
- net GFX_A4: now also E13.4 (A4), E14.4 (A4), E15.4 (A4), E16.4 (A4)
- net GFX_A5: now reaches B17.20 (A5)
- net GFX_A5: now also E13.3 (A5), E14.3 (A5), E15.3 (A5), E16.3 (A5)
- net GFX_A6: now reaches B17.21 (A6)
- net GFX_A6: now also E13.2 (A6), E14.2 (A6), E15.2 (A6), E16.2 (A6)
- net GFX_A7: now reaches B17.22 (A7)
- net GFX_A7: now also E13.1 (A7), E14.1 (A7), E15.1 (A7), E16.1 (A7)
- net GFX_A8: now reaches B17.23 (A8)
- net GFX_A8: now also E13.23 (A8), E14.23 (A8), E15.23 (A8), E16.23 (A8)
- net GFX_A9: now reaches B17.24 (A9)
- net GFX_A9: now also E13.22 (A9), E14.22 (A9), E15.22 (A9), E16.22 (A9)
- net GFX_A10: now reaches B17.25 (A10)
- net GFX_A10: now also E13.19 (A10), E14.19 (A10), E15.19 (A10), E16.19 (A10)
- net GFX_A11: now reaches B17.28 (A11)
- net AB0 renamed D1
- net D1: now also E8.15 (D1)
- net AB1 renamed D0
- net D0: now also E8.14 (D0)
- net AB2 renamed D7
- net D7: now also E8.13 (D7)
- net AB3 renamed D6
- net D6: now also E8.10 (D6)
- net AB4 renamed D5
- net D5: now also E8.9 (D5)
- net AB5 renamed D4
- net D4: now also E8.7 (D4)
- net AB6 renamed D3
- net D3: now also E8.8 (D3)
- net AB7 renamed D2
- net D2: now also E8.12 (D2)
- net R_A0 renamed A0
- net A0: now also E8.30 (A0)
- net R_A1 renamed A1
- net A1: now also E8.31 (A1)
- net R_A10 renamed A10
- net A10: now also E8.40 (A10)
- net R_A11 renamed A11
- net A11: now also E8.1 (A11)
- net R_A12 renamed A12
- net A12: now also E8.2 (A12)
- net R_A13 renamed A13
- net A13: now also E8.3 (A13)
- net R_A2 renamed A2
- net A2: now also E8.32 (A2)
- net R_A3 renamed A3
- net A3: now also E8.33 (A3)
- net R_A4 renamed A4
- net A4: now also E8.34 (A4)
- net R_A5 renamed A5
- net A5: now also E8.35 (A5)
- net R_A6 renamed A6
- net A6: now also E8.36 (A6)
- net R_A7 renamed A7
- net A7: now also E8.37 (A7)
- net R_A8 renamed A8
- net A8: now also E8.38 (A8)
- net R_A9 renamed A9
- net A9: now also E8.39 (A9)
- net R_D0 renamed AD0
- net AD0: now also B5.3 (D0), C5.9 (A7)
- net R_D1 renamed AD1
- net AD1: now also B5.4 (D1), C5.8 (A6)
- net R_D2 renamed AD2
- net AD2: now also B5.6 (D2), C5.7 (A5)
- net R_D3 renamed AD3
- net AD3: now also B5.14 (D5), C5.6 (A4)
- net R_D4 renamed AD4
- net AD4: now also B5.13 (D4), C5.5 (A3)
- net R_D5 renamed AD5
- net AD5: now also B5.11 (D3), C5.4 (A2)
- net R_D6 renamed AD6
- net AD6: now also C5.3 (A1)
- net R_D7 renamed AD7
- net AD7: now also C5.2 (A0)
- new net: B11.11 (I0d), C8.10 (A0)
- new net: B11.4 (Za), C8.6 (A4)
- new net: B10.12 (Zc), C8.7 (A3)
- new net: B9.4 (Za), C8.8 (A2)
- new net: B11.14 (I0c), C8.9 (A1)
- new net A14: E8.4 (A14)
- new net A15: E8.5 (A15)
- new net AD_B0: C4.11 (B7), C5.11 (B7), C8.11 (D0)
- new net AD_B1: C4.12 (B6), C5.12 (B6), C8.12 (D1)
- new net AD_B2: C4.13 (B5), C5.13 (B5), C8.13 (D2)
- new net AD_B3: C4.14 (B4), C5.14 (B4), C8.15 (D3)
- new net AD_B4: C4.15 (B3), C5.15 (B3), C8.16 (D4)
- new net AD_B5: C4.16 (B2), C5.16 (B2), C8.17 (D5)
- new net AD_B6: C4.17 (B1), C5.17 (B1), C8.18 (D6)
- new net AD_B7: C4.18 (B0), C5.18 (B0), C8.19 (D7)
- no-connect marks 3 -> 1
Other:
- note added: "BIDIRECCIONAL?"
- note added: "CPU OBJECTS"
- note added: "GDA2?"
- moved on the sheet: A10, A12, A13, A15, A16, A2, A4, A5, A7, A8, B15, B17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

Commit message: wip main
Parts:
- added C2: PAL16L8, symbol Logic_Programmable:PAL16L8
- renumbered B10 to B11, B11 to B12
Connections:
- net VCC: now also C2.20 (VCC)
- net VSS: now also C2.10 (GND)
- net ~{GFX_CE}: no longer B1.11
- net MAIN_A8: now reaches B8.2 (I0a)
- net MAIN_A8: now also D3.38 (A8)
- net LUTA_A8: now reaches B8.4 (Za)
- net LUTA_A8: now also C8.25 (A8)
- net MAIN_A9: now reaches B8.5 (I0b)
- net MAIN_A9: now also D3.39 (A9)
- net LUTA_A9: now reaches B8.7 (Zb)
- net LUTA_A9: now also C8.24 (A9)
- net RAM_~{OE}: now reaches B8.9 (Zd)
- net RAM_~{OE}: now also C8.22 (~{OE})
- net MAIN_D7: now reaches C4.2 (A0)
- net MAIN_D7: now also D3.13 (D7)
- net MAIN_D6: now reaches C4.3 (A1)
- net MAIN_D6: now also D3.10 (D6)
- net MAIN_D5: now reaches C4.4 (A2)
- net MAIN_D5: now also D3.9 (D5)
- net MAIN_D4: now reaches C4.5 (A3)
- net MAIN_D4: now also D3.7 (D4)
- net MAIN_D3: now reaches C4.6 (A4)
- net MAIN_D3: now also D3.8 (D3)
- net MAIN_D2: now reaches C4.7 (A5)
- net MAIN_D2: now also D3.12 (D2)
- net MAIN_D1: now reaches C4.8 (A6)
- net MAIN_D1: now also D3.15 (D1)
- net MAIN_D0: now reaches C4.9 (A7)
- net MAIN_D0: now also D3.14 (D0)
- net LUTA_A0: now reaches C8.10 (A0)
- net LUTA_A0: now also B12.9 (Zd); no longer B12.11 (I0d)
- net LUTA_A12: now reaches C8.2 (A12)
- net LUTA_A12: now also B9.9 (Zd)
- net LUTA_A10: now reaches C8.21 (A10)
- net LUTA_A10: now also B9.12 (Zc)
- net LUTA_A11: now reaches C8.23 (A11)
- net LUTA_A11: now also B11.4 (Za)
- net LUTA_A7: now reaches C8.3 (A7)
- net LUTA_A7: now also B11.7 (Zb)
- net LUTA_A6: now reaches C8.4 (A6)
- net LUTA_A6: now also B11.9 (Zd)
- net LUTA_A5: now reaches C8.5 (A5)
- net LUTA_A5: now also B12.7 (Zb)
- net LUTA_A4: now reaches B12.4 (Za), C8.6 (A4)
- net LUTA_A3: now reaches B11.12 (Zc), C8.7 (A3)
- net LUTA_A2: now reaches B9.4 (Za), C8.8 (A2)
- net LUTA_A1: now reaches C8.9 (A1)
- net LUTA_A1: now also B12.12 (Zc); no longer B12.14 (I0c)
- net MAIN_A6: now reaches B11.11 (I0d)
- net MAIN_A6: now also D3.36 (A6)
- net MAIN_A3: now reaches B11.14 (I0c)
- net MAIN_A3: now also D3.33 (A3)
- net MAIN_A11: now reaches B11.2 (I0a)
- net MAIN_A11: now also D3.1 (A11)
- net MAIN_A7: now reaches B11.5 (I0b)
- net MAIN_A7: now also D3.37 (A7)
- net MAIN_A4: now reaches B12.2 (I0a)
- net MAIN_A4: now also D3.34 (A4)
- net MAIN_A5: now reaches B12.5 (I0b)
- net MAIN_A5: now also D3.35 (A5)
- net MAIN_A10: now reaches B9.11 (I0d)
- net MAIN_A10: now also D3.40 (A10)
- net MAIN_A12: now reaches B9.14 (I0c)
- net MAIN_A12: now also D3.2 (A12)
- net MAIN_A2: now reaches B9.2 (I0a)
- net MAIN_A2: now also D3.32 (A2)
- net MAIN_A13: now reaches D3.3 (A13)
- net MAIN_A13: now also C2.3 (I3)
- net MAIN_A0: now reaches D3.30 (A0)
- net MAIN_A0: now also B12.11 (I0d)
- net MAIN_A1: now reaches D3.31 (A1)
- net MAIN_A1: now also B12.14 (I0c)
- net MAIN_A14: now reaches D3.4 (A14)
- net MAIN_A14: now also C2.2 (I2)
- net MAIN_A15: now reaches D3.5 (A15)
- net MAIN_A15: now also C2.1 (I1)
- no-connect marks 1 -> 5
Other:
- note added: "BY C 13"
- note added: "MAIN"
- moved on the sheet: A10, A12, A13, A15, A16, A2, A4, A5, A7, A8, B11, B12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

Commit message: wip main gfx snd
Parts:
- added B13, C13: 74LS367, symbol jt74:74LS367
- added U?: 74LS74, symbol jt74:74LS74
- renumbered C10 to C11
Connections:
- net A0 is gone; now on net MAIN_A0: C11.10 (A0), C9.10 (A0), E8.30 (A0)
- net A1 is gone; now on net MAIN_A1: C11.9 (A1), C9.9 (A1), E8.31 (A1)
- net A10 is gone; now on net MAIN_A10: C11.21 (A10), C9.21 (A10), E8.40 (A10)
- net A11 is gone; now on net MAIN_A11: C11.23 (A11), C9.23 (A11), E8.1 (A11)
- net A12 is gone; now on net MAIN_A12: C11.2 (A12), C9.2 (A12), E8.2 (A12)
- net A13 is gone; now on net MAIN_A13: C11.26 (A13), C9.26 (A13), E8.3 (A13)
- net A14 is gone; now on net MAIN_A14: E8.4 (A14)
- net A15 is gone; now on net MAIN_A15: E8.5 (A15)
- net A2 is gone; now on net MAIN_A2: C11.8 (A2), C9.8 (A2), E8.32 (A2)
- net A3 is gone; now on net MAIN_A3: C11.7 (A3), C9.7 (A3), E8.33 (A3)
- net A4 is gone; now on net MAIN_A4: C11.6 (A4), C9.6 (A4), E8.34 (A4)
- net A5 is gone; now on net MAIN_A5: C11.5 (A5), C9.5 (A5), E8.35 (A5)
- net A6 is gone; now on net MAIN_A6: C11.4 (A6), C9.4 (A6), E8.36 (A6)
- net A7 is gone; now on net MAIN_A7: C11.3 (A7), C9.3 (A7), E8.37 (A7)
- net A8 is gone; now on net MAIN_A8: C11.25 (A8), C9.25 (A8), E8.38 (A8)
- net A9 is gone; now on net MAIN_A9: C11.24 (A9), C9.24 (A9), E8.39 (A9)
- net D0 is gone; now on net MAIN_D0: E11.3 (A1), E12.3 (A1), E8.14 (D0)
- net D1 is gone; now on net MAIN_D1: E11.2 (A0), E12.2 (A0), E8.15 (D1)
- net D2 is gone; now on net MAIN_D2: E11.9 (A7), E12.9 (A7), E8.12 (D2)
- net D3 is gone; now on net MAIN_D3: E11.8 (A6), E12.8 (A6), E8.8 (D3)
- net D4 is gone; now on net MAIN_D4: E11.7 (A5), E12.7 (A5), E8.7 (D4)
- net D5 is gone; now on net MAIN_D5: E11.6 (A4), E12.6 (A4), E8.9 (D5)
- net D6 is gone; now on net MAIN_D6: E11.5 (A3), E12.5 (A3), E8.10 (D6)
- net D7 is gone; now on net MAIN_D7: E11.4 (A2), E12.4 (A2), E8.13 (D7)
- net GFX_A0: now also B13.9 (O4a)
- net GFX_A1: now also B13.11 (O5b)
- net GFX_A10: now also C13.13 (O6b)
- net GFX_A2: now also B12.13 (I1c), B13.13 (O6b)
- net GFX_A3: now also B13.3 (O1a)
- net GFX_A4: now also B13.5 (O2a)
- net GFX_A5: now also B13.7 (O3a)
- net GFX_A6: now also C13.5 (O2a)
- net GFX_A7: now also C13.7 (O3a)
- net GFX_A8: now also C13.9 (O4a)
- net GFX_A9: now also C13.11 (O5b)
- net MAIN_A0: now also B12.10 (I1d), B13.10 (I4); no longer B12.11 (I0d), D3.30 (A0)
- net MAIN_A1: now also B13.12 (I5); no longer B12.14 (I0c), D3.31 (A1)
- net MAIN_A10: now also B9.10 (I1d), C13.14 (I6); no longer B9.11 (I0d), D3.40 (A10)
- net MAIN_A11: now also B11.3 (I1a); no longer B11.2 (I0a), D3.1 (A11)
- net MAIN_A12: now also B9.13 (I1c); no longer B9.14 (I0c), D3.2 (A12)
- net MAIN_A13: no longer C2.3 (I3), D3.3 (A13)
- net MAIN_A14: no longer C2.2 (I2), D3.4 (A14)
- net MAIN_A15: no longer C2.1 (I1), D3.5 (A15)
- net MAIN_A2: now also B9.3 (I1a), B13.14 (I6); no longer B9.2 (I0a), D3.32 (A2)
- net MAIN_A3: now also B11.13 (I1c), B13.2 (I1); no longer B11.14 (I0c), D3.33 (A3)
- net MAIN_A4: now also B12.3 (I1a), B13.4 (I2); no longer B12.2 (I0a), D3.34 (A4)
- net MAIN_A5: now also B12.6 (I1b), B13.6 (I3); no longer B12.5 (I0b), D3.35 (A5)
- net MAIN_A6: now also B11.10 (I1d), C13.4 (I2); no longer B11.11 (I0d), D3.36 (A6)
- net MAIN_A7: now also B11.6 (I1b), C13.6 (I3); no longer B11.5 (I0b), D3.37 (A7)
- net MAIN_A8: now also B8.3 (I1a), C13.10 (I4); no longer B8.2 (I0a), D3.38 (A8)
- net MAIN_A9: now also B8.6 (I1b), C13.12 (I5); no longer B8.5 (I0b), D3.39 (A9)
- net MAIN_D0: no longer C4.9 (A7), D3.14 (D0)
- net MAIN_D1: no longer C4.8 (A6), D3.15 (D1)
- net MAIN_D2: no longer C4.7 (A5), D3.12 (D2)
- net MAIN_D3: no longer C4.6 (A4), D3.8 (D3)
- net MAIN_D4: no longer C4.5 (A3), D3.7 (D4)
- net MAIN_D5: no longer C4.4 (A2), D3.9 (D5)
- net MAIN_D6: no longer C4.3 (A1), D3.10 (D6)
- net MAIN_D7: no longer C4.2 (A0), D3.13 (D7)
- net ~{GFX_CE}: now also B1.11
- net DVAL: now reaches B17.26 (DVAL)
- net DVAL: now also C13.3 (O1a)
- net AD0 renamed MAIN_AD0
- net AD1 renamed MAIN_AD1
- net AD2 renamed MAIN_AD2
- net AD3 renamed MAIN_AD3
- net AD4 renamed MAIN_AD4
- net AD5 renamed MAIN_AD5
- net AD6 renamed MAIN_AD6
- net AD7 renamed MAIN_AD7
- net AD_B0 renamed MAIN_DB0
- net AD_B1 renamed MAIN_DB1
- net AD_B2 renamed MAIN_DB2
- net AD_B3 renamed MAIN_DB3
- net AD_B4 renamed MAIN_DB4
- net AD_B5 renamed MAIN_DB5
- net AD_B6 renamed MAIN_DB6
- net AD_B7 renamed MAIN_DB7
- net LUTA_A0 renamed SND_M0
- net LUTA_A1 renamed SND_M1
- net LUTA_A10 renamed SND_M10
- net SND_M10: now also B9.9 (Zd); no longer B9.12 (Zc)
- net LUTA_A11 renamed SND_M11
- net LUTA_A12 renamed SND_M12
- net SND_M12: now also B9.12 (Zc); no longer B9.9 (Zd)
- net LUTA_A2 renamed SND_M2
- net LUTA_A3 renamed SND_M3
- net LUTA_A4 renamed SND_M4
- net LUTA_A5 renamed SND_M5
- net LUTA_A6 renamed SND_M6
- net LUTA_A7 renamed SND_M7
- net LUTA_A8 renamed SND_M8
- net LUTA_A9 renamed SND_M9
- new net SND_A0: B12.11 (I0d), D3.30 (A0)
- new net SND_A1: B12.14 (I0c), D3.31 (A1)
- new net SND_A10: B9.11 (I0d), D3.40 (A10)
- new net SND_A11: B11.2 (I0a), D3.1 (A11)
- new net SND_A12: B9.14 (I0c), D3.2 (A12)
- new net SND_A13: C2.3 (I3), D3.3 (A13)
- new net SND_A14: C2.2 (I2), D3.4 (A14)
- new net SND_A15: C2.1 (I1), D3.5 (A15)
- new net SND_A2: B9.2 (I0a), D3.32 (A2)
- new net SND_A3: B11.14 (I0c), D3.33 (A3)
- new net SND_A4: B12.2 (I0a), D3.34 (A4)
- new net SND_A5: B12.5 (I0b), D3.35 (A5)
- new net SND_A6: B11.11 (I0d), D3.36 (A6)
- new net SND_A7: B11.5 (I0b), D3.37 (A7)
- new net SND_A8: B8.2 (I0a), D3.38 (A8)
- new net SND_A9: B8.5 (I0b), D3.39 (A9)
- new net SND_D0: C4.9 (A7), D3.14 (D0)
- new net SND_D1: C4.8 (A6), D3.15 (D1)
- new net SND_D2: C4.7 (A5), D3.12 (D2)
- new net SND_D3: C4.6 (A4), D3.8 (D3)
- new net SND_D4: C4.5 (A3), D3.7 (D4)
- new net SND_D5: C4.4 (A2), D3.9 (D5)
- new net SND_D6: C4.3 (A1), D3.10 (D6)
- new net SND_D7: C4.2 (A0), D3.13 (D7)
- no-connect marks 5 -> 7
Other:
- note added: "CPU MAIN"
- note added: "GXF"
- note added: "MAIN_DB"
- note added: "REVISAR"
- note added: "SE CONECTA A CPU SND?"
- note added: "SOUND"
- note added: "TRIESTADO?"
- note removed: "BIDIRECCIONAL?"
- note removed: "BY C 13"
- note removed: "CPU OBJECTS"
- note removed: "GDA2?"
- note removed: "OBJECTS"
- moved on the sheet: A10, A12, A13, A15, A16, A2, A4, A5, A7, A8, B11, B12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

Commit message: main
Parts:
- removed B17: YM3906, symbol yamaha:YM3906
- added unit 1 of B1
- added B13: 74LS245, symbol jt74:74LS245
- added B2: 74LS08, symbol jt74:74LS08
- added unit 2 of B3
- added unit 3 of B3
- added B4, B7: 74LS74, symbol jt74:74LS74
- added C4: C101, symbol Device:C
- added C6: 74LS32, symbol jt74:74LS32
- added D6: PAL16L8, symbol Logic_Programmable:PAL16L8
- added E4: 27C512, Package_DIP:DIP-28_W15.24mm, symbol Memory_EPROM:27C512
- added F8: YM2203, Package_DIP:DIP-40_W15.24mm, symbol yamaha:YM2203
- added G13: 74LS04, symbol jt74:74LS04
- added R150Ω, R330Ω: R20, symbol Device:R_US
- added SWA, SWB: SW_DIPS_08, symbol Mod_KC_Symbols:SW_DIPS_08
- added U?: YM3906, symbol yamaha:YM3906
- gave numbers to parts that had none: 1
Connections:
- net DVAL: now also U?.26 (DVAL)
- net GA0: now also U?.35 (CHA0)
- net GA1: now also U?.36 (CHA1)
- net GA2: now also U?.37 (CHA2)
- net GA4: now also U?.38 (CHA4)
- net GFX_A0: now also U?.15 (A0)
- net GFX_A1: now also U?.16 (A1)
- net GFX_A10: now also U?.25 (A10)
- net GFX_A11: now also U?.28 (A11)
- net GFX_A2: now also U?.17 (A2)
- net GFX_A3: now also U?.18 (A3)
- net GFX_A4: now also U?.19 (A4)
- net GFX_A5: now also U?.20 (A5)
- net GFX_A6: now also U?.21 (A6)
- net GFX_A7: now also U?.22 (A7)
- net GFX_A8: now also U?.23 (A8)
- net GFX_A9: now also U?.24 (A9)
- net GFX_CLK: now also B13.11 (B7)
- net HC0: now also U?.46 (HC0)
- net HC1: now also U?.47 (HC1)
- net HC2: now also U?.48 (HC2)
- net HC3: now also U?.49 (HC3)
- net HC4: now also U?.50 (HC4)
- net HC5: now also U?.51 (HC5)
- net HC6: now also U?.52 (HC6)
- net HC7: now also U?.53 (HC7)
- net HC8: now also U?.54 (HC8)
- net HR8: now also U?.34 (H8B)
- net MAIN_A15: now also B2.10, D6.1 (I1)
- net SND_A0: now also E4.10 (A0), F8.37 (A0)
- net SND_A1: now also E4.9 (A1)
- net SND_A10: now also E4.21 (A10)
- net SND_A11: now also E4.23 (A11)
- net SND_A12: now also E4.2 (A12)
- net SND_A13: now also E4.26 (A13)
- net SND_A14: now also E4.27 (A14)
- net SND_A15: now also E4.1 (A15)
- net SND_A2: now also E4.8 (A2)
- net SND_A3: now also E4.7 (A3)
- net SND_A4: now also E4.6 (A4)
- net SND_A5: now also E4.5 (A5)
- net SND_A6: now also E4.4 (A6)
- net SND_A7: now also E4.3 (A7)
- net SND_A8: now also E4.25 (A8)
- net SND_A9: now also E4.24 (A9)
- net SND_D0: now also E4.11 (D0), F8.40 (D0)
- net SND_D1: now also E4.12 (D1), F8.2 (D1)
- net SND_D2: now also E4.13 (D2), F8.3 (D2)
- net SND_D3: now also E4.15 (D3), F8.4 (D3)
- net SND_D4: now also E4.16 (D4), F8.5 (D4)
- net SND_D5: now also E4.17 (D5), F8.6 (D5)
- net SND_D6: now also E4.18 (D6), F8.7 (D6)
- net SND_D7: now also E4.19 (D7), F8.8 (D7)
- net VCC: now also B3.1 (~{R}), B13.1 (A->B), B2.14 (VCC), B3.10 (~{S}), B3.13 (~{R}), B3.14 (VCC), B4.10 (~{S}), B4.13 (~{R}), B4.14 (VCC), B4.2 (D), B4.4 (~{S}), B7.10 (~{S}), B7.12 (D), B7.14 (VCC), C6.14 (VCC), D6.20 (VCC), E4.28 (VCC), F8.21 (VCC), G13.14 (VCC), R330Ω.1, U?.1 (VCC), U?.33 (VCC)
- net VSS: now also B13.19 (~{CE}), B2.7 (VSS), B3.7 (VSS), B4.7 (VSS), B7.7 (VSS), C4.2, C6.7 (VSS), D6.10 (GND), E4.14 (GND), E4.20 (~{CE}), F8.1 (VSS), G13.7 (VSS), SWA.10, SWA.11, SWA.12, SWA.13, SWA.14, SWA.15, SWA.16, SWA.9, SWB.1, SWB.2, SWB.3, SWB.4, SWB.5, SWB.6, SWB.7, SWB.8, U?.32 (VSS), U?.64 (VSS)
- net ~{RD}: now reaches B8.10 (I1d)
- net ~{RD}: now also D3.21 (~{RD}), F8.36 (~{RD})
- net SND_~{OE}: now reaches C2.12 (IO8)
- net SND_~{OE}: now also E4.22 (~{OE})
- net ~{WDRES}: now reaches B5.1 (~{Mr})
- net ~{WDRES}: now also B2.1, U?.29 (~{WDRES)
- net MAIN_AD'5: now reaches B5.10 (Q3)
- net MAIN_AD'4: now reaches B5.12 (Q4)
- net MAIN_AD'4: now also B2.2
- net MAIN_AD'3: now reaches B5.15 (Q5)
- net MAIN_AD'0: now reaches B5.2 (Q0)
- net MAIN_AD'1: now reaches B5.5 (Q1)
- net MAIN_AD'1: now also C9.1 (A15), B2.9
- net MAIN_AD'2: now reaches B5.7 (Q2)
- net ~{CS}: now reaches B3.2 (D)
- net ~{CS}: now also F8.34 (~{CS})
- net at B3.3 (C): now also B13.15 (B3), B3.11 (C), B7.11 (C)
- net ~{WR}: now reaches D3.22 (~{WR})
- net ~{WR}: now also F8.35 (~{WR})
- net ~{RESET}: now reaches D3.26 (~{RESET})
- net ~{RESET}: now also B2.12, B2.3
- net R_A15 renamed MAIN_AD
- net MAIN_AD: now also B2.8; no longer C9.1 (A15)
- new net: F8.32 (IOB6), SWB.10
- new net: F8.31 (IOB5), SWB.11
- new net: F8.30 (IOB4), SWB.12
- new net: F8.29 (IOB3), SWB.13
- new net: F8.28 (IOB2), SWB.14
- new net: F8.27 (IOB1), SWB.15
- new net: F8.26 (IOB0), SWB.16
- new net: F8.33 (IOB7), SWB.9
- new net: B13.12 (B6), B2.5, C6.13, C6.2
- new net: B2.6, B4.12 (D)
- new net: C4.1, R150Ω.2
- new net: B13.13 (B5), G13.11, R330Ω.2
- new net: F8.16 (IOA0), SWA.1
- new net: F8.15 (IOA1), SWA.2
- new net: F8.14 (IOA2), SWA.3
- new net: F8.13 (IOA3), SWA.4
- new net: F8.12 (IOA4), SWA.5
- new net: F8.11 (IOA5), SWA.6
- new net: F8.10 (IOA6), SWA.7
- new net: F8.9 (IOA7), SWA.8
- new net: B1.5 (Q1), B2.13
- new net H0: B13.4 (A2), B13.5 (A3), B13.6 (A4), U?.40 (HPH90)
- new net H1: B13.7 (A5), U?.39 (H)
- new net H2: B13.2 (A0), U?.41 (H2)
- new net H3: B13.8 (A6), U?.42 (H4)
- new net H4: B13.9 (A7), U?.43 (H8)
- new net PHM: B13.18 (B0), B2.4, F8.38 (PHM)
- new net PIN3INTEL: G13.10
- new net PIN4INTEL: B2.11
- new net PULL DOWN: B13.16 (B2), R150Ω.1
- new net ~{IC}: B1.1 (~{Mr}), F8.24 (~{IC})
Other:
- note added: "BIDIRECCIONAL?"
- note added: "DRIVER"
- note added: "FALTA OTRA ENTRADA"
- note added: "PIN10INTEL"
- note added: "PIN2INTEL"
- note added: "PIN8INTEL"
- note added: "PIN9INTEL"
- moved on the sheet: B3A
