File: cores/exterm/sch/exterm.kicad_sch (KiCad schematic)
At the start: 50 parts

Commit message: gates logics and drivers
Parts:
- added A17: 12.000MHz, Oscillator:Oscillator_SMD_Abracon_ASDMB-4Pin_2.5x2.0mm, symbol Oscillator:ASDMB-xxxMHz
- added unit 4 of B1
- added unit 1 of B1
- added unit 6 of B1
- added unit 7 of B1
- added unit 3 of B1
- added unit 2 of B1
- added B6: 74LS08, symbol jt74:74LS08
- added G4: INTEL8742, symbol Intel:INTEL8742
- added J8: TL7705A, symbol Power_Supervisor:TL7705A
- added JP1: Jumper_2_Bridged, symbol Jumper:Jumper_2_Bridged
- added R1KΩ: R7, symbol Device:R_US
- added SW1: SW_DIP_x02, symbol Switch:SW_DIP_x02
- gave numbers to parts that had none: 1
- renumbered B13 to B14, C13 to C14, D10 to D9, B1 to E1, E15 to E17
Connections:
- net AB is gone; now on net MAIN_~{RD}: E11.1 (A->B), E12.1 (A->B)
- net DB0: now also B17.14 (D0)
- net DB1: now also B17.13 (D1)
- net DB2: now also B17.12 (D2)
- net DB3: now also B17.11 (D3)
- net DB4: now also B17.10 (D4)
- net DB5: now also B17.9 (D5)
- net DB6: now also B17.8 (D6)
- net DB7: now also B17.7 (D7)
- net DBB0: now also B17.4 (XC0)
- net DBB2: now also B15.10 (UK)
- net DBB3: now also B15.9 (PAL0)
- net DBB4: now also B15.8 (PAL1)
- net DBB5: now also B15.7 (PAL2)
- net DBB6: now also B15.6 (PAL3), B17.59 (FLIPY)
- net DBB7: now also B15.5 (PAL4), B17.60 (FLIPX)
- net GFX_CLK: now also B15.3 (CLK), B17.62 (CLK)
- net SND_A0: now also G4.28 (P11)
- net VCC: now also A17.4 (VDD), B1.14 (VCC), B6.14 (VCC)
- net VSS: now also B17.31 (UK), B17.45 (UK), E13.20 (~{OE}), E14.20 (~{OE}), E16.20 (~{OE}), E17.20 (~{OE}), A17.2 (GND), B1.7 (VSS), B6.7 (VSS), SW1.2, SW1.3
- net ~{GFX_CE}: no longer A12.20 (~{CE}), A2.20 (~{CE}), A5.20 (~{CE}), A8.20 (~{CE})
- net ~{WDRES}: now also R1KΩ.1
- net H3B: now reaches B13.12 (B6), B2.5, C6.13, C6.2
- net H3B: now also B14.1 (OEa), B14.15 (OEb), C14.1 (OEa), C14.15 (OEb), D6.11 (I10)
- net /WR: now reaches D9.13 (IO7)
- net /WR: now also B17.3 (/WR), B6.1
- net DREQ: now reaches D9.5 (I5)
- net DREQ: now also B17.27 (DREQ)
- net XTAL1: now reaches B13.13 (B5), G13.11, R330Ω.2
- net XTAL1: now also G4.2 (XTAL1)
- net COL0: now reaches B15.20 (COL0)
- net COL1: now reaches B15.21 (COL1)
- net COL2: now reaches B15.22 (COL2)
- net COL3: now reaches B15.23 (COL3)
- net COL4: now reaches B15.24 (COL4)
- net COL5: now reaches B15.25 (COL5)
- net COL6: now reaches B15.26 (COL6)
- net COL7: now reaches B15.27 (COL7)
- net COL8: now reaches B15.28 (COL8)
- net DATAEN: now reaches B15.4 (DATAEN)
- net DATAEN: now also B17.61 (DATAEN)
- net RW: now reaches C6.5
- net RW: now also B17.30 (RW)
- net GFX_~{CS}: now reaches E16.18 (~{CS})
- net GFX_~{CS}: now also D6.18 (IO2), E13.18 (~{CS}), E14.18 (~{CS}), E17.18 (~{CS})
- net GFX_~{WR}: now reaches E16.21 (~{WR})
- net GFX_~{WR}: now also E13.21 (~{WR}), E14.21 (~{WR}), E17.21 (~{WR})
- net GFX_CE: now reaches B1.10
- net GFX_CE: now also A12.20 (~{CE}), A2.20 (~{CE}), A5.20 (~{CE}), A8.20 (~{CE})
- net MBB_~{CE}: now reaches E12.19 (~{CE})
- net MBB_~{CE}: now also C6.3
- net MAB_~{CE}: now reaches C6.11
- net MAB_~{CE}: now also E11.19 (~{CE})
- net MAIN_~{RD}: now reaches B17.2 (/RDACT)
- net MAIN_~{RD}: now also B8.10 (I1d), E8.21 (~{RD}), G13.9
- net HBLK: now reaches B17.55 (HBLK)
- net VSYNC: now reaches B17.56 (VSYNC)
- net VBLK: now reaches B17.58 (VBLK)
- net VBLK: now also B1.13
- net at B17.63 (CLK): now also A17.3 (Out)
- net at G13.8: now also JP1.1 (A)
- net PIN3INTEL renamed XTAL2
- net XTAL2: now also G4.3 (XTAL2)
- net ~{RD} renamed SND_~{RD}
- net SND_~{RD}: now also G4.8 (~{RD}); no longer B8.10 (I1d)
- net ~{WR} renamed SND_~{WR}
- net SND_~{WR}: now also G4.10 (~{WR})
- new net: JP1.2 (B), SW1.1, SW1.4
- new net: J8.5 (~{RESET}), R1KΩ.2
- no-connect marks 7 -> 13
Other:
- note added: "?"
- note added: "COLMIX"
- note added: "DEL 19 AL 1 F15"
- note added: "DRIVER?"
- note added: "PIN19SETA003"
- note added: "PIN20SETA003"
- note removed: "BIDIRECCIONAL?"
- note removed: "MAIN_DB"
- note removed: "PIN10INTEL"
- note removed: "PIN2INTEL"
- note removed: "PIN8INTEL"
- note removed: "PIN9INTEL"
- moved on the sheet: C6B, C6C, G13D

Commit message: address decoders
Parts:
- added C3: PAL16L8, symbol Logic_Programmable:PAL16L8
- added G14: 74HC4024, Package_SO:SOIC-14_3.9x8.7mm_P1.27mm, symbol 74xx:74HC4024
- added R1KΩ: R6, symbol Device:R_US
- added R1KΩ: R1, symbol Device:R_US
- added R330Ω: R20, symbol Device:R_US
- added R330Ω: R19, symbol Device:R_US
- renumbered D9 to D8
Connections:
- net DREQ is gone; now on net MAIN_A11: B17.27 (DREQ), D8.5 (I5)
- net GFX_~{WR}: now also C6.6
- net MAIN_A10: now also D8.6 (I6)
- net MAIN_A12: now also D8.4 (I4)
- net MAIN_A13: now also D8.3 (I3)
- net MAIN_A14: now also D6.2 (I2), D8.2 (I2)
- net MAIN_A15: now also D8.1 (I1)
- net MAIN_A9: now also D8.7 (I7)
- net MAIN_AD'0: now also D6.7 (I7)
- net MAIN_AD'1: now also D6.6 (I6)
- net MAIN_AD'2: now also D6.5 (I5)
- net MAIN_~{RD}: now also B1.9, C5.1 (A->B); no longer G13.9
- net SND_~{RD}: now also B8.11 (I0d), C4.1 (A->B)
- net SND_~{WR}: now also C3.4 (I4)
- net VCC: now also D8.20 (VCC), E8.17 (~{NMI}), J8.8 (VCC), R1KΩ.1, C3.20 (VCC), G14.14 (VCC), R1KΩ.1, R1KΩ.1, R330Ω.1, R330Ω.1
- net VSS: now also B11.15 (E), B12.15 (E), B8.15 (E), B9.15 (E), D8.10 (GND), J8.4 (GND), C3.10 (GND), G14.7 (GND)
- net ~{WDRES}: now also E8.26 (~{RESET}), J8.5 (~{RESET}), R1KΩ.2; no longer R1KΩ.1
- net CLK_SND: now reaches B13.15 (B3), B3.11 (C), B3.3 (C), B7.11 (C)
- net CLK_SND: now also D3.6 (~{CLK}), R330Ω.2
- net at B3.12 (D): now also B3.5 (Q)
- net SND_CLK': now reaches B3.9 (Q)
- net SND_CLK': now also B3.4 (~{S}), C3.9 (I9)
- net ~{SND_WR}: now reaches C5.19 (~{CE})
- net ~{SND_WR}: now also C3.16 (IO4)
- net MAIN_~{WR}: now reaches D8.11 (I10)
- net MAIN_~{WR}: now also E8.22 (~{WR}), C3.2 (I2)
- net ~{BGTRNSP}: now reaches D8.14 (IO6)
- net ~{BGTRNSP}: now also B15.2 (~{BGTRNSP})
- net ~{MAIN_A11}: now reaches D8.15 (IO5)
- net ~{MAIN_A11}: now also B1.5, B5.9 (Cp)
- net ~{MAIN_WR}: now reaches D8.16 (IO4)
- net ~{MAIN_WR}: now also B6.2, D6.8 (I8)
- net ~{MAIN_A13}: now reaches D8.17 (I03)
- net ~{MAIN_A13}: now also D6.9 (I9)
- net at D8.18 (IO2): now also C3.1 (I1)
- net ~{SB_CE}: now reaches D8.19 (IO1)
- net ~{SB_CE}: now also C3.5 (I5)
- net M_~{MREQ}: now reaches D8.8 (I8)
- net M_~{MREQ}: now also D6.3 (I3), E8.19 (~{MREQ})
- net M_~{RFSH}: now reaches D8.9 (I9)
- net M_~{RFSH}: now also D6.4 (I4), E8.28 (~{RFSH})
- net SND_SELECT: now reaches B8.1 (S)
- net SND_SELECT: now also B11.1 (S), B12.1 (S), B9.1 (S), C3.19 (IO1)
- net CLK_MAIN: now reaches B4.11 (C)
- net CLK_MAIN: now also E8.6 (~{CLK}), R330Ω.2
- net QB: now reaches B4.9 (Q)
- net QB: now also C3.6 (I6)
- net RAM_~{CS1}: now reaches C8.20 (~{CS1})
- net RAM_~{CS1}: now also C3.17 (I03)
- net RAM_~{WE}: now reaches C8.27 (~{WE})
- net RAM_~{WE}: now also C3.18 (IO2)
- net at B1.8: now also C6.4
- net S_~{IORQ}: now reaches B7.13 (~{R})
- net S_~{IORQ}: now also D3.20 (~{IORQ})
- net SND_~{INT}: now reaches B7.8 (~{Q})
- net SND_~{INT}: now also D3.16 (~{INT})
- net ~{SND_MREQ}: now reaches C2.13 (IO7)
- net ~{SND_MREQ}: now also C3.3 (I3)
- net S_~{MREQ}: now reaches C2.7 (I7)
- net S_~{MREQ}: now also D3.19 (~{MREQ})
- net SND_~{RFSH}: now reaches C2.8 (I8)
- net SND_~{RFSH}: now also D3.28 (~{RFSH})
- net M_~{IORQ}: now reaches B4.1 (~{R})
- net M_~{IORQ}: now also E8.20 (~{IORQ})
- net ~{VBLK}: now reaches B4.3 (C)
- net ~{VBLK}: now also B1.12
- net MAIN_~{INT}: now reaches B4.6 (~{Q})
- net MAIN_~{INT}: now also E8.16 (~{INT})
- net MAIN_WR: now reaches C6.12
- net MAIN_WR: now also B6.3
- net SB_~{CE}: now reaches C4.19 (~{CE})
- net SB_~{CE}: now also C3.15 (IO5)
- net MAIN_~{WAIT}: now reaches E8.24 (~{WAIT})
- net MAIN_~{WAIT}: now also C3.14 (IO6)
- net at B1.6: now also G14.2 (MR)
- net ~{SND_CLK'}: now reaches B3.6 (~{Q})
- net ~{SND_CLK'}: now also C3.11 (I10)
- net at D3.17 (~{NMI}): now also R1KΩ.2
- net SND_~{WAIT}: now reaches D3.24 (~{WAIT})
- net SND_~{WAIT}: now also C3.13 (IO7)
- net /WR renamed ~{GFX_WR}
- new net: C3.7 (I7), R1KΩ.2
- new net: G13.9, G14.5 (Q4)
- no-connect marks 13 -> 24
Other:
- note removed: "DRIVER?"
- note removed: "FALTA OTRA ENTRADA"
- moved on the sheet: A17, B1C, B1D, B1F, B2A, B2C, C4, C5, C6B, D6, D8, G13D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

Commit message: wip
Parts:
- removed unit 1 of B7
Connections:
- net ~{CS} is gone; now on net YM_~{CS}: B3.2 (D), F8.34 (~{CS})
- net ~{IC} is gone; now on net ~{RESET}: E1.1 (~{Mr}), F8.24 (~{IC})
- net CLK_MAIN: now also B13.17 (B1)
- net MAIN_A13: now also C8.26 (~{CS2})
- net R_A14: no longer C11.27 (A14)
- net SND_A11: now also C2.5 (I5)
- net SND_A12: now also C2.4 (I4)
- net SND_A13: no longer E4.26 (A13)
- net SND_A14: no longer E4.27 (A14)
- net SND_D0: now also E1.14 (D5)
- net SND_D1: now also E1.13 (D4)
- net SND_D2: now also E1.11 (D3)
- net SND_D3: now also E1.6 (D2)
- net SND_D4: now also E1.4 (D1)
- net SND_D5: now also E1.3 (D0)
- net SND_~{WR}: now also C2.6 (I6)
- net ~{SND_WR}: now also C2.14 (IO6), E1.9 (Cp)
- net DD_~{CS}: now reaches G4.6 (~{CS})
- net DD_~{CS}: now also C2.16 (IO4)
- net SND_D'0: now reaches C2.11 (I10)
- net SND_D'0: now also E1.15 (Q5)
- net YM_~{CS}: now reaches C2.15 (IO5)
- net ~{SND_A14}: now reaches C2.18 (IO2)
- net ~{SND_A14}: now also E4.26 (A13)
- net ~{SND_A15}: now reaches C2.19 (IO1)
- net ~{SND_A15}: now also E4.27 (A14)
- net SND_D'1: now reaches C2.9 (I9)
- net SND_D'1: now also E1.12 (Q4)
- net ~{RM_OEA}: now reaches D6.12 (IO8)
- net ~{RM_OEA}: now also C9.22 (~{OE})
- net ~{RM_OEB}: now reaches D6.13 (IO7)
- net ~{RM_OEB}: now also C11.22 (~{OE})
- net ~{MAIN_AD'1}: now reaches D6.14 (IO6)
- net ~{MAIN_AD'1}: now also C11.27 (A14)
- net GFXD_~{CS}: now reaches D6.15 (IO5)
- net GFXD_~{CS}: now also E17.18 (~{CS})
- net GFXC_~{CS}: now reaches D6.16 (IO4)
- net GFXC_~{CS}: now also E16.18 (~{CS})
- net GFXB_~{CS}: now reaches D6.17 (I03)
- net GFXB_~{CS}: now also E14.18 (~{CS})
- net ?: now reaches D6.19 (IO1)
- net ?: now also B13.14 (B4), B13.3 (A1), D8.12 (IO8)
- removed net GFX_~{CS}: D6.18 (IO2), E13.18 (~{CS}), E14.18 (~{CS}), E16.18 (~{CS}), E17.18 (~{CS})
- net XTAL2 renamed ~{XTAL2}
- removed net ~{RM_OE}: C11.22 (~{OE}), C9.22 (~{OE}), D8.12 (IO8)
- new net GFXA_~{CS}: D6.18 (IO2), E13.18 (~{CS})
- no-connect marks 24 -> 31
Other:
- note added: "POSIBLEMENTE PXCLK"
- note removed: "DRIVER"
- moved on the sheet: E1, G4

Commit message: address decoders
Parts:
- added 8.2KΩ, R1KΩ: R7, symbol Device:R_US
- added C10: C104, symbol Device:C
- added C13: 1μF, symbol Device:CP1
- added H11: YM3014, Package_DIP:DIP-8_W7.62mm, symbol yamaha:YM3014
- added H12: NJM4558, symbol Amplifier_Operational:NJM4558
- added RV?: R_POT_US, symbol Device:R_POT_US
- R1KΩ: value R7 -> R16
Connections:
- net VCC: now also H11.1 (VCC)
- net VSS: now also H11.6 (VSS), R1KΩ.1, RV?.3
- net at F8.18 (CHC): now also F8.19 (CHB), F8.20 (CHA), C10.1, R1KΩ.2
- net at F8.22 (SH): now also H11.3 (LOAD)
- net at F8.23 (OPO): now also H11.4 (SD)
- net SND_~{NMI}: now reaches F8.25 (~{IRQ})
- net SND_~{NMI}: now also D3.17 (~{NMI}), R1KΩ.2
- net at F8.39 (PHS): now also H11.5 (PH1)
- new net: H12.1, H12.2 (-)
- new net: H11.2 (BUFF), H12.3 (+)
- new net: H11.7 (RB), H12.5 (+)
- new net: H11.8 (MP), H12.6 (-), H12.7
- new net: C13.1, RV?.2
- new net: 8.2KΩ.2, C10.2
- new net: 8.2KΩ.1, RV?.1
- no-connect marks 31 -> 30
Other:
- moved on the sheet: A10, A12, A13, A15, A16, A17, A2, A4, A5, A7, A8, B1D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
