File: cores/exterm/sch/exterm.kicad_sch (KiCad schematic)
At the start: 71 parts, among them J8 TL7705A, SW1 SW_DIP_x02

Commit message: wip snd
Parts:
- added 2.2Ω: R10, symbol Device:R_US
- added 2.2Ω?: R11, symbol Device:R_US
- added 6.2Ω: R8, symbol Device:R_US
- added C11, C14, C15, C16, C17, C19, C2, C7: 4.7μF, symbol Device:CP1
- added C13: 1μF, symbol Device:CP1
- added C2: 220μF, symbol Device:CP1
- added C20: C1041, symbol Device:C
- added C6: C104, symbol Device:C
- added C9: 10μF, symbol Device:CP1
- added F13: MB7124E, symbol arcade:MB7124E
- added H5, U5: 74LS02, symbol jt74:74LS02
- added J1: Conn_01x04_Male, symbol Connector:Conn_01x04_Male
- added J16: HA1388, symbol hitachi:HA1388
- added JM1: JAMMA_CONN, symbol arcade:JAMMA_CONN
- added R100Ω: R13, symbol Device:R_US
- added R100Ω?: R14, symbol Device:R_US
- added ZD2: 18, Diode_SMD:D_SMF, symbol Diode:BZD27Cxx
- C18: renamed from C13; value 1μF -> 4.7μF
- gave numbers to parts that had none: 1
Connections:
- net COL0: now also F13.1 (A0)
- net COL1: now also F13.2 (A1)
- net COL2: now also F13.3 (A2)
- net COL3: now also F13.4 (A3)
- net COL4: now also F13.5 (A4)
- net COL5: now also F13.16 (A6)
- net COL6: now also F13.17 (A7)
- net COL7: now also F13.18 (A8)
- net COL8: now also F13.19 (A9)
- net VCC: now also G4.26 (VDD), G4.40 (VCC), C2.1, F13.20 (VCC), H5.14 (VCC), J16.10 (VCC), R100Ω.1
- net VSS: now also C18.2, G4.20 (VSS), 2.2Ω?.1, C14.2, C15.2, C17.2, C2.2, C2.2, C20.2, C6.2, C7.2, C9.2, F13.10 (VSS), F13.15 (~{CE}), H5.7 (VSS), J1.1 (Pin_1), J1.2 (Pin_2), J16.9 (VSS)
- net at H12.1, H12.2 (-): now also C11.1
- net at H11.7 (RB), H12.5 (+): now also C9.1
- net at JP1.2 (B), SW1.1, SW1.4: now also J8.2 (~{RESIN})
- net at J8.1 (REF): now also C6.1
- net at J8.3 (CT): now also C7.1
- net at J8.6 (RESET): now also H5.3
- net at J8.7 (SENSE): now also R100Ω.2, R100Ω?.2
- net at C18.1: now also J16.1; no longer RV1.2
- net ~{MR}: now reaches B1.6, G14.2 (MR)
- new net: C16.1, J16.11
- new net: C17.1, J16.2
- new net: C13.1, J16.3
- new net: C14.1, J16.5
- new net: C15.1, J16.6
- new net: C19.1, J16.8
- new net: 2.2Ω?.2, C19.2
- new net: 6.2Ω.2, C11.2
- new net: 2.2Ω.1, C20.1
- new net: C13.2, RV1.2
- new net +12V: C2.1, J1.4 (Pin_4), JM1.6 (+12V), R100Ω?.1, ZD2.1 (K)
- new net -5V: JM1.5 (-5V), ZD2.2 (A)
- new net N.C: 6.2Ω.1, JM1.K (NC)
- new net PIN2PC050CM: J1.3 (Pin_3)
- new net SPEAKER(+): 2.2Ω.2, C16.2, J16.12, JM1.10 (SPEAKER_(+))
- new net SPEAKER(-): J16.7, JM1.L (SPEAKER_(-))
Other:
- added sheet capacitors (capacitors.kicad_sch)
- note added: "NO MOUNTED"
- note added: "PIN16 G15"
- note added: "PIN23PC050"
- note removed: "DEL 19 AL 1 F15"
- note removed: "SE CONECTA A CPU SND?"
- company: (none) -> JOTEGO
- title: (none) -> EXTERMINATION
- moved on the sheet: 8.2KΩ, A10, A12, A13, A15, A16, A17, A2, A4, A5, A7, A8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

Commit message: jamma inputs
Parts:
- added H2: SETA-X1-004, symbol yamaha:SETA-X1-004
- added J1, J2, J5: R_Pack08, symbol Device:R_Pack08
Connections:
- net N.C: now also J5.5 (R5.1)
- net VCC: now also H2.27 (VCC), H2.53 (VCC), J1.1 (R1.1), J1.8 (R8.1), J2.1 (R1.1), J2.8 (R8.1), J5.1 (R1.1), J5.8 (R8.1)
- net VSS: now also H2.1 (VSS), H2.18 (VSS), H2.19 (VSS), H2.20 (VSS), H2.21 (UK), H2.38 (VSS), H2.39 (VSS), H2.42 (VSS), H2.43 (VSS), J1.16 (R1.2), J1.9 (R8.2), J2.16 (R1.2), J2.9 (R8.2), J5.16 (R1.2), J5.9 (R8.2)
- net 1P_START: now reaches JM1.17 (1P_START)
- net 1P_START: now also J5.2 (R2.1)
- net 1P_BNT_3: now reaches JM1.24 (1P_BTN_3)
- net 1P_BNT_3: now also J2.3 (R3.1)
- new net 1P_BNT_1: J5.3 (R3.1)
- new net 1P_BNT_2: J2.2 (R2.1)
- new net 1P_DOWN: J2.4 (R4.1)
- new net 1P_LEFT: H2.17 (UK), J1.7 (R7.1), J2.7 (R7.1)
- new net 1P_RIGHT: H2.16 (UK), J1.6 (R6.1), J2.6 (R6.1)
- new net 1P_UP: J2.5 (R5.1)
- new net 2P_BNT_1: J5.7 (R7.1)
- new net 2P_BNT_2: H2.12 (UK), J1.3 (R3.1)
- new net 2P_BNT_3: J1.2 (R2.1)
- new net 2P_DOWN: H2.14 (UK), J1.4 (R4.1)
- new net 2P_START: J5.6 (R6.1)
- new net 2P_UP: H2.15 (UK), J1.5 (R5.1)
- new net SERVICE: J5.4 (R4.1)
Other:
- note added: "CONTROLS"
- note added: "RC Filters"
- moved on the sheet: JM1, ZD2

Commit message: colmix jamma
Parts:
- removed H2: SETA-X1-004, symbol yamaha:SETA-X1-004
- added H11: PC050CM, symbol arcade:PC050CM
- added H15, H16, H17: R0-012, symbol arcade:R0-012
- added H3: SETA-X1-004, symbol yamaha:SETA-X1-004
- added HH16: SETAX1-003, symbol yamaha:SETAX1-003
- J2, J5: value R_Pack08 -> R_P
Connections:
- net 1P_BNT_2 is gone; now on net VCC: J2.2 (R2.1)
- net 1P_BNT_3 is gone; now on net VCC: J2.3 (R3.1), JM1.24 (1P_BTN_3)
- net 1P_DOWN is gone; now on net VCC: J2.4 (R4.1)
- net 1P_LEFT is gone; now on net VCC: J1.7 (R7.1), J2.7 (R7.1)
- net 1P_RIGHT is gone; now on net VCC: J1.6 (R6.1), J2.6 (R6.1)
- net 1P_UP is gone; now on net VCC: J2.5 (R5.1)
- net +12V: now also JM1.F (+12V)
- net -5V: now also JM1.E (-5V)
- net 1P_BNT_1: now also JM1.22 (1P_BTN_1)
- net 2P_BNT_1: now also JM1.Z (2P_BTN_1)
- net 2P_BNT_2: now also JM1.a (2P_BTN_2)
- net 2P_BNT_3: now also JM1.b (2P_BTN_3)
- net 2P_DOWN: now also JM1.W (2P_DOWN)
- net 2P_START: now also JM1.U (2P_START)
- net 2P_UP: now also JM1.V (2P_UP)
- net N.C: now also JM1.15 (NC)
- net SERVICE: now also JM1.R (SERVICE)
- net SND_A0: now also G4.9 (A0); no longer G4.28 (P11)
- net VCC: now also JM1.18 (1P_UP), JM1.19 (1P_DOWN), JM1.20 (1P_LEFT), JM1.21 (1P_RIGHT), JM1.23 (1P_BTN_2), JM1.3 (VDDA), JM1.4 (+5V), JM1.C (+5V), JM1.D (+5V), JM1.X (2P_LEFT), JM1.Y (2P_RIGHT), H11.21 (VCC), H11.5 (VCC), H11.9 (VCC), H3.27 (VCC), H3.53 (VCC), HH16.42 (VCC)
- net VSS: now also J2.10 (R7.2), J2.11 (R6.2), J2.12 (R5.2), J2.13 (R4.2), J2.14 (R3.2), J2.15 (R2.2), JM1.1 (GND), JM1.14 (VIDEO_GND), JM1.2 (VSSA), JM1.27 (GND), JM1.28 (GND), JM1.A (GND), JM1.B (GND), JM1.e (GND), JM1.f (GND), H11.1 (VSS), H11.11 (VSS), H11.15 (VSS), H11.24 (VSS), H11.6 (VSS), H15.8 (VSS), H16.8 (VSS), H17.8 (VSS), H3.1 (VSS), H3.18 (VSS), H3.19 (VSS), H3.20 (VSS), H3.21 (VSS), H3.3 (1P_BNT_3), H3.36 (VSS), H3.38 (VSS), H3.39 (VSS), H3.4 (1P_BNT_2), H3.42 (VSS), H3.43 (VSS), H3.52 (VSS), H3.6 (1P_DOWN), H3.7 (1P_UP), H3.8 (1P_RIGHT), H3.9 (1P_LEFT), HH16.21 (VSS)
- net P20: now reaches G4.21 (P20)
- net P20: now also H3.37 (P20)
- net P21: now reaches G4.22 (P21)
- net P21: now also H3.41 (P21)
- net P22: now reaches G4.23 (P22)
- net P22: now also H3.40 (P22)
- net P23: now reaches G4.24 (P23)
- net P10: now reaches G4.27 (P10)
- net P10: now also H3.28 (P10), H3.44 (P10)
- net P12: now reaches G4.29 (P12)
- net P12: now also H3.30 (P12), H3.46 (P12)
- net P13: now reaches G4.30 (P13)
- net P13: now also H3.31 (P13), H3.47 (P13)
- net P14: now reaches G4.31 (P14)
- net P14: now also H3.32 (P14), H3.48 (P14)
- net P15: now reaches G4.32 (P15)
- net P15: now also H3.33 (P15), H3.49 (P15)
- net P16: now reaches G4.33 (P16)
- net P16: now also H3.34 (P16), H3.50 (P16)
- net P17: now reaches G4.34 (P17)
- net P17: now also H3.35 (P17), H3.51 (P17)
- net C11: now reaches J5.10 (R7.2)
- net C11: now also H3.13 (2P_BNT_1)
- net C8: now reaches J5.11 (R6.2)
- net C8: now also H3.10 (2P_START)
- net C18: now reaches J5.12 (R5.2)
- net C18: now also H3.24 (N.C)
- net C19: now reaches J5.13 (R4.2)
- net C19: now also H3.25 (SERVICE)
- net C3: now reaches J5.14 (R3.2)
- net C3: now also H3.5 (1P_BNT_1)
- net C0: now reaches J5.15 (R2.2)
- net C0: now also H3.2 (1P_STAR)
- net C15: now reaches J1.10 (R7.2)
- net C15: now also H3.17 (1P_LEFT)
- net C14: now reaches J1.11 (R6.2)
- net C14: now also H3.16 (1P_RIGHT)
- net C13: now reaches J1.12 (R5.2)
- net C13: now also H3.15 (2P_UP)
- net C12: now reaches J1.13 (R4.2)
- net C12: now also H3.14 (2P_DOWN)
- net C10: now reaches J1.14 (R3.2)
- net C10: now also H3.12 (2P_BNT_2)
- net C9: now reaches J1.15 (R2.2)
- net C9: now also H3.11 (2P_BNT_3)
- net RED: now reaches JM1.12 (RED)
- net RED: now also H17.1 (R1)
- net BLUE: now reaches JM1.13 (BLUE)
- net BLUE: now also H16.1 (R1)
- net COIN_1: now reaches JM1.16 (COIN_1)
- net COIN_1: now also H11.27 (COIN_1)
- net 1P_BNT_4: now reaches JM1.25 (1P_BTN_4)
- net 1P_BNT_4: now also JM1.c (2P_BTN_4)
- net 1P_SELECT: now reaches JM1.26 (1P_SELECT)
- net 1P_SELECT: now also JM1.d (2P_SELECT)
- net COIN_CNT_1: now reaches JM1.8 (COIN_CNT_1)
- net COIN_CNT_1: now also H11.16 (COIN_CNT_1)
- net COIN_CNT_2: now reaches JM1.J (COIN_CNT_2)
- net COIN_CNT_2: now also H11.4 (COIN_CNT_2)
- net GREEN: now reaches JM1.N (GREEN)
- net GREEN: now also H15.1 (R1)
- net SYNC: now reaches JM1.P (SYNC)
- net SYNC: now also HH16.22 (UK), HH16.23 (UK)
- net COIN_2: now reaches JM1.T (COIN_2)
- net COIN_2: now also H11.28 (COIN_2)
- new net: H16.3 (R3), HH16.10 (UK)
- new net: H16.4 (R4), HH16.11 (UK)
- new net: H16.5 (R5), HH16.12 (UK)
- new net: H16.6 (R6), HH16.13 (UK)
- new net: H16.7 (R7), HH16.14 (UK)
- new net: H15.2 (R2), HH16.3 (UK)
- new net: H17.2 (R2), HH16.36 (UK)
- new net: H17.3 (R3), HH16.37 (UK)
- new net: H17.4 (R4), HH16.38 (UK)
- new net: H17.5 (R5), HH16.39 (UK)
- new net: H15.3 (R3), HH16.4 (UK)
- new net: H17.6 (R6), HH16.40 (UK)
- new net: H17.7 (R7), HH16.41 (UK)
- new net: H15.4 (R4), HH16.5 (UK)
- new net: H15.5 (R5), HH16.6 (UK)
- new net: H15.6 (R6), HH16.7 (UK)
- new net: H15.7 (R7), HH16.8 (UK)
- new net: H16.2 (R2), HH16.9 (UK)
- new net C16: H11.13 (UK), H3.22 (UK)
- new net C17: H11.14 (UK), H3.23 (UK)
- new net P11: G4.28 (P11), H3.29 (P11), H3.45 (P11)
Other:
- note added: "RC Filters?"
- moved on the sheet: 2.2Ω, 2.2Ω?, 6.2Ω, 8.2KΩ, B11, B12, B2A, B2D, B8, B9, C10, C11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

Commit message: to review
Parts:
- removed unit 2 of B1
- removed unit 3 of B6
- removed unit 4 of B6
- removed unit 3 of C6
- removed unit 3 of G13
- removed HH16: SETAX1-003, symbol yamaha:SETAX1-003
- added C8: C683J, symbol Device:C
- added F17: MB7124E, symbol arcade:MB7124E
- added G15, G17: R_P, symbol Device:R_Pack08
- added R2.2KΩ: R12, symbol Device:R_US
- added U?: SETAX1-003, symbol yamaha:SETAX1-003
- renumbered H17 to H15, U5 to H5
Connections:
- net PIN2PC050CM is gone; now on net CNN1A: J1.3 (Pin_3)
- net PIN4INTEL is gone; now on net ~{RST}: B2.11
- net ?: no longer D6.19 (IO1), D8.12 (IO8)
- net COL0: now also F17.1 (A0)
- net COL1: now also F17.2 (A1)
- net COL2: now also F17.3 (A2)
- net COL3: now also F17.4 (A3)
- net COL4: now also F17.5 (A4)
- net COL5: now also F17.16 (A6)
- net COL6: now also F17.17 (A7)
- net COL7: now also F17.18 (A8)
- net COL8: now also F17.19 (A9)
- net H3: now also B1.1
- net SND_D0: now also G4.12 (D0)
- net SND_D1: now also G4.13 (D1)
- net SND_D2: now also G4.14 (D2)
- net SND_D3: now also G4.15 (D3)
- net SND_D4: now also G4.16 (D4)
- net SND_D5: now also G4.17 (D5)
- net SND_D6: now also G4.18 (D6)
- net SND_D7: now also G4.19 (D7)
- net SYNC: now also U?.22 (UK), U?.23 (UK)
- net VCC: now also B17.29 (~{WDRES), B2.1, B5.1 (~{Mr}), E8.26 (~{RESET}), G4.5 (~{SS}), F17.20 (VCC), U?.18 (UK), U?.42 (VCC)
- net VSS: now also G4.7 (EA), F17.10 (VSS), F17.15 (~{CE}), U?.21 (VSS); no longer J1.1 (Pin_1)
- net XTAL1: now also G15.9 (R8.2)
- net ~{BGTRNSP}: now also B6.4
- net ~{MAIN_A13}: now also B6.5
- net TEST0: now reaches G4.1 (TEST0)
- net TEST0: now also H11.25 (UK)
- net at G4.35 (P24_OBF): now also H5.11
- net at G4.36 (P25_~{IBF}): now also H5.8
- net P26_DRQ: now reaches G4.37 (P26_DRQ)
- net P26_DRQ: now also H5.2
- net at G4.38 (P27_~{DACK}): now also H5.5
- net TEST1: now reaches G4.39 (TEST1)
- net TEST1: now also H11.26 (UK)
- net ~{RST}: now reaches G4.4 (~{RESET})
- net at H5.12: now also H5.3, J8.6 (RESET)
- net ~{OBF}: now reaches H5.13
- net ~{OBF}: now also H11.17 (UK)
- net AQUI: now reaches B1.2
- net AQUI: now also D6.19 (IO1), D8.12 (IO8)
- net at H16.3 (R3): now also U?.31 (UK)
- net at H16.4 (R4): now also U?.32 (UK)
- net at H16.5 (R5): now also U?.33 (UK)
- net at H16.6 (R6): now also U?.34 (UK)
- net at H16.7 (R7): now also U?.35 (UK)
- net at H15.2 (R2): now also U?.29 (UK)
- net at H15.2 (R2): now also U?.36 (UK)
- net at H15.3 (R3): now also U?.37 (UK)
- net at H15.4 (R4): now also U?.38 (UK)
- net at H15.5 (R5): now also U?.39 (UK)
- net at H15.3 (R3): now also U?.28 (UK)
- net at H15.6 (R6): now also U?.40 (UK)
- net at H15.7 (R7): now also U?.41 (UK)
- net at H15.4 (R4): now also U?.27 (UK)
- net at H15.5 (R5): now also U?.26 (UK)
- net at H15.6 (R6): now also U?.25 (UK)
- net at H15.7 (R7): now also U?.24 (UK)
- net at H16.2 (R2): now also U?.30 (UK)
- net at G13.3: now also G13.12
- net at G13.4: now also G13.1, C8.2
- net at G13.13: now also R2.2KΩ.1
- net CNN1B: now reaches H11.10 (UK)
- net CNN1B: now also J1.1 (Pin_1)
- net N.C3: now reaches H11.18 (LOCK-OUT2)
- net N.C3: now also JM1.K (NC)
- net N.C0: now reaches H11.19 (LOCK-OUT3)
- net N.C0: now also JM1.9 (NC)
- net CNN1A: now reaches H11.2 (UK)
- net ~{DACK}: now reaches H11.20 (UK)
- net ~{DACK}: now also H5.4
- net ~{COIN}: now reaches H11.23 (UK)
- net ~{COIN}: now also H5.1
- net ~{IBF}: now reaches H11.8 (UK)
- net ~{IBF}: now also H5.10
- net at B6.6: now also C6.1
- net at H5.9: now also H5.6
- net at G14.1 (~{CP}): now also G13.2
- net at F13.11 (D4): now also G15.12 (R5.2)
- net at F13.12 (D5): now also G15.11 (R6.2)
- net at F13.13 (D6): now also G15.10 (R7.2)
- net at F13.6 (D0): now also G15.16 (R1.2)
- net at F13.7 (D1): now also G15.15 (R2.2)
- net at F13.8 (D2): now also G15.14 (R3.2)
- net at F13.9 (D3): now also G15.13 (R4.2)
- net N.C1: now reaches JM1.11 (NC)
- net N.C1: now also 6.2Ω.1
- net N.C4: now reaches JM1.S (NC)
- net N.C4: now also J5.5 (R5.1)
- removed net N.C: 6.2Ω.1, J5.5 (R5.1), JM1.15 (NC), JM1.K (NC)
- removed net ~{WDRES}: B17.29 (~{WDRES), B2.1, B5.1 (~{Mr}), E8.26 (~{RESET}), J8.5 (~{RESET}), R1KΩ.2
- new net: G15.1 (R1.1), U?.9 (UK)
- new net: G15.2 (R2.1), U?.8 (UK)
- new net: G15.3 (R3.1), U?.7 (UK)
- new net: G15.4 (R4.1), U?.6 (UK)
- new net: G15.5 (R5.1), U?.5 (UK)
- new net: G15.6 (R6.1), U?.4 (UK)
- new net: G15.7 (R7.1), U?.3 (UK)
- new net: G15.8 (R8.1), U?.2 (UK)
- new net: J8.5 (~{RESET}), R1KΩ.2
- new net: C8.1, R2.2KΩ.2
- new net: G17.1 (R1.1), U?.10 (UK)
- new net: F17.13 (D6), G17.10 (R7.2)
- new net: F17.12 (D5), G17.11 (R6.2)
- new net: F17.11 (D4), G17.12 (R5.2)
- new net: F17.9 (D3), G17.13 (R4.2)
- new net: F17.8 (D2), G17.14 (R3.2)
- new net: F17.7 (D1), G17.15 (R2.2)
- new net: F17.6 (D0), G17.16 (R1.2)
- new net: G17.2 (R2.1), U?.11 (UK)
- new net: G17.3 (R3.1), U?.12 (UK)
- new net: G17.4 (R4.1), U?.13 (UK)
- new net: G17.5 (R5.1), U?.14 (UK)
- new net: G17.6 (R6.1), U?.15 (UK)
- new net: G17.7 (R7.1), U?.16 (UK)
- new net: G17.8 (R8.1), U?.17 (UK)
- new net: F17.14 (D7), G17.9 (R8.2)
- no-connect marks 30 -> 47
Other:
- note removed: "PIN19SETA003"
- note removed: "PIN20SETA003"
- note removed: "PIN23PC050"
- note removed: "RC Filters?"
- moved on the sheet: B1A, B6B, C2, C4, C6, C7, G13A, G13B, G13D, G13F, G14, H11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

Commit message: distribution
Parts:
- removed A10, A12, A13, A2, A4, A5, A7, A8, C11, C9: 27C512, Package_DIP:DIP-28_W15.24mm, symbol Memory_EPROM:27C512
- removed A15, B5: 74LS174, symbol jt74:74LS174
- removed A16: 74LS273, symbol jt74:74LS273
- removed A17: 12.000MHz, Oscillator:Oscillator_SMD_Abracon_ASDMB-4Pin_2.5x2.0mm, symbol Oscillator:ASDMB-xxxMHz
- removed unit 4 of B1
- removed unit 5 of B1
- removed unit 1 of B1
- removed unit 6 of B1
- removed unit 3 of B1
- removed B13, C4, C5, E11, E12: 74LS245, symbol jt74:74LS245
- removed B14, C14: 74LS367, symbol jt74:74LS367
- removed B15: YM3909, symbol yamaha:YM3909
- removed B17: YM3906, symbol yamaha:YM3906
- removed unit 2 of B2
- removed unit 1 of B2
- removed unit 3 of B2
- removed unit 2 of B3
- removed unit 1 of B3
- removed unit 2 of B4
- removed unit 1 of B4
- removed unit 1 of B6
- removed unit 2 of B6
- removed unit 2 of B7
- removed C3, D6, D8: PAL16L8, symbol Logic_Programmable:PAL16L8
- removed C4: C101, symbol Device:C
- removed unit 2 of C6
- removed unit 4 of C6
- removed E13, E14, E16, E17: HM6116P-3, symbol arcade:HM6116P-3
- removed E8: Z80CPU, symbol CPU:Z80CPU
- removed F13, F17: MB7124E, symbol arcade:MB7124E
- removed unit 5 of G13
- removed G15, G17: R_P, symbol Device:R_Pack08
- removed H15 (x2), H16: R0-012, symbol arcade:R0-012
- removed R150Ω, R330Ω (x2): R20, symbol Device:R_US
- removed R330Ω: R19, symbol Device:R_US
- removed SW1: SW_DIP_x02, symbol Switch:SW_DIP_x02
- removed U?: SETAX1-003, symbol yamaha:SETAX1-003
- added 1KΩ: R21, symbol Device:R_US
- added C12: C103J, symbol Device:C
- added C21: C104J, symbol Device:C
- added R1MΩ: R18, symbol Device:R_US
- added SW1: SW_Push, symbol Switch:SW_Push
- 8.2KΩ: value R7 -> R9
- C20: value C1041 -> C104J
- R1KΩ: value R1 -> R15
- gave numbers to parts that had none: 2
Connections:
- net GFX_A2 is gone; now on net MAIN_A1: B12.13 (I1c)
- net VCC: no longer J1.6 (R6.1), J1.7 (R7.1), J2.2 (R2.1), J2.3 (R3.1), J2.4 (R4.1), J2.5 (R5.1), J2.6 (R6.1), J2.7 (R7.1), JM1.18 (1P_UP), JM1.19 (1P_DOWN), JM1.20 (1P_LEFT), JM1.21 (1P_RIGHT), JM1.23 (1P_BTN_2), JM1.24 (1P_BTN_3), JM1.X (2P_LEFT), JM1.Y (2P_RIGHT), R1KΩ.1
- net VSS: now also J16.4 (VSS), R1KΩ.2, 1KΩ.1, C12.2, C21.2, SW1.1; no longer 2.2Ω.1, H3.3 (1P_BNT_3), H3.4 (1P_BNT_2), H3.6 (1P_DOWN), H3.7 (1P_UP), H3.8 (1P_RIGHT), H3.9 (1P_LEFT), J2.10 (R7.2), J2.11 (R6.2), J2.12 (R5.2), J2.13 (R4.2), J2.14 (R3.2), J2.15 (R2.2)
- net at J8.2 (~{RESIN}), JP1.2 (B): now also SW1.2
- net at H5.12, H5.3, J8.6 (RESET): now also R1KΩ.1
- net at C8.1, R2.2KΩ.2: now also R1MΩ.1
- net at G13.12, G13.3: now also R1MΩ.2
- net CI/O1: now reaches H11.3 (UK)
- net CI/O1: now also H3.23 (UK)
- net at 8.2KΩ.1, RV1.1: now also 1KΩ.2, C12.1
- net C16: no longer names the net of H11.13 (UK)
- net C16: no longer H3.22 (UK)
- net C17 renamed CI/O2
- net CI/O2: now also H3.22 (UK); no longer H3.23 (UK)
- net MAIN_DB0 renamed SHD0
- net MAIN_DB1 renamed SHD1
- net MAIN_DB2 renamed SHD2
- net MAIN_DB3 renamed SHD3
- net MAIN_DB4 renamed SHD4
- net MAIN_DB5 renamed SHD5
- net MAIN_DB6 renamed SHD6
- net MAIN_DB7 renamed SHD7
- net SND_M0 renamed SHA0
- net SND_M1 renamed SHA1
- net SND_M10 renamed SHA10
- net SND_M11 renamed SHA11
- net SND_M12 renamed SHA12
- net SND_M2 renamed SHA2
- net SND_M3 renamed SHA3
- net SND_M4 renamed SHA4
- net SND_M5 renamed SHA5
- net SND_M6 renamed SHA6
- net SND_M7 renamed SHA7
- net SND_M8 renamed SHA8
- net SND_M9 renamed SHA9
- net ~{COIN} renamed ~{COIN_LOCK}
- net ~{MR} renamed ~{WATCHDOG}
- new net: 2.2Ω.1, C21.1
- new net 1P_BNT_2: J2.2 (R2.1), JM1.23 (1P_BTN_2)
- new net 1P_BNT_3: J2.3 (R3.1), JM1.24 (1P_BTN_3)
- new net 1P_DOWN: J2.4 (R4.1), JM1.19 (1P_DOWN)
- new net 1P_LEFT: J1.7 (R7.1), J2.7 (R7.1), JM1.20 (1P_LEFT), JM1.X (2P_LEFT)
- new net 1P_RIGHT: J1.6 (R6.1), J2.6 (R6.1), JM1.21 (1P_RIGHT), JM1.Y (2P_RIGHT)
- new net 1P_UP: J2.5 (R5.1), JM1.18 (1P_UP)
- new net C1: H3.3 (1P_BNT_3), J2.14 (R3.2)
- new net C2: H3.4 (1P_BNT_2), J2.15 (R2.2)
- new net C4: H3.6 (1P_DOWN), J2.13 (R4.2)
- new net C5: H3.7 (1P_UP), J2.12 (R5.2)
- new net C6: H3.8 (1P_RIGHT), J2.11 (R6.2)
- new net C7: H3.9 (1P_LEFT), J2.10 (R7.2)
- no-connect marks 47 -> 26
Other:
- added sheet colmix (colmix.kicad_sch)
- added sheet gfx (gfx.kicad_sch)
- added sheet main (main.kicad_sch)
- note added: "CABINET I/O"
- note added: "MCU"
- note added: "Shared RAM"
- note removed: "?"
- note removed: "COLMIX"
- note removed: "CONTROLS"
- note removed: "CPU MAIN"
- note removed: "GXF"
- note removed: "MAIN"
- note removed: "NOT MOUNTED"
- note removed: "PIN16 G15"
- note removed: "POSIBLEMENTE PXCLK"
- note removed: "REVISAR"
- note removed: "TRIESTADO?"
- moved on the sheet: 2.2Ω, 6.2Ω, 8.2KΩ, B11, B12, B1G, B2D, B2E, B3C, B4C, B6E, B7C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

Commit message: almost ready
Parts:
- removed 1KΩ: R21, symbol Device:R_US
- removed 2.2Ω: R11, symbol Device:R_US
- removed 2.2Ω: R10, symbol Device:R_US
- removed 6.2Ω: R8, symbol Device:R_US
- removed 8.2KΩ: R9, symbol Device:R_US
- removed B1, G13: 74LS04, symbol jt74:74LS04
- removed B11, B12, B8, B9: 74LS157, symbol jt74:74LS157
- removed B2, B6: 74LS08, symbol jt74:74LS08
- removed B3, B4, B7: 74LS74, symbol jt74:74LS74
- removed C10, C6: C104, symbol Device:C
- removed C11, C14, C15, C16, C17, C18, C19, C2, C7: 4.7μF, symbol Device:CP1
- removed C12: C103J, symbol Device:C
- removed C13: 1μF, symbol Device:CP1
- removed C2: PAL16L8, symbol Logic_Programmable:PAL16L8
- removed C2: 220μF, symbol Device:CP1
- removed C20, C21: C104J, symbol Device:C
- removed C8: MB8464A-10L-LL, symbol fujitsu:MB8464A-10L-LL
- removed C8: C683J, symbol Device:C
- removed C9: 10μF, symbol Device:CP1
- removed D3: Z80CPU, symbol CPU:Z80CPU
- removed E1: 74LS174, symbol jt74:74LS174
- removed E4: 27C512, Package_DIP:DIP-28_W15.24mm, symbol Memory_EPROM:27C512
- removed F8: YM2203, Package_DIP:DIP-40_W15.24mm, symbol yamaha:YM2203
- removed G14: 74HC4024, Package_SO:SOIC-14_3.9x8.7mm_P1.27mm, symbol 74xx:74HC4024
- removed G4: INTEL8742, symbol Intel:INTEL8742
- removed H11: YM3014, Package_DIP:DIP-8_W7.62mm, symbol yamaha:YM3014
- removed H11: PC050CM, symbol arcade:PC050CM
- removed H12: NJM4558, symbol Amplifier_Operational:NJM4558
- removed H5: 74LS02, symbol jt74:74LS02
- removed J1: Conn_01x04_Male, symbol Connector:Conn_01x04_Male
- removed J16: HA1388, symbol hitachi:HA1388
- removed J8: TL7705A, symbol Power_Supervisor:TL7705A
- removed JP1: Jumper_2_Bridged, symbol Jumper:Jumper_2_Bridged
- removed R100Ω: R14, symbol Device:R_US
- removed R100Ω: R13, symbol Device:R_US
- removed R1KΩ: R7, symbol Device:R_US
- removed R1KΩ: R15, symbol Device:R_US
- removed R1KΩ: R16, symbol Device:R_US
- removed R1KΩ: R6, symbol Device:R_US
- removed R1MΩ: R18, symbol Device:R_US
- removed R2.2KΩ: R12, symbol Device:R_US
- removed RV1: R_POT_US, symbol Device:R_POT_US
- removed SW1: SW_Push, symbol Switch:SW_Push
- removed SWA, SWB: SW_DIPS_08, symbol Mod_KC_Symbols:SW_DIPS_08
- ZD2: value 18 -> BZD27C
Connections:
- no-connect marks 26 -> 0
Other:
- added sheet mcu (mcu.kicad_sch)
- added sheet sound (sound.kicad_sch)
- added sheet watchdog (watchdog.kicad_sch)
- sheet colmix ports: added BLUE, DATAEN, DBB[7..0], GDA[7..0], GDB[7..0], GDC[7..0], GDD[0..7], GFX_CLK, GREEN, HC[8..0], RED, SYNC, XTAL1, ~{BGTRNSP}, ~{HBLK}, ~{VSYNC}; removed none
- sheet gfx ports: added DATAEN, DBB[7..0], GDA[7..0], GDB[7..0], GDC[7..0], GDD[7..0], GFXA_~{CS}, GFXB_~{CS}, GFXC_~{CS}, GFXD_~{CS}, GFX_A[11..0], GFX_CLK, HC[8..0], H[4..0], MAB_~{CE}, MAIN_A[15..0], MAIN_D[7..0], MAIN_~{RD}, MBB_~{CE}, SPBANK1, ~{GFX_WR}, ~{HBLK}, ~{MAIN_WR}, ~{VBLK}, ~{VSYNC}, ~{WDRES}, ~{WR}; removed none
- sheet main ports: added CLK_SND, GFXA_~{CS}, GFXB_~{CS}, GFXC_~{CS}, GFXD_~{CS}, GFX_A[11..0], H[4..0], MAB_~{CE}, MAIN_A[15..0], MAIN_D[7..0], MAIN_~{RD}, MBB_~{CE}, PHM, RAM_~{CS1}, RAM_~{WE}, SHD[7..0], SND_D[7..0], SND_SELECT, SND_~{INT}, SND_~{RD}, SND_~{WAIT}, SND_~{WR}, SPBANK1, S_~{IORQ}, XTAL1, YM_~{CS}, ~{BGTRNSP}, ~{GFX_WR}, ~{MAIN_WR}, ~{RESET}, ~{SND_MREQ}, ~{VBLK}, ~{WATCHDOG}, ~{WDRES}, ~{WR}, ~{XTAL2}; removed none
- note removed: "MCU"
- note removed: "NO MOUNTED"
- note removed: "SOUND"
- note removed: "Shared RAM"
- moved on the sheet: H3, J1, J2, J5, JM1

Commit message: terminated exterminator
Parts:
- ZD1: renamed from ZD2; value BZD27C -> BZD27
Connections:
- net +12V: no longer ZD1.1 (K)
- net -5V: now also ZD1.1 (K); no longer ZD1.2 (A)
- net 1P_BNT_4: no longer JM1.c (2P_BTN_4)
- net 1P_LEFT: no longer JM1.X (2P_LEFT)
- net 1P_RIGHT: no longer JM1.Y (2P_RIGHT)
- net 1P_SELECT: no longer JM1.d (2P_SELECT)
- net VCC: now also ZD1.2 (A)
- new net 2P_BNT_4: JM1.c (2P_BTN_4)
- new net 2P_LEFT: JM1.X (2P_LEFT)
- new net 2P_RIGHT: JM1.Y (2P_RIGHT)
- new net 2P_SELECT: JM1.d (2P_SELECT)
Other:
- sheet mcu ports: added P[23..10]; removed none
- moved on the sheet: JM1, ZD1
