File: cores/exterm/sch/exterm.kicad_sch (KiCad schematic)
At the start: 6 parts, among them J1 R_Pack08, J2 R_P, J5 R_P

Commit message: x-004 skutis
Parts:
- removed H3: SETA-X1-004, symbol yamaha:SETA-X1-004
Changed lines of the file:
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@@
     (comment 1 "E.Triana")
   )
-  (junction (at 64.77 186.69) (diameter 0) (color 0 0 0 0)
-  )
-  (junction (at 88.9 184.15) (diameter 0) (color 0 0 0 0)
-  )
   (junction (at 88.9 185.42) (diameter 0) (color 0 0 0 0)
   )
@@
   (junction (at 36.83 144.78) (diameter 0) (color 0 0 0 0)
   )
-  (junction (at 64.77 184.15) (diameter 0) (color 0 0 0 0)
-  )
-  (junction (at 64.77 189.23) (diameter 0) (color 0 0 0 0)
-  )
   (junction (at 26.67 144.78) (diameter 0) (color 0 0 0 0)
   )
-  (junction (at 64.77 181.61) (diameter 0) (color 0 0 0 0)
-  )
-  (junction (at 88.9 189.23) (diameter 0) (color 0 0 0 0)
-  )
   (junction (at 36.83 168.91) (diameter 0) (color 0 0 0 0)
   )
@@
   (junction (at 34.29 33.02) (diameter 0) (color 0 0 0 0)
   )
-  (junction (at 88.9 186.69) (diameter 0) (color 0 0 0 0)
-  )
   (junction (at 34.29 92.71) (diameter 0) (color 0 0 0 0)
   )
@@
     (stroke (width 0) (type default) (color 0 0 0 0))
   )
-  (wire (pts (xy 88.9 189.23) (xy 88.9 191.77))
-    (stroke (width 0) (type default) (color 0 0 0 0))
-  )
   (wire (pts (xy 182.88 30.48) (xy 199.39 30.48))
     (stroke (width 0) (type default) (color 0 0 0 0))
@@
     (stroke (width 0) (type default) (color 0 0 0 0))
   )
-  (wire (pts (xy 64.77 186.69) (xy 64.77 189.23))
-    (stroke (width 0) (type default) (color 0 0 0 0))
-  )
   (wire (pts (xy 82.55 82.55) (xy 95.25 82.55))
     (stroke (width 0) (type default) (color 0 0 0 0))
@@
     (stroke (width 0) (type default) (color 0 0 0 0))
   )
-  (wire (pts (xy 88.9 181.61) (xy 88.9 184.15))
-    (stroke (width 0) (type default) (color 0 0 0 0))
-  )
   (wire (pts (xy 88.9 143.51) (xy 95.25 143.51))
     (stroke (width 0) (type default) (color 0 0 0 0))
@@
     (stroke (width 0) (type default) (color 0 0 0 0))
   )
-  (wire (pts (xy 64.77 185.42) (xy 64.77 186.69))
-    (stroke (width 0) (type default) (color 0 0 0 0))
-  )
   (wire (pts (xy 36.83 161.29) (xy 44.45 161.29))
     (stroke (width 0) (type default) (color 0 0 0 0))
@@
     (stroke (width 0) (type default) (color 0 0 0 0))
   )
-  (wire (pts (xy 64.77 179.07) (xy 64.77 181.61))
+  (wire (pts (xy 64.77 179.07) (xy 64.77 185.42))
     (stroke (width 0) (type default) (color 0 0 0 0))
   )
@@
     (stroke (width 0) (type default) (color 0 0 0 0))
   )
-  (wire (pts (xy 88.9 184.15) (xy 88.9 185.42))
+  (wire (pts (xy 88.9 181.61) (xy 88.9 181.61))
     (stroke (width 0) (type default) (color 0 0 0 0))
   )
@@
     (stroke (width 0) (type default) (color 0 0 0 0))
   )
-  (wire (pts (xy 64.77 189.23) (xy 64.77 191.77))
-    (stroke (width 0) (type default) (color 0 0 0 0))
-  )
   (wire (pts (xy 58.42 135.89) (xy 64.77 135.89))
     (stroke (width 0) (type default) (color 0 0 0 0))
@@
     (stroke (width 0) (type default) (color 0 0 0 0))
   )
+  (wire (pts (xy 64.77 185.42) (xy 64.77 191.77))
+    (stroke (width 0) (type default) (color 0 0 0 0))
+  )
   (wire (pts (xy 215.9 71.12) (xy 229.87 71.12))
     (stroke (width 0) (type default) (color 0 0 0 0))
@@
     (stroke (width 0) (type default) (color 0 0 0 0))
   )
-  (wire (pts (xy 88.9 185.42) (xy 88.9 186.69))
-    (stroke (width 0) (type default) (color 0 0 0 0))
-  )
   (wire (pts (xy 215.9 91.44) (xy 229.87 91.44))
     (stroke (width 0) (type default) (color 0 0 0 0))
@@
     (stroke (width 0) (type default) (color 0 0 0 0))
   )
-  (wire (pts (xy 88.9 186.69) (xy 88.9 189.23))
-    (stroke (width 0) (type default) (color 0 0 0 0))
-  )
   (wire (pts (xy 137.16 63.5) (xy 153.67 63.5))
     (stroke (width 0) (type default) (color 0 0 0 0))
@@
     (stroke (width 0) (type default) (color 0 0 0 0))
   )
+  (wire (pts (xy 88.9 184.15) (xy 88.9 185.42))
+    (stroke (width 0) (type default) (color 0 0 0 0))
+  )
   (wire (pts (xy 215.9 135.89) (xy 229.87 135.89))
     (stroke (width 0) (type default) (color 0 0 0 0))
@@
     (stroke (width 0) (type default) (color 0 0 0 0))
   )
+  (wire (pts (xy 88.9 185.42) (xy 88.9 191.77))
+    (stroke (width 0) (type default) (color 0 0 0 0))
+  )
   (wire (pts (xy 17.78 180.34) (xy 26.67 180.34))
     (stroke (width 0) (type default) (color 0 0 0 0))
@@
     (stroke (width 0) (type default) (color 0 0 0 0))
   )
-  (wire (pts (xy 64.77 184.15) (xy 64.77 185.42))
-    (stroke (width 0) (type default) (color 0 0 0 0))
-  )
   (wire (pts (xy 58.42 163.83) (xy 64.77 163.83))
     (stroke (width 0) (type default) (color 0 0 0 0))
@@
     (stroke (width 0) (type default) (color 0 0 0 0))
   )
-  (wire (pts (xy 64.77 181.61) (xy 64.77 184.15))
-    (stroke (width 0) (type default) (color 0 0 0 0))
-  )
   (wire (pts (xy 76.2 123.19) (xy 77.47 123.19))
     (stroke (width 0) (type default) (color 0 0 0 0))
@@
     (pin "9")
   )
-  (symbol (lib_id "yamaha:SETA-X1-004") (at 77.47 167.64 0) (unit 1)
-    (in_bom yes) (on_board yes)
-    (property "Reference" "H3" (id 0) (at 83.82 124.46 0))
-    (property "Value" "SETA-X1-004" (id 1) (at 77.47 185.42 90))
-    (property "Footprint" "" (id 2) (at 77.47 158.75 90)
-      (effects (font (size 1.27 1.27)) hide)
-    )
-    (property "Datasheet" "" (id 3) (at 77.47 158.75 90)
-      (effects (font (size 1.27 1.27)) hide)
-    )
-    (pin "1")
-    (pin "10")
-    (pin "11")
-    (pin "12")
-    (pin "13")
-    (pin "14")
-    (pin "15")
-    (pin "16")
-    (pin "17")
-    (pin "18")
-    (pin "19")
-    (pin "2")
-    (pin "20")
-    (pin "21")
-    (pin "22")
-    (pin "23")
-    (pin "24")
-    (pin "25")
-    (pin "27")
-    (pin "28")
-    (pin "29")
-    (pin "3")
-    (pin "30")
-    (pin "31")
-    (pin "32")
-    (pin "33")
-    (pin "34")
-    (pin "35")
-    (pin "36")
-    (pin "37")
-    (pin "38")
-    (pin "39")
-    (pin "4")
-    (pin "40")
-    (pin "41")
-    (pin "42")
-    (pin "43")
-    (pin "44")
-    (pin "45")
-    (pin "46")
-    (pin "47")
-    (pin "48")
-    (pin "49")
-    (pin "5")
-    (pin "50")
-    (pin "51")
-    (pin "52")
-    (pin "53")
-    (pin "6")
-    (pin "7")
-    (pin "8")
-    (pin "9")
-  )
   (symbol (lib_id "arcade:JAMMA_CONN") (at 50.8 22.86 0) (unit 1)
     (in_bom yes) (on_board yes)
@@
       (reference "G17") (unit 1) (value "R_P") (footprint "")
     )
-    (path "/b65be5db-dc8a-48f5-b0d7-9101a7f00bd7"
-      (reference "H3") (unit 1) (value "SETA-X1-004") (footprint "")
-    )
     (path "/c6841e36-369c-4ec5-8775-45ccee2f40f8/6c379fdb-aaa4-431a-9d8a-f50c20b60bb1"
