File: cores/exterm/sch/exterm.kicad_sch (KiCad schematic)
At the start: 5 parts, among them J1 R_Pack08, J2 R_P, J5 R_P

Commit message: issues_exterm
Parts:
- added H3: SETA-X1-004, symbol yamaha:SETA-X1-004
Connections:
- net C0: now also H3.2 (1P_STAR)
- net C1: now also H3.3 (1P_BNT_3)
- net C10: now also H3.12 (2P_BNT_2)
- net C11: now also H3.13 (2P_BNT_1)
- net C12: now also H3.14 (2P_DOWN)
- net C13: now also H3.15 (2P_UP)
- net C14: now also H3.16 (1P_RIGHT)
- net C15: now also H3.17 (1P_LEFT)
- net C18: now also H3.24 (N.C)
- net C19: now also H3.25 (SERVICE)
- net C2: now also H3.4 (1P_BNT_2)
- net C3: now also H3.5 (1P_BNT_1)
- net C4: now also H3.6 (1P_DOWN)
- net C5: now also H3.7 (1P_UP)
- net C6: now also H3.8 (1P_RIGHT)
- net C7: now also H3.9 (1P_LEFT)
- net C8: now also H3.10 (2P_START)
- net C9: now also H3.11 (2P_BNT_3)
- net CI/O1: now also H3.23 (UK)
- net CI/O2: now also H3.22 (UK)
- net P10: now also H3.28 (P10), H3.44 (X10)
- net P11: now also H3.29 (P11), H3.45 (X11)
- net P12: now also H3.30 (P12), H3.46 (X12)
- net P13: now also H3.31 (P13), H3.47 (X13)
- net P14: now also H3.32 (P14), H3.48 (X14)
- net P15: now also H3.33 (P15), H3.49 (X15)
- net P16: now also H3.34 (P16), H3.50 (X16)
- net P17: now also H3.35 (P17), H3.51 (X17)
- net P20: now also H3.37 (P20)
- net P21: now also H3.41 (P21)
- net P22: now also H3.40 (P22)
- net VCC: now also H3.27 (VCC), H3.53 (VCC)
- net VSS: now also H3.1 (VSS), H3.18 (VSS), H3.19 (VSS), H3.20 (VSS), H3.21 (VSS), H3.36 (VSS), H3.38 (VSS), H3.39 (VSS), H3.42 (VSS), H3.43 (VSS), H3.52 (VSS)
Other:
- sheet main ports: added ~{SND_RST}, ~{SND_SELECT}; removed SND_SELECT, ~{RESET}
- sheet sound ports: added ~{SND_RST}, ~{SND_SELECT}; removed SND_SELECT, ~{RESET}
Changed lines of the file:
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@@
     (comment 1 "E.Triana")
   )
+  (junction (at 88.9 189.23) (diameter 0) (color 0 0 0 0)
+  )
   (junction (at 88.9 185.42) (diameter 0) (color 0 0 0 0)
   )
+  (junction (at 88.9 184.15) (diameter 0) (color 0 0 0 0)
+  )
   (junction (at 95.25 92.71) (diameter 0) (color 0 0 0 0)
   )
@@
   (junction (at 36.83 144.78) (diameter 0) (color 0 0 0 0)
   )
+  (junction (at 64.77 186.69) (diameter 0) (color 0 0 0 0)
+  )
   (junction (at 26.67 144.78) (diameter 0) (color 0 0 0 0)
   )
+  (junction (at 64.77 184.15) (diameter 0) (color 0 0 0 0)
+  )
+  (junction (at 64.77 189.23) (diameter 0) (color 0 0 0 0)
+  )
   (junction (at 36.83 168.91) (diameter 0) (color 0 0 0 0)
   )
   (junction (at 25.4 35.56) (diameter 0) (color 0 0 0 0)
   )
+  (junction (at 64.77 181.61) (diameter 0) (color 0 0 0 0)
+  )
   (junction (at 34.29 33.02) (diameter 0) (color 0 0 0 0)
   )
+  (junction (at 88.9 186.69) (diameter 0) (color 0 0 0 0)
+  )
   (junction (at 34.29 92.71) (diameter 0) (color 0 0 0 0)
   )
@@
     (stroke (width 0) (type default) (color 0 0 0 0))
   )
+  (wire (pts (xy 88.9 189.23) (xy 88.9 191.77))
+    (stroke (width 0) (type default) (color 0 0 0 0))
+  )
   (bus (pts (xy 97.79 151.13) (xy 97.79 148.59))
     (stroke (width 0) (type default) (color 0 0 0 0))
@@
     (stroke (width 0) (type default) (color 0 0 0 0))
   )
+  (wire (pts (xy 88.9 181.61) (xy 88.9 184.15))
+    (stroke (width 0) (type default) (color 0 0 0 0))
+  )
   (wire (pts (xy 215.9 151.13) (xy 229.87 151.13))
     (stroke (width 0) (type default) (color 0 0 0 0))
@@
     (stroke (width 0) (type default) (color 0 0 0 0))
   )
-  (wire (pts (xy 64.77 179.07) (xy 64.77 185.42))
+  (wire (pts (xy 64.77 179.07) (xy 64.77 181.61))
+    (stroke (width 0) (type default) (color 0 0 0 0))
+  )
+  (wire (pts (xy 88.9 186.69) (xy 88.9 189.23))
     (stroke (width 0) (type default) (color 0 0 0 0))
   )
@@
     (stroke (width 0) (type default) (color 0 0 0 0))
   )
-  (wire (pts (xy 88.9 181.61) (xy 88.9 181.61))
-    (stroke (width 0) (type default) (color 0 0 0 0))
-  )
   (wire (pts (xy 34.29 67.31) (xy 46.99 67.31))
     (stroke (width 0) (type default) (color 0 0 0 0))
@@
     (stroke (width 0) (type default) (color 0 0 0 0))
   )
+  (wire (pts (xy 64.77 189.23) (xy 64.77 191.77))
+    (stroke (width 0) (type default) (color 0 0 0 0))
+  )
   (wire (pts (xy 82.55 69.85) (xy 95.25 69.85))
     (stroke (width 0) (type default) (color 0 0 0 0))
@@
     (stroke (width 0) (type default) (color 0 0 0 0))
   )
-  (wire (pts (xy 88.9 176.53) (xy 95.25 176.53))
+  (wire (pts (xy 64.77 171.45) (xy 58.42 171.45))
     (stroke (width 0) (type default) (color 0 0 0 0))
   )
@@
     (stroke (width 0) (type default) (color 0 0 0 0))
   )
-  (wire (pts (xy 64.77 185.42) (xy 64.77 191.77))
+  (wire (pts (xy 64.77 185.42) (xy 64.77 186.69))
     (stroke (width 0) (type default) (color 0 0 0 0))
   )
@@
     (stroke (width 0) (type default) (color 0 0 0 0))
   )
+  (wire (pts (xy 64.77 181.61) (xy 64.77 184.15))
+    (stroke (width 0) (type default) (color 0 0 0 0))
+  )
   (wire (pts (xy 26.67 166.37) (xy 26.67 168.91))
     (stroke (width 0) (type default) (color 0 0 0 0))
@@
     (stroke (width 0) (type default) (color 0 0 0 0))
   )
+  (wire (pts (xy 64.77 186.69) (xy 64.77 189.23))
+    (stroke (width 0) (type default) (color 0 0 0 0))
+  )
   (wire (pts (xy 34.29 80.01) (xy 46.99 80.01))
     (stroke (width 0) (type default) (color 0 0 0 0))
@@
     (stroke (width 0) (type default) (color 0 0 0 0))
   )
+  (wire (pts (xy 64.77 184.15) (xy 64.77 185.42))
+    (stroke (width 0) (type default) (color 0 0 0 0))
+  )
   (bus (pts (xy 182.88 35.56) (xy 199.39 35.56))
     (stroke (width 0) (type default) (color 0 0 0 0))
   )
-  (wire (pts (xy 88.9 179.07) (xy 95.25 179.07))
+  (wire (pts (xy 64.77 168.91) (xy 58.42 168.91))
     (stroke (width 0) (type default) (color 0 0 0 0))
   )
@@
     (stroke (width 0) (type default) (color 0 0 0 0))
   )
-  (wire (pts (xy 88.9 185.42) (xy 88.9 191.77))
+  (wire (pts (xy 88.9 185.42) (xy 88.9 186.69))
     (stroke (width 0) (type default) (color 0 0 0 0))
   )
@@
     (effects (font (size 1.27 1.27)) (justify left bottom))
   )
-  (label "SND_SELECT" (at 199.39 86.36 180)
+  (label "~{SND_SELECT}" (at 199.39 86.36 180)
     (effects (font (size 1.27 1.27)) (justify right bottom))
   )
@@
     (effects (font (size 1.27 1.27)) (justify left bottom))
   )
-  (label "~{RESET}" (at 215.9 128.27 0)
+  (label "~{SND_RST}" (at 215.9 128.27 0)
     (effects (font (size 1.27 1.27)) (justify left bottom))
   )
@@
     (effects (font (size 1.27 1.27)) (justify right bottom))
   )
-  (label "SND_SELECT" (at 215.9 118.11 0)
+  (label "~{SND_SELECT}" (at 215.9 118.11 0)
     (effects (font (size 1.27 1.27)) (justify left bottom))
   )
@@
     (effects (font (size 1.27 1.27)) (justify right bottom))
   )
-  (label "~{RESET}" (at 199.39 58.42 180)
+  (label "~{SND_RST}" (at 199.39 58.42 180)
     (effects (font (size 1.27 1.27)) (justify right bottom))
   )
@@
     (effects (font (size 1.27 1.27)) (justify right bottom))
   )
-  (label "CI{slash}O1" (at 95.25 176.53 180)
-    (effects (font (size 1.27 1.27)) (justify right bottom))
+  (label "CI{slash}O1" (at 58.42 171.45 0)
+    (effects (font (size 1.27 1.27)) (justify left bottom))
   )
   (label "2P_DOWN" (at 17.78 177.8 0)
@@
     (effects (font (size 1.27 1.27)) (justify left bottom))
   )
-  (label "CI{slash}O2" (at 95.25 179.07 180)
-    (effects (font (size 1.27 1.27)) (justify right bottom))
+  (label "CI{slash}O2" (at 58.42 168.91 0)
+    (effects (font (size 1.27 1.27)) (justify left bottom))
   )
   (label "C18" (at 58.42 173.99 0)
@@
     (pin "9")
   )
+  (symbol (lib_id "yamaha:SETA-X1-004") (at 77.47 167.64 0) (unit 1)
+    (in_bom yes) (on_board yes)
+    (property "Reference" "H3" (id 0) (at 83.82 124.46 0))
+    (property "Value" "SETA-X1-004" (id 1) (at 77.47 185.42 90))
+    (property "Footprint" "" (id 2) (at 77.47 158.75 90)
+      (effects (font (size 1.27 1.27)) hide)
+    )
+    (property "Datasheet" "" (id 3) (at 77.47 158.75 90)
+      (effects (font (size 1.27 1.27)) hide)
+    )
+    (pin "1")
+    (pin "10")
+    (pin "11")
+    (pin "12")
+    (pin "13")
+    (pin "14")
+    (pin "15")
+    (pin "16")
+    (pin "17")
+    (pin "18")
+    (pin "19")
+    (pin "2")
+    (pin "20")
+    (pin "21")
+    (pin "22")
+    (pin "23")
+    (pin "24")
+    (pin "25")
+    (pin "27")
+    (pin "28")
+    (pin "29")
+    (pin "3")
+    (pin "30")
+    (pin "31")
+    (pin "32")
+    (pin "33")
+    (pin "34")
+    (pin "35")
+    (pin "36")
+    (pin "37")
+    (pin "38")
+    (pin "39")
+    (pin "4")
+    (pin "40")
+    (pin "41")
+    (pin "42")
+    (pin "43")
+    (pin "44")
+    (pin "45")
+    (pin "46")
+    (pin "47")
+    (pin "48")
+    (pin "49")
+    (pin "5")
+    (pin "50")
+    (pin "51")
+    (pin "52")
+    (pin "53")
+    (pin "6")
+    (pin "7")
+    (pin "8")
+    (pin "9")
+  )
   (symbol (lib_name "BZD27Cxx_1") (lib_id "Diode:BZD27Cxx") (at 20.32 35.56 180) (unit 1)
     (in_bom yes) (on_board yes)
@@
       (effects (font (size 1.27 1.27)) (justify left))
     )
-    (pin "~{RESET}" output (at 182.88 58.42 0)
+    (pin "~{SND_RST}" output (at 182.88 58.42 0)
       (effects (font (size 1.27 1.27)) (justify right))
     )
@@
       (effects (font (size 1.27 1.27)) (justify right))
     )
-    (pin "SND_SELECT" output (at 182.88 86.36 0)
+    (pin "~{SND_SELECT}" output (at 182.88 86.36 0)
       (effects (font (size 1.27 1.27)) (justify right))
     )
@@
       (effects (font (size 1.27 1.27)) (justify left))
     )
-    (pin "SND_SELECT" input (at 229.87 118.11 180)
+    (pin "~{SND_SELECT}" input (at 229.87 118.11 180)
       (effects (font (size 1.27 1.27)) (justify left))
     )
@@
       (effects (font (size 1.27 1.27)) (justify left))
     )
-    (pin "~{RESET}" input (at 229.87 128.27 180)
+    (pin "~{SND_RST}" input (at 229.87 128.27 180)
       (effects (font (size 1.27 1.27)) (justify left))
     )
@@
       (reference "G17") (unit 1) (value "R_P") (footprint "")
     )
+    (path "/44487ed6-2123-4ff8-95e9-ef90a6083a30"
+      (reference "H3") (unit 1) (value "SETA-X1-004") (footprint "")
+    )
     (path "/c6841e36-369c-4ec5-8775-45ccee2f40f8/6c379fdb-aaa4-431a-9d8a-f50c20b60bb1"

Commit message: exterm_kiwi
Parts:
- removed H3: SETA-X1-004, symbol yamaha:SETA-X1-004
Other:
- sheet main ports: added ~{SND_SELECT} ; removed ~{SND_SELECT}
- sheet sound ports: added ~{SND_SELECT} ; removed ~{SND_SELECT}
Changed lines of the file:
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@@
     (comment 1 "E.Triana")
   )
-  (junction (at 88.9 189.23) (diameter 0) (color 0 0 0 0)
-  )
   (junction (at 88.9 185.42) (diameter 0) (color 0 0 0 0)
   )
-  (junction (at 88.9 184.15) (diameter 0) (color 0 0 0 0)
-  )
   (junction (at 95.25 92.71) (diameter 0) (color 0 0 0 0)
   )
@@
   (junction (at 36.83 144.78) (diameter 0) (color 0 0 0 0)
   )
-  (junction (at 64.77 186.69) (diameter 0) (color 0 0 0 0)
-  )
   (junction (at 26.67 144.78) (diameter 0) (color 0 0 0 0)
   )
-  (junction (at 64.77 184.15) (diameter 0) (color 0 0 0 0)
-  )
-  (junction (at 64.77 189.23) (diameter 0) (color 0 0 0 0)
-  )
   (junction (at 36.83 168.91) (diameter 0) (color 0 0 0 0)
   )
   (junction (at 25.4 35.56) (diameter 0) (color 0 0 0 0)
   )
-  (junction (at 64.77 181.61) (diameter 0) (color 0 0 0 0)
-  )
   (junction (at 34.29 33.02) (diameter 0) (color 0 0 0 0)
   )
-  (junction (at 88.9 186.69) (diameter 0) (color 0 0 0 0)
-  )
   (junction (at 34.29 92.71) (diameter 0) (color 0 0 0 0)
   )
@@
     (stroke (width 0) (type default) (color 0 0 0 0))
   )
-  (wire (pts (xy 88.9 189.23) (xy 88.9 191.77))
-    (stroke (width 0) (type default) (color 0 0 0 0))
-  )
   (bus (pts (xy 97.79 151.13) (xy 97.79 148.59))
     (stroke (width 0) (type default) (color 0 0 0 0))
@@
     (stroke (width 0) (type default) (color 0 0 0 0))
   )
-  (wire (pts (xy 88.9 181.61) (xy 88.9 184.15))
-    (stroke (width 0) (type default) (color 0 0 0 0))
-  )
   (wire (pts (xy 215.9 151.13) (xy 229.87 151.13))
     (stroke (width 0) (type default) (color 0 0 0 0))
@@
     (stroke (width 0) (type default) (color 0 0 0 0))
   )
-  (wire (pts (xy 64.77 179.07) (xy 64.77 181.61))
-    (stroke (width 0) (type default) (color 0 0 0 0))
-  )
-  (wire (pts (xy 88.9 186.69) (xy 88.9 189.23))
+  (wire (pts (xy 64.77 179.07) (xy 64.77 185.42))
     (stroke (width 0) (type default) (color 0 0 0 0))
   )
@@
     (stroke (width 0) (type default) (color 0 0 0 0))
   )
-  (wire (pts (xy 64.77 189.23) (xy 64.77 191.77))
-    (stroke (width 0) (type default) (color 0 0 0 0))
-  )
   (wire (pts (xy 82.55 69.85) (xy 95.25 69.85))
     (stroke (width 0) (type default) (color 0 0 0 0))
@@
     (stroke (width 0) (type default) (color 0 0 0 0))
   )
-  (wire (pts (xy 64.77 171.45) (xy 58.42 171.45))
+  (wire (pts (xy 88.9 176.53) (xy 95.25 176.53))
     (stroke (width 0) (type default) (color 0 0 0 0))
   )
@@
     (stroke (width 0) (type default) (color 0 0 0 0))
   )
-  (wire (pts (xy 64.77 185.42) (xy 64.77 186.69))
+  (wire (pts (xy 64.77 185.42) (xy 64.77 191.77))
     (stroke (width 0) (type default) (color 0 0 0 0))
   )
@@
     (stroke (width 0) (type default) (color 0 0 0 0))
   )
-  (wire (pts (xy 64.77 181.61) (xy 64.77 184.15))
-    (stroke (width 0) (type default) (color 0 0 0 0))
-  )
   (wire (pts (xy 26.67 166.37) (xy 26.67 168.91))
     (stroke (width 0) (type default) (color 0 0 0 0))
@@
     (stroke (width 0) (type default) (color 0 0 0 0))
   )
-  (wire (pts (xy 64.77 186.69) (xy 64.77 189.23))
-    (stroke (width 0) (type default) (color 0 0 0 0))
-  )
   (wire (pts (xy 34.29 80.01) (xy 46.99 80.01))
     (stroke (width 0) (type default) (color 0 0 0 0))
@@
     (stroke (width 0) (type default) (color 0 0 0 0))
   )
-  (wire (pts (xy 64.77 184.15) (xy 64.77 185.42))
-    (stroke (width 0) (type default) (color 0 0 0 0))
-  )
   (bus (pts (xy 182.88 35.56) (xy 199.39 35.56))
     (stroke (width 0) (type default) (color 0 0 0 0))
   )
-  (wire (pts (xy 64.77 168.91) (xy 58.42 168.91))
+  (wire (pts (xy 88.9 179.07) (xy 95.25 179.07))
     (stroke (width 0) (type default) (color 0 0 0 0))
   )
@@
     (stroke (width 0) (type default) (color 0 0 0 0))
   )
-  (wire (pts (xy 88.9 185.42) (xy 88.9 186.69))
+  (wire (pts (xy 88.9 185.42) (xy 88.9 191.77))
     (stroke (width 0) (type default) (color 0 0 0 0))
   )
@@
     (effects (font (size 1.27 1.27)) (justify left bottom))
   )
-  (label "~{SND_SELECT}" (at 199.39 86.36 180)
+  (label "~{SND_SELECT} " (at 199.39 86.36 180)
     (effects (font (size 1.27 1.27)) (justify right bottom))
   )
@@
     (effects (font (size 1.27 1.27)) (justify right bottom))
   )
-  (label "~{SND_SELECT}" (at 215.9 118.11 0)
+  (label "~{SND_SELECT} " (at 215.9 118.11 0)
     (effects (font (size 1.27 1.27)) (justify left bottom))
   )
@@
     (effects (font (size 1.27 1.27)) (justify right bottom))
   )
-  (label "CI{slash}O1" (at 58.42 171.45 0)
-    (effects (font (size 1.27 1.27)) (justify left bottom))
+  (label "CI{slash}O1" (at 95.25 176.53 180)
+    (effects (font (size 1.27 1.27)) (justify right bottom))
   )
   (label "2P_DOWN" (at 17.78 177.8 0)
@@
     (effects (font (size 1.27 1.27)) (justify left bottom))
   )
-  (label "CI{slash}O2" (at 58.42 168.91 0)
-    (effects (font (size 1.27 1.27)) (justify left bottom))
+  (label "CI{slash}O2" (at 95.25 179.07 180)
+    (effects (font (size 1.27 1.27)) (justify right bottom))
   )
   (label "C18" (at 58.42 173.99 0)
@@
     (pin "9")
   )
-  (symbol (lib_id "yamaha:SETA-X1-004") (at 77.47 167.64 0) (unit 1)
-    (in_bom yes) (on_board yes)
-    (property "Reference" "H3" (id 0) (at 83.82 124.46 0))
-    (property "Value" "SETA-X1-004" (id 1) (at 77.47 185.42 90))
-    (property "Footprint" "" (id 2) (at 77.47 158.75 90)
-      (effects (font (size 1.27 1.27)) hide)
-    )
-    (property "Datasheet" "" (id 3) (at 77.47 158.75 90)
-      (effects (font (size 1.27 1.27)) hide)
-    )
-    (pin "1")
-    (pin "10")
-    (pin "11")
-    (pin "12")
-    (pin "13")
-    (pin "14")
-    (pin "15")
-    (pin "16")
-    (pin "17")
-    (pin "18")
-    (pin "19")
-    (pin "2")
-    (pin "20")
-    (pin "21")
-    (pin "22")
-    (pin "23")
-    (pin "24")
-    (pin "25")
-    (pin "27")
-    (pin "28")
-    (pin "29")
-    (pin "3")
-    (pin "30")
-    (pin "31")
-    (pin "32")
-    (pin "33")
-    (pin "34")
-    (pin "35")
-    (pin "36")
-    (pin "37")
-    (pin "38")
-    (pin "39")
-    (pin "4")
-    (pin "40")
-    (pin "41")
-    (pin "42")
-    (pin "43")
-    (pin "44")
-    (pin "45")
-    (pin "46")
-    (pin "47")
-    (pin "48")
-    (pin "49")
-    (pin "5")
-    (pin "50")
-    (pin "51")
-    (pin "52")
-    (pin "53")
-    (pin "6")
-    (pin "7")
-    (pin "8")
-    (pin "9")
-  )
   (symbol (lib_name "BZD27Cxx_1") (lib_id "Diode:BZD27Cxx") (at 20.32 35.56 180) (unit 1)
     (in_bom yes) (on_board yes)
@@
       (effects (font (size 1.27 1.27)) (justify right))
     )
-    (pin "~{SND_SELECT}" output (at 182.88 86.36 0)
+    (pin "~{SND_SELECT} " output (at 182.88 86.36 0)
       (effects (font (size 1.27 1.27)) (justify right))
     )
@@
       (effects (font (size 1.27 1.27)) (justify left))
     )
-    (pin "~{SND_SELECT}" input (at 229.87 118.11 180)
+    (pin "~{SND_SELECT} " input (at 229.87 118.11 180)
       (effects (font (size 1.27 1.27)) (justify left))
     )
@@
       (reference "G17") (unit 1) (value "R_P") (footprint "")
     )
-    (path "/44487ed6-2123-4ff8-95e9-ef90a6083a30"
-      (reference "H3") (unit 1) (value "SETA-X1-004") (footprint "")
-    )
     (path "/c6841e36-369c-4ec5-8775-45ccee2f40f8/6c379fdb-aaa4-431a-9d8a-f50c20b60bb1"

Commit message: issues_exterm
Parts:
- added H3: SETA-X1-004, symbol yamaha:SETA-X1-004
Connections:
- net VSS is gone; now on net GNDPWR: J1.16 (R1.2), J1.9 (R8.2), J2.16 (R1.2), J2.9 (R8.2), J5.16 (R1.2), J5.9 (R8.2), JM1.1 (GND), JM1.14 (VIDEO_GND), JM1.2 (VSSA), JM1.27 (GND), JM1.28 (GND), JM1.A (GND), JM1.B (GND), JM1.e (GND), JM1.f (GND)
- net 1P_BNT_1: no longer JM1.22 (1P_BTN_1)
- net 1P_BNT_2: no longer JM1.23 (1P_BTN_2)
- net 1P_BNT_3: no longer JM1.24 (1P_BTN_3)
- net 2P_BNT_1: no longer JM1.Z (2P_BTN_1)
- net 2P_BNT_2: no longer JM1.a (2P_BTN_2)
- net 2P_BNT_3: no longer JM1.b (2P_BTN_3)
- net C0: now also H3.2 (1P_STAR)
- net C1: now also H3.3 (1P_BNT_3)
- net C10: now also H3.12 (2P_BNT_2)
- net C11: now also H3.13 (2P_BNT_1)
- net C12: now also H3.14 (2P_DOWN)
- net C13: now also H3.15 (2P_UP)
- net C14: now also H3.16 (2P_RIGHT)
- net C15: now also H3.17 (2P_LEFT)
- net C18: now also H3.24 (INC1)
- net C19: now also H3.25 (INC0)
- net C2: now also H3.4 (1P_BNT_2)
- net C3: now also H3.5 (1P_BNT_1)
- net C4: now also H3.6 (1P_DOWN)
- net C5: now also H3.7 (1P_UP)
- net C6: now also H3.8 (1P_RIGHT)
- net C7: now also H3.9 (1P_LEFT)
- net C8: now also H3.10 (2P_START)
- net C9: now also H3.11 (2P_BNT_3)
- net CI/O1: now also H3.23 (INC2)
- net CI/O2: now also H3.22 (INC3)
- net P10: now also H3.28 (P10), H3.44 (X10)
- net P11: now also H3.29 (P11), H3.45 (X11)
- net P12: now also H3.30 (P12), H3.46 (X12)
- net P13: now also H3.31 (P13), H3.47 (X13)
- net P14: now also H3.32 (P14), H3.48 (X14)
- net P15: now also H3.33 (P15), H3.49 (X15)
- net P16: now also H3.34 (P16), H3.50 (X16)
- net P17: now also H3.35 (P17), H3.51 (X17)
- net P20: now also H3.37 (P20)
- net P21: now also H3.41 (P21)
- net P22: now also H3.40 (P22)
- net VCC: now also H3.27 (VCC), H3.53 (VCC)
- net -5V renamed GNDPWR
- net GNDPWR: now also H3.1 (VSS), H3.18 (VSS), H3.19 (VSS), H3.20 (VSS), H3.21 (VSS), H3.36 (VSS), H3.38 (VSS), H3.39 (VSS), H3.42 (VSS), H3.43 (VSS), H3.52 (VSS)
- net 1P_BNT_4 renamed 1P_BTN_4
- net 2P_BNT_4 renamed 2P_BTN_4
- new net 1P_BTN_1: JM1.22 (1P_BTN_1)
- new net 1P_BTN_2: JM1.23 (1P_BTN_2)
- new net 1P_BTN_3: JM1.24 (1P_BTN_3)
- new net 2P_BTN_1: JM1.Z (2P_BTN_1)
- new net 2P_BTN_2: JM1.a (2P_BTN_2)
- new net 2P_BTN_3: JM1.b (2P_BTN_3)
Other:
- moved on the sheet: JM1, ZD1

Commit message: Extermination schematics updated (issue #33)
Connections:
- net 1P_BNT_1 is gone; now on net 1P_BTN_1: J5.3 (R3.1)
- net 1P_BNT_2 is gone; now on net 1P_BTN_2: J2.2 (R2.1)
- net 1P_BNT_3 is gone; now on net 1P_BTN_3: J2.3 (R3.1)
- net 2P_BNT_1 is gone; now on net 2P_BTN_1: J5.7 (R7.1)
- net 2P_BNT_2 is gone; now on net 2P_BTN_2: J1.3 (R3.1)
- net 2P_BNT_3 is gone; now on net 2P_BTN_3: J1.2 (R2.1)
- net C0 is gone; now on net 1P_START: H3.2 (1P_STAR), J5.15 (R2.2)
- net C1 is gone; now on net 1P_BTN_3: H3.3 (1P_BNT_3), J2.14 (R3.2)
- net C10 is gone; now on net 2P_BTN_2: H3.12 (2P_BNT_2), J1.14 (R3.2)
- net C11 is gone; now on net 2P_BTN_1: H3.13 (2P_BNT_1), J5.10 (R7.2)
- net C12 is gone; now on net 2P_DOWN: H3.14 (2P_DOWN), J1.13 (R4.2)
- net C13 is gone; now on net 2P_UP: H3.15 (2P_UP), J1.12 (R5.2)
- net C14 is gone; now on net 2P_RIGHT: H3.16 (2P_RIGHT), J1.11 (R6.2)
- net C15 is gone; now on net 2P_LEFT: H3.17 (2P_LEFT), J1.10 (R7.2)
- net C19 is gone; now on net SERVICE: H3.25 (SERVICE), J5.13 (R4.2)
- net C2 is gone; now on net 1P_BTN_2: H3.4 (1P_BNT_2), J2.15 (R2.2)
- net C3 is gone; now on net 1P_BTN_1: H3.5 (1P_BNT_1), J5.14 (R3.2)
- net C4 is gone; now on net 1P_DOWN: H3.6 (1P_DOWN), J2.13 (R4.2)
- net C5 is gone; now on net 1P_UP: H3.7 (1P_UP), J2.12 (R5.2)
- net C6 is gone; now on net 1P_RIGHT: H3.8 (1P_RIGHT), J2.11 (R6.2)
- net C7 is gone; now on net 1P_LEFT: H3.9 (1P_LEFT), J2.10 (R7.2)
- net C8 is gone; now on net 2P_START: H3.10 (2P_START), J5.11 (R6.2)
- net C9 is gone; now on net 2P_BTN_3: H3.11 (2P_BNT_3), J1.15 (R2.2)
- net 1P_BTN_4: no longer names the net of JM1.25 (1P_BTN_4)
- net 1P_SELECT: no longer names the net of JM1.26 (1P_SELECT)
- net 2P_BTN_4: no longer names the net of JM1.c (2P_BTN_4)
- net 2P_SELECT: no longer names the net of JM1.d (2P_SELECT)
- net C18 renamed TILT
- net GNDPWR renamed VSS
- net VSS: no longer JM1.5 (-5V), JM1.E (-5V), ZD1.1 (K)
- new net -5V: JM1.5 (-5V), JM1.E (-5V), ZD1.1 (K)
- no-connect marks 0 -> 4
Other:
- sheet colmix ports: added H1B, VD[7..0]; removed DBB[7..0], XTAL1
- sheet gfx ports: added H3B, H4B, VA[11..0], VD[15..0]; removed DBB[7..0], GFX_A[11..0], SPBANK1
- sheet main ports: added H1B, H3B, H4B, VA[11..0]; removed GFX_A[11..0], SPBANK1, XTAL1, ~{XTAL2}
- sheet mcu ports: added H1B; removed XTAL1, ~{XTAL2}
