File: cores/exterm/sch/colmix.kicad_sch (KiCad schematic)
At the start: 9 parts

Commit message: almost ready
Changed lines of the file:
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@@
+    (stroke (width 0) (type default) (color 0 0 0 0))
+  )
+  (bus (pts (xy 106.68 38.1) (xy 116.84 38.1))
     (stroke (width 0) (type default) (color 0 0 0 0))
   )
@@
     (stroke (width 0) (type default) (color 0 0 0 0))
   )
-  (bus (pts (xy 39.37 69.85) (xy 54.61 69.85))
+  (bus (pts (xy 48.26 69.85) (xy 54.61 69.85))
     (stroke (width 0) (type default) (color 0 0 0 0))
   )
@@
   )
   (wire (pts (xy 57.15 116.84) (xy 68.58 116.84))
+    (stroke (width 0) (type default) (color 0 0 0 0))
+  )
+  (bus (pts (xy 106.68 46.99) (xy 106.68 38.1))
     (stroke (width 0) (type default) (color 0 0 0 0))
   )
@@
     (effects (font (size 1.27 1.27)) (justify left bottom))
   )
+  (label "COL[8..0]" (at 116.84 38.1 180)
+    (effects (font (size 1.27 1.27)) (justify right bottom))
+  )
   (label "DBB3" (at 63.5 62.23 180)
     (effects (font (size 1.27 1.27)) (justify right bottom))
@@
   )
   (label "GDC2" (at 57.15 142.24 0)
-    (effects (font (size 1.27 1.27)) (justify left bottom))
-  )
-  (label "HC[8..0]" (at 39.37 69.85 0)
     (effects (font (size 1.27 1.27)) (justify left bottom))
   )
@@
   (hierarchical_label "RED" (shape output) (at 257.81 44.45 0)
     (effects (font (size 1.27 1.27)) (justify left))
+  )
+  (hierarchical_label "HC[8..0]" (shape input) (at 48.26 69.85 180)
+    (effects (font (size 1.27 1.27)) (justify right))
   )
   (hierarchical_label "GDB[7..0]" (shape input) (at 49.53 114.3 180)
@@
     (pin "9")
   )
-  (symbol (lib_name "VSS_1") (lib_id "power:VSS") (at 203.2 100.33 0) (mirror x) (unit 1)
-    (in_bom yes) (on_board yes)
-    (property "Reference" "#PWR?" (id 0) (at 203.2 96.52 0)
-      (effects (font (size 1.27 1.27)) hide)
-    )
-    (property "Value" "VSS" (id 1) (at 203.2 104.14 0))
-    (property "Footprint" "" (id 2) (at 203.2 100.33 0)
-      (effects (font (size 1.27 1.27)) hide)
-    )
-    (property "Datasheet" "" (id 3) (at 203.2 100.33 0)
-      (effects (font (size 1.27 1.27)) hide)
-    )
-    (pin "1")
-  )
-  (symbol (lib_id "Device:R_Network07_US") (at 245.11 90.17 270) (unit 1)
-    (in_bom yes) (on_board yes)
-    (property "Reference" "H17" (id 0) (at 250.19 88.9 90))
-    (property "Value" "R0-012" (id 1) (at 252.73 91.44 90))
-    (property "Footprint" "Resistor_THT:R_Array_SIP8" (id 2) (at 245.11 102.235 90)
-      (effects (font (size 1.27 1.27)) hide)
-    )
-    (property "Datasheet" "http://www.vishay.com/docs/31509/csc.pdf" (id 3) (at 245.11 90.17 0)
-      (effects (font (size 1.27 1.27)) hide)
-    )
-    (pin "1")
-    (pin "2")
-    (pin "3")
-    (pin "4")
-    (pin "5")
-    (pin "6")
-    (pin "7")
-    (pin "8")
-  )
-  (symbol (lib_id "Device:R_Network07_US") (at 245.11 52.07 270) (unit 1)
-    (in_bom yes) (on_board yes)
-    (property "Reference" "H15" (id 0) (at 251.46 49.53 90))
-    (property "Value" "R0-012" (id 1) (at 252.73 52.07 90))
-    (property "Footprint" "Resistor_THT:R_Array_SIP8" (id 2) (at 245.11 64.135 90)
-      (effects (font (size 1.27 1.27)) hide)
-    )
-    (property "Datasheet" "http://www.vishay.com/docs/31509/csc.pdf" (id 3) (at 245.11 52.07 0)
-      (effects (font (size 1.27 1.27)) hide)
-    )
-    (pin "1")
-    (pin "2")
-    (pin "3")
-    (pin "4")
-    (pin "5")
-    (pin "6")
-    (pin "7")
-    (pin "8")
-  )
-  (symbol (lib_id "yamaha:SETAX1-003") (at 203.2 67.31 0) (unit 1)
-    (in_bom yes) (on_board yes)
-    (property "Reference" "UHH16" (id 0) (at 209.55 40.64 0))
-    (property "Value" "SETAX1-003" (id 1) (at 203.2 67.31 90))
-    (property "Footprint" "" (id 2) (at 204.47 67.31 0)
-      (effects (font (size 1.27 1.27)) hide)
-    )
-    (property "Datasheet" "" (id 3) (at 204.47 67.31 0)
-      (effects (font (size 1.27 1.27)) hide)
-    )
-    (pin "1")
-    (pin "10")
-    (pin "11")
-    (pin "12")
-    (pin "13")
-    (pin "14")
-    (pin "15")
-    (pin "16")
-    (pin "17")
-    (pin "18")
-    (pin "19")
-    (pin "2")
-    (pin "20")
-    (pin "21")
-    (pin "22")
-    (pin "23")
-    (pin "24")
-    (pin "25")
-    (pin "26")
-    (pin "27")
-    (pin "28")
-    (pin "29")
-    (pin "3")
-    (pin "30")
-    (pin "31")
-    (pin "32")
-    (pin "33")
-    (pin "34")
-    (pin "35")
-    (pin "36")
-    (pin "37")
-    (pin "38")
-    (pin "39")
-    (pin "4")
-    (pin "40")
-    (pin "41")
-    (pin "42")
-    (pin "5")
-    (pin "6")
-    (pin "7")
-    (pin "8")
-    (pin "9")
-  )
-  (symbol (lib_name "YM3909_1") (lib_id "yamaha:YM3909") (at 82.55 107.95 0) (unit 1)
+  (symbol (lib_id "yamaha:YM3909") (at 82.55 107.95 0) (unit 1)
     (in_bom yes) (on_board yes)
     (property "Reference" "B15" (id 0) (at 74.93 38.1 0)
@@
     (pin "9")
   )
+  (symbol (lib_id "Device:R_Network07_US") (at 245.11 90.17 270) (unit 1)
+    (in_bom yes) (on_board yes)
+    (property "Reference" "H17" (id 0) (at 250.19 88.9 90))
+    (property "Value" "R0-012" (id 1) (at 252.73 91.44 90))
+    (property "Footprint" "Resistor_THT:R_Array_SIP8" (id 2) (at 245.11 102.235 90)
+      (effects (font (size 1.27 1.27)) hide)
+    )
+    (property "Datasheet" "http://www.vishay.com/docs/31509/csc.pdf" (id 3) (at 245.11 90.17 0)
+      (effects (font (size 1.27 1.27)) hide)
+    )
+    (pin "1")
+    (pin "2")
+    (pin "3")
+    (pin "4")
+    (pin "5")
+    (pin "6")
+    (pin "7")
+    (pin "8")
+  )
+  (symbol (lib_id "Device:R_Network07_US") (at 245.11 52.07 270) (unit 1)
+    (in_bom yes) (on_board yes)
+    (property "Reference" "H15" (id 0) (at 251.46 49.53 90))
+    (property "Value" "R0-012" (id 1) (at 252.73 52.07 90))
+    (property "Footprint" "Resistor_THT:R_Array_SIP8" (id 2) (at 245.11 64.135 90)
+      (effects (font (size 1.27 1.27)) hide)
+    )
+    (property "Datasheet" "http://www.vishay.com/docs/31509/csc.pdf" (id 3) (at 245.11 52.07 0)
+      (effects (font (size 1.27 1.27)) hide)
+    )
+    (pin "1")
+    (pin "2")
+    (pin "3")
+    (pin "4")
+    (pin "5")
+    (pin "6")
+    (pin "7")
+    (pin "8")
+  )
+  (symbol (lib_id "yamaha:SETAX1-003") (at 203.2 67.31 0) (unit 1)
+    (in_bom yes) (on_board yes)
+    (property "Reference" "UHH16" (id 0) (at 209.55 40.64 0))
+    (property "Value" "SETAX1-003" (id 1) (at 203.2 67.31 90))
+    (property "Footprint" "" (id 2) (at 204.47 67.31 0)
+      (effects (font (size 1.27 1.27)) hide)
+    )
+    (property "Datasheet" "" (id 3) (at 204.47 67.31 0)
+      (effects (font (size 1.27 1.27)) hide)
+    )
+    (pin "1")
+    (pin "10")
+    (pin "11")
+    (pin "12")
+    (pin "13")
+    (pin "14")
+    (pin "15")
+    (pin "16")
+    (pin "17")
+    (pin "18")
+    (pin "19")
+    (pin "2")
+    (pin "20")
+    (pin "21")
+    (pin "22")
+    (pin "23")
+    (pin "24")
+    (pin "25")
+    (pin "26")
+    (pin "27")
+    (pin "28")
+    (pin "29")
+    (pin "3")
+    (pin "30")
+    (pin "31")
+    (pin "32")
+    (pin "33")
+    (pin "34")
+    (pin "35")
+    (pin "36")
+    (pin "37")
+    (pin "38")
+    (pin "39")
+    (pin "4")
+    (pin "40")
+    (pin "41")
+    (pin "42")
+    (pin "5")
+    (pin "6")
+    (pin "7")
+    (pin "8")
+    (pin "9")
+  )
   (symbol (lib_id "Device:R_Pack08") (at 160.02 54.61 90) (mirror x) (unit 1)
     (in_bom yes) (on_board yes)
@@
     (pin "8")
     (pin "9")
+  )
+  (symbol (lib_id "power:VSS") (at 203.2 100.33 180) (unit 1)
+    (in_bom yes) (on_board yes)
+    (property "Reference" "#PWR0104" (id 0) (at 203.2 96.52 0)
+      (effects (font (size 1.27 1.27)) hide)
+    )
+    (property "Value" "VSS" (id 1) (at 203.2 104.14 0))
+    (property "Footprint" "" (id 2) (at 203.2 100.33 0)
+      (effects (font (size 1.27 1.27)) hide)
+    )
+    (property "Datasheet" "" (id 3) (at 203.2 100.33 0)
+      (effects (font (size 1.27 1.27)) hide)
+    )
+    (pin "1")
   )
   (symbol (lib_id "arcade:MB7124E") (at 128.27 55.88 0) (unit 1)
@@
     (pin "9")
   )
-  (symbol (lib_name "VCC_1") (lib_id "power:VCC") (at 203.2 36.83 0) (mirror y) (unit 1)
+  (symbol (lib_id "power:VCC") (at 203.2 36.83 0) (unit 1)
     (in_bom yes) (on_board yes)
-    (property "Reference" "#PWR?" (id 0) (at 203.2 40.64 0)
-      (effects (font (size 1.27 1.27)) hide)
-    )
+    (property "Reference" "#PWR0105" (id 0) (at 203.2 40.64 0)
+      (effects (font (size 1.27 1.27)) hide)
+    )

Commit message: terminated exterminator
Parts:
- removed UHH16: SETAX1-003, symbol yamaha:SETAX1-003
- added HH16: SETAX1-003, symbol yamaha:SETAX1-003
Connections:
- net SYNC: now also HH16.22 (HBLK), HH16.23 (SYNC)
- net VCC: now also HH16.18 (UK), HH16.42 (VCC)
- net VSS: now also HH16.21 (VSS)
- net ~{HBLK}: now also HH16.19 (~{HBLK})
- net ~{VSYNC}: now also HH16.20 (~{VSYNC})
- net at H16.2 (R1): now also HH16.30 (GDC)
- net at H16.3 (R2): now also HH16.31 (G0)
- net at H16.4 (R3): now also HH16.32 (G1)
- net at H16.5 (R4): now also HH16.33 (G2)
- net at H16.6 (R5): now also HH16.34 (G3)
- net at H16.7 (R6): now also HH16.35 (G4)
- net at H17.2 (R1): now also HH16.29 (BDC)
- net at H17.3 (R2): now also HH16.28 (B0)
- net at H17.4 (R3): now also HH16.27 (B1)
- net at H17.5 (R4): now also HH16.26 (B2)
- net at H17.6 (R5): now also HH16.25 (B3)
- net at H17.7 (R6): now also HH16.24 (B4)
- net at H15.2 (R1): now also HH16.36 (RDC)
- net at H15.3 (R2): now also HH16.37 (R0)
- net at H15.4 (R3): now also HH16.38 (R1)
- net at H15.5 (R4): now also HH16.39 (R2)
- net at H15.6 (R5): now also HH16.40 (R3)
- net at H15.7 (R6): now also HH16.41 (R4)
- net at G17.1 (R1.1): now also HH16.10 (D0)
- net at G17.2 (R2.1): now also HH16.11 (D1)
- net at G17.3 (R3.1): now also HH16.12 (D2)
- net at G17.4 (R4.1): now also HH16.13 (D3)
- net at G17.5 (R5.1): now also HH16.14 (D4)
- net at G17.6 (R6.1): now also HH16.15 (D5)
- net at G17.7 (R7.1): now also HH16.16 (D6)
- net at G17.8 (R8.1): now also HH16.17 (D7)
- net at G15.8 (R8.1): now also HH16.2 (D15)
- net at G15.7 (R7.1): now also HH16.3 (D14)
- net at G15.6 (R6.1): now also HH16.4 (D13)
- net at G15.5 (R5.1): now also HH16.5 (D12)
- net at G15.4 (R4.1): now also HH16.6 (D11)
- net at G15.3 (R3.1): now also HH16.7 (D10)
- net at G15.2 (R2.1): now also HH16.8 (D9)
- net at G15.1 (R1.1): now also HH16.9 (D8)
Other:
- note removed: "COLMIX"
- note removed: "PIN16 G15"

Commit message: issues_exterm
Other:
- note removed: "?"
Changed lines of the file:
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@@
     (effects (font (size 1.27 1.27)) (justify left bottom))
-  )
-  (text "?" (at 160.02 40.64 180)
-    (effects (font (size 3 3)) (justify right bottom))
   )
   (text "0,7kΩ" (at 232.41 54.61 0)
