File: cores/exterm/sch/colmix.kicad_sch (KiCad schematic)
At the start: 9 parts

Commit message: issues_solved_#21
Other:
- note removed: "?"
- moved on the sheet: B15

Commit message: Extermination schematics updated (issue #33)
Parts:
- renumbered F13 to F15
Connections:
- net DBB2 renamed VD2
- net DBB3 renamed VD3
- net DBB4 renamed VD4
- net DBB5 renamed VD5
- net DBB6 renamed VD6
- net DBB7 renamed VD7
- net XTAL1 renamed H1B
Changed lines of the file:
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@@
     )
   )
-  (text "MSB" (at 254 57.15 180)
+  (text "MSB" (at 254 60.96 180)
     (effects (font (size 1.27 1.27)) (justify right bottom))
   )
@@
     (effects (font (size 1.27 1.27)) (justify left bottom))
   )
-  (label "DBB5" (at 63.5 57.15 180)
+  (label "VD5" (at 63.5 57.15 180)
     (effects (font (size 1.27 1.27)) (justify right bottom))
   )
@@
     (effects (font (size 1.27 1.27)) (justify left bottom))
   )
-  (label "DBB6" (at 63.5 54.61 180)
+  (label "VD6" (at 63.5 54.61 180)
     (effects (font (size 1.27 1.27)) (justify right bottom))
   )
@@
     (effects (font (size 1.27 1.27)) (justify left bottom))
   )
-  (label "DBB4" (at 63.5 59.69 180)
+  (label "VD4" (at 63.5 59.69 180)
     (effects (font (size 1.27 1.27)) (justify right bottom))
   )
@@
     (effects (font (size 1.27 1.27)) (justify left bottom))
   )
-  (label "DBB7" (at 63.5 52.07 180)
+  (label "VD7" (at 63.5 52.07 180)
     (effects (font (size 1.27 1.27)) (justify right bottom))
   )
@@
     (effects (font (size 1.27 1.27)) (justify right bottom))
   )
-  (label "DBB3" (at 63.5 62.23 180)
+  (label "VD3" (at 63.5 62.23 180)
     (effects (font (size 1.27 1.27)) (justify right bottom))
   )
@@
     (effects (font (size 1.27 1.27)) (justify left bottom))
   )
-  (label "DBB2" (at 63.5 64.77 180)
+  (label "VD2" (at 63.5 64.77 180)
     (effects (font (size 1.27 1.27)) (justify right bottom))
   )
@@
     (effects (font (size 1.27 1.27)) (justify left))
   )
-  (hierarchical_label "DBB[7..0]" (shape input) (at 48.26 49.53 180)
+  (hierarchical_label "VD[7..0]" (shape input) (at 48.26 49.53 180)
     (effects (font (size 1.27 1.27)) (justify right))
   )
@@
     (effects (font (size 1.27 1.27)) (justify right))
   )
-  (hierarchical_label "XTAL1" (shape input) (at 149.86 107.95 180)
+  (hierarchical_label "H1B" (shape input) (at 149.86 107.95 180)
     (effects (font (size 1.27 1.27)) (justify right))
   )
@@
     (pin "8")
   )
-  (symbol (lib_id "arcade:MB7124E") (at 128.27 101.6 0) (unit 1)
+  (symbol (lib_name "MB7124E_1") (lib_id "arcade:MB7124E") (at 128.27 101.6 0) (unit 1)
     (in_bom yes) (on_board yes)
-    (property "Reference" "F13" (id 0) (at 128.27 97.79 0))
+    (property "Reference" "F15" (id 0) (at 128.27 97.79 0))
     (property "Value" "MB7124E" (id 1) (at 128.27 101.6 0))
     (property "Footprint" "" (id 2) (at 128.27 97.79 0)
@@
   (symbol (lib_id "Device:R_Network07_US") (at 245.11 52.07 270) (unit 1)
     (in_bom yes) (on_board yes)
-    (property "Reference" "H15" (id 0) (at 251.46 49.53 90))
-    (property "Value" "R0-012" (id 1) (at 252.73 52.07 90))
+    (property "Reference" "H15" (id 0) (at 252.73 52.07 90))
+    (property "Value" "R0-012" (id 1) (at 254 54.61 90))
     (property "Footprint" "Resistor_THT:R_Array_SIP8" (id 2) (at 245.11 64.135 90)
       (effects (font (size 1.27 1.27)) hide)
