File: cores/exterm/sch/gfx.kicad_sch (KiCad schematic)
At the start: 23 parts

Commit message: almost ready
Parts:
- removed B17: YM3906, symbol yamaha:YM3906
- added C17: YM3906, symbol yamaha:YM3906
- R3: renamed from 22Ω; value R3 -> 22Ω
- R4: renamed from 3.3kΩ; value R4 -> 3.3kΩ
Connections:
- net DATAEN: now also C17.61 (DATAEN)
- net DB0: now also C17.14 (D0)
- net DB1: now also C17.13 (D1)
- net DB2: now also C17.12 (D2)
- net DB3: now also C17.11 (D3)
- net DB4: now also C17.10 (D4)
- net DB5: now also C17.9 (D5)
- net DB6: now also C17.8 (D6)
- net DB7: now also C17.7 (D7)
- net DBB0: now also C17.4 (XC0)
- net DBB6: now also C17.59 (FLIPY)
- net DBB7: now also C17.60 (FLIPX)
- net GA0: now also C17.35 (CHA0)
- net GA1: now also C17.36 (CHA1)
- net GA2: now also C17.37 (CHA2)
- net GA4: now also C17.38 (CHA4)
- net GFX_A0: now also C17.15 (A0)
- net GFX_A1: now also C17.16 (A1)
- net GFX_A10: now also C17.25 (A10)
- net GFX_A11: now also C17.28 (A11)
- net GFX_A2: now also C17.17 (A2)
- net GFX_A3: now also C17.18 (A3)
- net GFX_A4: now also C17.19 (A4)
- net GFX_A5: now also C17.20 (A5)
- net GFX_A6: now also C17.21 (A6)
- net GFX_A7: now also C17.22 (A7)
- net GFX_A8: now also C17.23 (A8)
- net GFX_A9: now also C17.24 (A9)
- net GFX_CLK: now also C17.62 (CLKO)
- net H0: now also C17.40 (HPH90)
- net H1: now also C17.39 (H)
- net H2: now also C17.41 (H2)
- net H3: now also C17.42 (H4)
- net H4: now also C17.43 (H8)
- net HC0: now also C17.46 (HC0)
- net HC1: now also C17.47 (HC1)
- net HC2: now also C17.48 (HC2)
- net HC3: now also C17.49 (HC3)
- net HC4: now also C17.50 (HC4)
- net HC5: now also C17.51 (HC5)
- net HC6: now also C17.52 (HC6)
- net HC7: now also C17.53 (HC7)
- net HC8: now also C17.54 (HC8)
- net HR8: now also C17.34 (H8B)
- net MAIN_A11: now also C17.27 (SPBANK2)
- net MAIN_~{RD}: now also C17.2 (~{RD})
- net RW: now also C17.30 (RW)
- net VBLK: now also C17.58 (~{VBLK})
- net VCC: now also R4.1; no longer R4.2
- net VSS: now also C17.31 (UK), C17.45 (UK)
- net ~{GFX_WR}: now also C17.3 (~{WR})
- net ~{HBLK}: now also C17.55 (~{HBLK})
- net ~{VSYNC}: now also C17.56 (~{VSYNC})
- net ~{WDRES}: now also C17.29 (~{WDRES)
- net AQUI: no longer names the net of R3.2
- net AQUI: now also A17.3 (Out), R4.2, C17.63 (CLK)
- net MAIN_WR renamed ~{WR}
- new net: C17.1 (VCC), C17.33 (VCC)
- new net: C17.32 (VSS), C17.64 (VSS)
- new net SPBANK1: C17.26 (SPBANK1)
- now unconnected: R3.1
- no-connect marks 6 -> 7
Other:
- note added: "DRIVER"
- note added: "ENABLE"
- moved on the sheet: R4

Commit message: issues_exterm
Other:
- note removed: "?"
- note removed: "DRIVER"
- note removed: "GXF"
- note removed: "TRIESTADO?"
Changed lines of the file:
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@@
     )
   )
-  (text "?" (at 321.31 376.555 0)
-    (effects (font (size 5 5)) (justify left bottom))
-  )
-  (text "TRIESTADO?" (at 257.81 290.83 90)
-    (effects (font (size 1.27 1.27)) (justify left bottom))
-  )
-  (text "DRIVER" (at 217.17 299.72 0)
-    (effects (font (size 1.27 1.27)) (justify left bottom))
-  )
-  (text "GXF\n" (at 351.79 74.93 0)
-    (effects (font (size 5 5)) (justify left bottom))
-  )
   (text "ENABLE" (at 207.01 234.95 0)
     (effects (font (size 1.27 1.27)) (justify left bottom))
@@
     (effects (font (size 1.27 1.27)) (justify right bottom))
   )
-  (label "MAIN_D[7..0]" (at 115.57 121.92 0)
-    (effects (font (size 1.27 1.27)) (justify left bottom))
-  )
   (label "GA12" (at 322.58 351.79 0)
