File: cores/exterm/sch/gfx.kicad_sch (KiCad schematic)
At the start: 23 parts

Commit message: issues_exterm
Connections:
- net GFX_CE renamed ~{GFX_CE'}
Other:
- note removed: "?"
Changed lines of the file:
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@@
     (stroke (width 0) (type default) (color 0 0 0 0))
   )
+  (wire (pts (xy 369.57 364.49) (xy 369.57 388.62))
+    (stroke (width 0) (type default) (color 0 0 0 0))
+  )
   (bus (pts (xy 320.04 190.5) (xy 320.04 193.04))
     (stroke (width 0) (type default) (color 0 0 0 0))
@@
     (stroke (width 0) (type default) (color 0 0 0 0))
   )
-  (bus (pts (xy 181.61 260.35) (xy 184.785 260.35))
+  (bus (pts (xy 181.61 260.35) (xy 191.77 260.35))
     (stroke (width 0) (type default) (color 0 0 0 0))
   )
@@
     (stroke (width 0) (type default) (color 0 0 0 0))
   )
+  (wire (pts (xy 369.57 364.49) (xy 379.73 364.49))
+    (stroke (width 0) (type default) (color 0 0 0 0))
+  )
   (wire (pts (xy 400.05 187.96) (xy 410.21 187.96))
     (stroke (width 0) (type default) (color 0 0 0 0))
@@
     (stroke (width 0) (type default) (color 0 0 0 0))
   )
-  (wire (pts (xy 370.84 364.49) (xy 379.73 364.49))
-    (stroke (width 0) (type default) (color 0 0 0 0))
-  )
   (bus (pts (xy 289.56 273.05) (xy 292.1 273.05))
     (stroke (width 0) (type default) (color 0 0 0 0))
@@
     (stroke (width 0) (type default) (color 0 0 0 0))
   )
-  (wire (pts (xy 345.44 388.62) (xy 353.695 388.62))
+  (wire (pts (xy 345.44 388.62) (xy 369.57 388.62))
     (stroke (width 0) (type default) (color 0 0 0 0))
   )
@@
     )
   )
-  (text "?" (at 321.31 376.555 0)
-    (effects (font (size 5 5)) (justify left bottom))
-  )
   (text "TRIESTADO?" (at 257.81 290.83 90)
     (effects (font (size 1.27 1.27)) (justify left bottom))
@@
     (effects (font (size 1.27 1.27)) (justify left bottom))
   )
-  (label "GFX_CE" (at 370.84 295.91 0)
-    (effects (font (size 1.27 1.27)) (justify left bottom))
-  )
   (label "DBB5" (at 175.26 166.37 180)
     (effects (font (size 1.27 1.27)) (justify right bottom))
@@
     (effects (font (size 1.27 1.27)) (justify left bottom))
   )
+  (label "~{GFX_CE'}" (at 370.84 295.91 0)
+    (effects (font (size 1.27 1.27)) (justify left bottom))
+  )
   (label "DBB7" (at 175.26 214.63 180)
     (effects (font (size 1.27 1.27)) (justify right bottom))
@@
     (effects (font (size 1.27 1.27)) (justify right bottom))
   )
-  (label "GFX_CE" (at 353.695 388.62 180)
-    (effects (font (size 1.27 1.27)) (justify right bottom))
-  )
   (label "~{GFX_CE}" (at 322.58 364.49 0)
     (effects (font (size 1.27 1.27)) (justify left bottom))
@@
     (effects (font (size 1.27 1.27)) (justify left bottom))
   )
-  (label "GFX_CE" (at 370.84 364.49 0)
+  (label "~{GFX_CE'}" (at 370.84 364.49 0)
     (effects (font (size 1.27 1.27)) (justify left bottom))
   )
@@
     (effects (font (size 1.27 1.27)) (justify right bottom))
   )
-  (label "GFX_CE" (at 370.84 218.44 0)
+  (label "~{GFX_CE'}" (at 370.84 218.44 0)
     (effects (font (size 1.27 1.27)) (justify left bottom))
   )
@@
     (effects (font (size 1.27 1.27)) (justify left bottom))
   )
-  (label "GFX_CE" (at 370.84 149.86 0)
+  (label "~{GFX_CE'}" (at 370.84 149.86 0)
     (effects (font (size 1.27 1.27)) (justify left bottom))
   )
@@
     (effects (font (size 1.27 1.27)) (justify left))
   )
-  (hierarchical_label "DBB[7..0]" (shape output) (at 184.785 260.35 0)
+  (hierarchical_label "DBB[7..0]" (shape output) (at 191.77 260.35 0)
     (effects (font (size 1.27 1.27)) (justify left))
   )

Commit message: issues_solved_#21
Connections:
- net VCC: now also C17.1 (VCC), C17.33 (VCC)
- net VSS: now also C17.32 (VSS), C17.5 (UK), C17.6 (UK), C17.64 (VSS); no longer C17.31 (UK), C17.45 (UK)
Other:
- note removed: "DRIVER"
- note removed: "GXF"
- note removed: "TRIESTADO?"
- moved on the sheet: A10, A12, A13, A15, A16, A17, A2, A4, A5, A7, A8, B1D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
