File: cores/exterm/sch/gfx.kicad_sch (KiCad schematic)
At the start: 23 parts

Commit message: Extermination schematics updated (issue #33)
Parts:
- removed A10, A12, A13, A2, A4, A5, A7, A8: 27C512, Package_DIP:DIP-28_W15.24mm, symbol Memory_EPROM:27C512
- removed unit 5 of B1
- removed E13, E14, E16, E17: HM6116P-3, symbol arcade:HM6116P-3
Connections:
- net GFX_CLK: no longer A15.9 (Cp), A16.11 (Cp)
- net DB0 renamed VD8
- net DB1 renamed VD9
- net DB2 renamed VD10
- net DB3 renamed VD11
- net DB4 renamed VD12
- net DB5 renamed VD13
- net DB6 renamed VD14
- net DB7 renamed VD15
- net DBB0 renamed VD0
- net DBB1 renamed VD1
- net DBB2 renamed VD2
- net DBB3 renamed VD3
- net DBB4 renamed VD4
- net DBB5 renamed VD5
- net DBB6 renamed VD6
- net DBB7 renamed VD7
- net GFX_A0 renamed VA0
- net GFX_A1 renamed VA1
- net GFX_A10 renamed VA10
- net GFX_A11 renamed VA11
- net GFX_A2 renamed VA2
- net GFX_A3 renamed VA3
- net GFX_A4 renamed VA4
- net GFX_A5 renamed VA5
- net GFX_A6 renamed VA6
- net GFX_A7 renamed VA7
- net GFX_A8 renamed VA8
- net GFX_A9 renamed VA9
- net ~{GFX_CE} renamed ~{ROM_CE}
- net ~{GFX_OE} renamed ~{ROM_OE}
- new net H4B: A15.9 (Cp), A16.11 (Cp)
Other:
- added sheet gfx_ram (gfx_ram.kicad_sch)
- added sheet gfx_rom (gfx_rom.kicad_sch)
- note removed: "NOT MOUNTED"
- moved on the sheet: A15, A16, A17, B1D, B1F, B6A, C17, C6B, E11, E12, R3, R4
