File: cores/exterm/sch/capacitors.kicad_sch (KiCad schematic)
At the start: 1 part

Commit message: distribution
Parts:
- added C22, C23, C24, C25, C26, C27, C28, C29, C30, C31, C32, C33, C34, C35, C36, C37: 104, symbol Device:C
Connections:
- net VCC: now reaches C1.1
- net VCC: now also C22.1, C23.1, C24.1, C25.1, C26.1, C27.1, C28.1, C29.1, C30.1, C31.1, C32.1, C33.1, C34.1, C35.1, C36.1, C37.1
- net VSS: now reaches C1.2
- net VSS: now also C22.2, C23.2, C24.2, C25.2, C26.2, C27.2, C28.2, C29.2, C30.2, C31.2, C32.2, C33.2, C34.2, C35.2, C36.2, C37.2

Commit message: almost ready
Parts:
- removed C1: 1000μF, symbol Device:CP1
- added B1, G13: 74LS04, symbol jt74:74LS04
- added B2, B6: 74LS08, symbol jt74:74LS08
- added B3, B4, B7: 74LS74, symbol jt74:74LS74
- added C1: 1000μF, symbol Device:C_Polarized_Small_US
- added C6: 74LS32, symbol jt74:74LS32
- added H12: NJM4558, symbol Amplifier_Operational:NJM4558
- added H5: 74LS02, symbol jt74:74LS02
Connections:
- net VCC: now also B1.14 (VCC), B2.14 (VCC), B3.14 (VCC), B4.14 (VCC), B6.14 (VCC), B7.14 (VCC), C1.1, C6.14 (VCC), G13.14 (VCC), H12.8 (V+), H5.14 (VCC)
- net VSS: now also B1.7 (VSS), B2.7 (VSS), B3.7 (VSS), B4.7 (VSS), B6.7 (VSS), B7.7 (VSS), C1.2, C6.7 (VSS), G13.7 (VSS), H12.4 (V-), H5.7 (VSS)

Commit message: terminated exterminator
Other:
- moved on the sheet: B1G, B2E, B3C, B4C, B6E, B7C, C1, C22, C23, C24, C25, C26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

Commit message: issues_exterm
Other:
- moved on the sheet: B1G, B2E, B3C, B4C, B6E, B7C, C1, C22, C23, C24, C25, C26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
