File: cores/exterm/sch/watchdog.kicad_sch (KiCad schematic)
At the start: 17 parts, among them J8 TL7705A, SW1 SW_Push

Commit message: terminated exterminator
Parts:
- added ZD2: BZD27C, Diode_SMD:D_SMF, symbol Diode:BZD27Cxx
Connections:
- net +12V: now also ZD2.2 (A)
- net VSS: now also ZD2.1 (K)

Commit message: issues_exterm
Other:
- moved on the sheet: CC2, CC6, CC7, CC8, G13A, G13B, G13D, G13F, G14, H5A, J8, JJ1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
