File: cores/exterm/sch/mcu.kicad_sch (KiCad schematic)
At the start: 3 parts

Commit message: terminated exterminator
Other:
- note removed: "BIDIRECCIONAL?"
- moved on the sheet: G3, H5B, H5C, H5D

Commit message: issues_exterm
Changed lines of the file:
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@@
     (stroke (width 0) (type default) (color 0 0 0 0))
   )
-  (wire (pts (xy 222.25 60.96) (xy 229.87 60.96))
+  (wire (pts (xy 222.25 60.96) (xy 234.95 60.96))
     (stroke (width 0) (type default) (color 0 0 0 0))
   )
@@
     (stroke (width 0) (type default) (color 0 0 0 0))
   )
-  (wire (pts (xy 222.25 63.5) (xy 229.87 63.5))
+  (wire (pts (xy 222.25 63.5) (xy 234.95 63.5))
     (stroke (width 0) (type default) (color 0 0 0 0))
   )
@@
     (effects (font (size 1.27 1.27)) (justify left bottom))
   )
-  (label "TEST0" (at 229.87 63.5 180)
+  (label "TEST0" (at 234.95 63.5 180)
     (effects (font (size 1.27 1.27)) (justify right bottom))
   )
@@
     (effects (font (size 1.27 1.27)) (justify left bottom))
   )
-  (label "TEST1" (at 229.87 60.96 180)
-    (effects (font (size 1.27 1.27)) (justify right bottom))
-  )
+  (label "TEST1" (at 234.95 60.96 180)
+    (effects (font (size 1.27 1.27)) (justify right bottom))
+  )

Commit message: issues_solved_#21
Other:
- moved on the sheet: G3, H5B, H5C, H5D, JJ10

Commit message: Extermination schematics updated (issue #33)
Parts:
- added G13: 74LS04, symbol jt74:74LS04
- added R20: R330Ω, symbol Device:R_US
Connections:
- net VCC: now also R20.2
- net XTAL1 renamed H1B
- net H1B: now also G13.11, R20.1
- net ~{XTAL2} renamed ~{H1B}
- net ~{H1B}: now also G13.10
Changed lines of the file:
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@@
     (comment 1 "E.Triana")
+  )
+  (junction (at 33.02 125.73) (diameter 0) (color 0 0 0 0)
   )
   (junction (at 81.28 83.82) (diameter 0) (color 0 0 0 0)
@@
     (stroke (width 0) (type default) (color 0 0 0 0))
   )
+  (wire (pts (xy 33.02 120.65) (xy 33.02 125.73))
+    (stroke (width 0) (type default) (color 0 0 0 0))
+  )
   (wire (pts (xy 67.31 55.88) (xy 71.12 55.88))
     (stroke (width 0) (type default) (color 0 0 0 0))
@@
     (stroke (width 0) (type default) (color 0 0 0 0))
   )
+  (wire (pts (xy 33.02 125.73) (xy 48.26 125.73))
+    (stroke (width 0) (type default) (color 0 0 0 0))
+  )
   (wire (pts (xy 107.95 97.79) (xy 121.92 97.79))
     (stroke (width 0) (type default) (color 0 0 0 0))
@@
     (stroke (width 0) (type default) (color 0 0 0 0))
   )
+  (wire (pts (xy 63.5 125.73) (xy 71.12 125.73))
+    (stroke (width 0) (type default) (color 0 0 0 0))
+  )
   (wire (pts (xy 67.31 30.48) (xy 78.74 30.48))
     (stroke (width 0) (type default) (color 0 0 0 0))
@@
     (stroke (width 0) (type default) (color 0 0 0 0))
   )
+  (wire (pts (xy 33.02 107.95) (xy 33.02 113.03))
+    (stroke (width 0) (type default) (color 0 0 0 0))
+  )
   (wire (pts (xy 81.28 83.82) (xy 81.28 95.25))
     (stroke (width 0) (type default) (color 0 0 0 0))
@@
     (stroke (width 0) (type default) (color 0 0 0 0))
   )
-  (wire (pts (xy 34.29 73.66) (xy 43.18 73.66))
-    (stroke (width 0) (type default) (color 0 0 0 0))
-  )
   (wire (pts (xy 88.9 53.34) (xy 92.71 53.34))
     (stroke (width 0) (type default) (color 0 0 0 0))
@@
     (stroke (width 0) (type default) (color 0 0 0 0))
   )
+  (wire (pts (xy 24.13 125.73) (xy 33.02 125.73))
+    (stroke (width 0) (type default) (color 0 0 0 0))
+  )
   (wire (pts (xy 177.8 60.96) (xy 177.8 63.5))
     (stroke (width 0) (type default) (color 0 0 0 0))
@@
   )
   (wire (pts (xy 151.13 57.15) (xy 151.13 58.42))
+    (stroke (width 0) (type default) (color 0 0 0 0))
+  )
+  (wire (pts (xy 29.21 73.66) (xy 43.18 73.66))
     (stroke (width 0) (type default) (color 0 0 0 0))
   )
@@
     (effects (font (size 1.27 1.27)) (justify right bottom))
   )
+  (label "VCC" (at 33.02 107.95 0)
+    (effects (font (size 1.27 1.27)) (justify left bottom))
+  )
   (label "P20" (at 34.29 50.8 0)
     (effects (font (size 1.27 1.27)) (justify left bottom))
@@
     (effects (font (size 1.27 1.27)) (justify right bottom))
   )
+  (label "H1B" (at 24.13 125.73 0)
+    (effects (font (size 1.27 1.27)) (justify left bottom))
+  )
   (label "P22" (at 34.29 55.88 0)
     (effects (font (size 1.27 1.27)) (justify left bottom))
@@
     (effects (font (size 1.27 1.27)) (justify left bottom))
   )
+  (label "~{H1B}" (at 29.21 73.66 0)
+    (effects (font (size 1.27 1.27)) (justify left bottom))
+  )
   (label "SND_D0" (at 76.2 27.94 180)
     (effects (font (size 1.27 1.27)) (justify right bottom))
@@
   (label "P14" (at 34.29 40.64 0)
     (effects (font (size 1.27 1.27)) (justify left bottom))
+  )
+  (label "~{H1B}" (at 71.12 125.73 180)
+    (effects (font (size 1.27 1.27)) (justify right bottom))
   )
   (label "VCC" (at 185.42 60.96 180)
@@
     (effects (font (size 1.27 1.27)) (justify left))
   )
-  (hierarchical_label "SND_~{WR}" (shape output) (at 71.12 58.42 0)
+  (hierarchical_label "SND_~{WR}" (shape input) (at 71.12 58.42 0)
     (effects (font (size 1.27 1.27)) (justify left))
   )
@@
     (effects (font (size 1.27 1.27)) (justify right))
   )
-  (hierarchical_label "XTAL1" (shape input) (at 34.29 71.12 180)
+  (hierarchical_label "H1B" (shape input) (at 34.29 71.12 180)
     (effects (font (size 1.27 1.27)) (justify right))
   )
@@
     (effects (font (size 1.27 1.27)) (justify left))
   )
-  (hierarchical_label "SND_D[7..0]" (shape output) (at 88.9 25.4 0)
+  (hierarchical_label "SND_D[7..0]" (shape tri_state) (at 88.9 25.4 0)
     (effects (font (size 1.27 1.27)) (justify left))
   )
-  (hierarchical_label "P26_DRQ" (shape bidirectional) (at 71.12 50.8 0)
+  (hierarchical_label "P26_DRQ" (shape output) (at 71.12 50.8 0)
     (effects (font (size 1.27 1.27)) (justify left))
   )
-  (hierarchical_label "SND_~{RD}" (shape output) (at 71.12 55.88 0)
+  (hierarchical_label "SND_~{RD}" (shape input) (at 71.12 55.88 0)
     (effects (font (size 1.27 1.27)) (justify left))
   )
@@
   )
   (hierarchical_label "SND_A[15..0]" (shape input) (at 27.94 25.4 180)
-    (effects (font (size 1.27 1.27)) (justify right))
-  )
-  (hierarchical_label "~{XTAL2}" (shape input) (at 34.29 73.66 180)
     (effects (font (size 1.27 1.27)) (justify right))
   )
@@
     (pin "14")
     (pin "7")
+  )
+  (symbol (lib_id "Device:R_US") (at 33.02 116.84 0) (mirror x) (unit 1)
+    (in_bom yes) (on_board yes)
+    (property "Reference" "R20" (id 0) (at 38.1 115.57 0))
+    (property "Value" "R330Ω" (id 1) (at 39.37 118.11 0))
+    (property "Footprint" "" (id 2) (at 34.036 116.586 90)
+      (effects (font (size 1.27 1.27)) hide)
+    )
+    (property "Datasheet" "~" (id 3) (at 33.02 116.84 0)
+      (effects (font (size 1.27 1.27)) hide)
+    )
+    (pin "1")
+    (pin "2")
   )
   (symbol (lib_id "power:VCC") (at 55.88 20.32 0) (unit 1)
@@
     (pin "9")
   )
+  (symbol (lib_id "jt74:74LS04") (at 55.88 125.73 0) (unit 5)
+    (in_bom yes) (on_board yes)
+    (property "Reference" "G13" (id 0) (at 55.88 124.46 0))
+    (property "Value" "74LS04" (id 1) (at 55.88 127 0))
+    (property "Footprint" "" (id 2) (at 55.88 125.73 0)
+      (effects (font (size 1.27 1.27)) hide)
+    )
+    (property "Datasheet" "http://www.ti.com/lit/gpn/sn74LS04" (id 3) (at 55.88 125.73 0)
+      (effects (font (size 1.27 1.27)) hide)
+    )
+    (pin "1")
+    (pin "2")
+    (pin "3")
+    (pin "4")
+    (pin "5")
+    (pin "6")
+    (pin "8")
+    (pin "9")
+    (pin "10")
+    (pin "11")
+    (pin "12")
+    (pin "13")
+    (pin "14")
+    (pin "7")
+  )
 )
