File: cores/exterm/sch/sound.kicad_sch (KiCad schematic)
At the start: 38 parts, among them J16 HA1388

Commit message: terminated exterminator
Parts:
- removed F8: YM2203, Package_DIP:DIP-40_W15.24mm, symbol yamaha:YM2203
- added YM_F8: YM2203, Package_DIP:DIP-40_W15.24mm, symbol yamaha:YM2203
Connections:
- net PHM: now also YM_F8.38 (PHM)
- net SND_A0: now also YM_F8.37 (A0)
- net SND_D0: now also YM_F8.40 (D0)
- net SND_D1: now also YM_F8.2 (D1)
- net SND_D2: now also YM_F8.3 (D2)
- net SND_D3: now also YM_F8.4 (D3)
- net SND_D4: now also YM_F8.5 (D4)
- net SND_D5: now also YM_F8.6 (D5)
- net SND_D6: now also YM_F8.7 (D6)
- net SND_D7: now also YM_F8.8 (D7)
- net SND_~{NMI}: now also YM_F8.25 (~{IRQ})
- net SND_~{RD}: now also YM_F8.36 (~{RD})
- net SND_~{WR}: now also YM_F8.35 (~{WR})
- net VCC: now also YM_F8.21 (VCC)
- net VSS: now also YM_F8.1 (VSS)
- net YM_~{CS}: now also YM_F8.34 (~{CS})
- net ~{RESET}: now also YM_F8.24 (~{IC})
- net at SWA1.7: now also YM_F8.10 (IOA6)
- net at SWA1.6: now also YM_F8.11 (IOA5)
- net at SWA1.5: now also YM_F8.12 (IOA4)
- net at SWA1.4: now also YM_F8.13 (IOA3)
- net at SWA1.3: now also YM_F8.14 (IOA2)
- net at SWA1.2: now also YM_F8.15 (IOA1)
- net at SWA1.1: now also YM_F8.16 (IOA0)
- net at CC10.1, R7.2: now also YM_F8.18 (CHC), YM_F8.19 (CHB), YM_F8.20 (CHA)
- net at H11.3 (LOAD): now also YM_F8.22 (SH)
- net at H11.4 (SD): now also YM_F8.23 (OPO)
- net at SWB2.16: now also YM_F8.26 (IOB0)
- net at SWB2.15: now also YM_F8.27 (IOB1)
- net at SWB2.14: now also YM_F8.28 (IOB2)
- net at SWB2.13: now also YM_F8.29 (IOB3)
- net at SWB2.12: now also YM_F8.30 (IOB4)
- net at SWB2.11: now also YM_F8.31 (IOB5)
- net at SWB2.10: now also YM_F8.32 (IOB6)
- net at SWB2.9: now also YM_F8.33 (IOB7)
- net at H11.5 (PH1): now also YM_F8.39 (PHS)
- net at SWA1.8: now also YM_F8.9 (IOA7)

Commit message: exterm_kiwi
Connections:
- net SND_SELECT renamed ~{SND_SELECT} 
- net ~{RESET} renamed ~{SND_RST}
Changed lines of the file:
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@@
   (junction (at 337.185 97.79) (diameter 0) (color 0 0 0 0)
   )
-  (junction (at 346.964 62.23) (diameter 0) (color 0 0 0 0)
-  )
   (junction (at 337.185 130.81) (diameter 0) (color 0 0 0 0)
   )
@@
     (stroke (width 0) (type default) (color 0 0 0 0))
   )
-  (wire (pts (xy 276.225 128.27) (xy 284.48 128.27))
-    (stroke (width 0) (type default) (color 0 0 0 0))
-  )
   (bus (pts (xy 107.95 109.22) (xy 107.95 106.68))
     (stroke (width 0) (type default) (color 0 0 0 0))
@@
     (stroke (width 0) (type default) (color 0 0 0 0))
   )
-  (wire (pts (xy 275.844 80.01) (xy 282.194 80.01))
+  (wire (pts (xy 271.78 80.01) (xy 282.194 80.01))
     (stroke (width 0) (type default) (color 0 0 0 0))
   )
@@
     (stroke (width 0) (type default) (color 0 0 0 0))
   )
+  (wire (pts (xy 307.594 59.69) (xy 331.47 59.69))
+    (stroke (width 0) (type default) (color 0 0 0 0))
+  )
   (wire (pts (xy 264.16 198.12) (xy 287.02 198.12))
     (stroke (width 0) (type default) (color 0 0 0 0))
@@
     (stroke (width 0) (type default) (color 0 0 0 0))
   )
+  (wire (pts (xy 346.71 62.23) (xy 355.6 62.23))
+    (stroke (width 0) (type default) (color 0 0 0 0))
+  )
   (bus (pts (xy 165.1 233.68) (xy 165.1 236.22))
     (stroke (width 0) (type default) (color 0 0 0 0))
@@
     (stroke (width 0) (type default) (color 0 0 0 0))
   )
-  (wire (pts (xy 275.59 125.73) (xy 284.48 125.73))
-    (stroke (width 0) (type default) (color 0 0 0 0))
-  )
   (wire (pts (xy 76.2 190.5) (xy 87.63 190.5))
     (stroke (width 0) (type default) (color 0 0 0 0))
@@
     (stroke (width 0) (type default) (color 0 0 0 0))
   )
-  (wire (pts (xy 346.964 62.23) (xy 355.6 62.23))
-    (stroke (width 0) (type default) (color 0 0 0 0))
-  )
   (wire (pts (xy 337.185 118.11) (xy 337.185 120.65))
     (stroke (width 0) (type default) (color 0 0 0 0))
@@
     (stroke (width 0) (type default) (color 0 0 0 0))
   )
+  (wire (pts (xy 275.59 128.27) (xy 284.48 128.27))
+    (stroke (width 0) (type default) (color 0 0 0 0))
+  )
   (wire (pts (xy 110.49 170.18) (xy 127 170.18))
     (stroke (width 0) (type default) (color 0 0 0 0))
@@
     (stroke (width 0) (type default) (color 0 0 0 0))
   )
+  (wire (pts (xy 275.59 123.19) (xy 284.48 123.19))
+    (stroke (width 0) (type default) (color 0 0 0 0))
+  )
   (wire (pts (xy 388.62 165.1) (xy 373.38 165.1))
     (stroke (width 0) (type default) (color 0 0 0 0))
@@
     (stroke (width 0) (type default) (color 0 0 0 0))
   )
-  (wire (pts (xy 324.739 64.77) (xy 331.724 64.77))
-    (stroke (width 0) (type default) (color 0 0 0 0))
-  )
   (bus (pts (xy 165.1 123.19) (xy 165.1 125.73))
     (stroke (width 0) (type default) (color 0 0 0 0))
@@
     (stroke (width 0) (type default) (color 0 0 0 0))
   )
-  (wire (pts (xy 276.225 118.11) (xy 284.48 118.11))
+  (wire (pts (xy 275.59 118.11) (xy 284.48 118.11))
     (stroke (width 0) (type default) (color 0 0 0 0))
   )
@@
     (stroke (width 0) (type default) (color 0 0 0 0))
   )
-  (wire (pts (xy 307.594 59.69) (xy 331.724 59.69))
-    (stroke (width 0) (type default) (color 0 0 0 0))
-  )
   (wire (pts (xy 152.4 176.53) (xy 162.56 176.53))
     (stroke (width 0) (type default) (color 0 0 0 0))
@@
     (stroke (width 0) (type default) (color 0 0 0 0))
   )
-  (wire (pts (xy 346.71 62.23) (xy 346.964 62.23))
-    (stroke (width 0) (type default) (color 0 0 0 0))
-  )
   (bus (pts (xy 107.95 33.02) (xy 107.95 35.56))
     (stroke (width 0) (type default) (color 0 0 0 0))
   )
-  (wire (pts (xy 27.94 162.56) (xy 40.64 162.56))
+  (wire (pts (xy 26.67 162.56) (xy 40.64 162.56))
     (stroke (width 0) (type default) (color 0 0 0 0))
   )
@@
     (stroke (width 0) (type default) (color 0 0 0 0))
   )
-  (wire (pts (xy 33.655 182.88) (xy 40.64 182.88))
+  (wire (pts (xy 27.305 182.88) (xy 40.64 182.88))
     (stroke (width 0) (type default) (color 0 0 0 0))
   )
@@
     (stroke (width 0) (type default) (color 0 0 0 0))
   )
-  (wire (pts (xy 276.225 123.19) (xy 284.48 123.19))
-    (stroke (width 0) (type default) (color 0 0 0 0))
-  )
   (bus (pts (xy 165.1 125.73) (xy 165.1 128.27))
     (stroke (width 0) (type default) (color 0 0 0 0))
@@
     (stroke (width 0) (type default) (color 0 0 0 0))
   )
-  (wire (pts (xy 284.48 120.65) (xy 276.225 120.65))
+  (wire (pts (xy 275.59 120.65) (xy 284.48 120.65))
     (stroke (width 0) (type default) (color 0 0 0 0))
   )
@@
     (stroke (width 0) (type default) (color 0 0 0 0))
   )
+  (wire (pts (xy 275.59 125.73) (xy 284.48 125.73))
+    (stroke (width 0) (type default) (color 0 0 0 0))
+  )
   (wire (pts (xy 320.04 153.67) (xy 320.04 148.59))
     (stroke (width 0) (type default) (color 0 0 0 0))
@@
     (stroke (width 0) (type default) (color 0 0 0 0))
   )
+  (wire (pts (xy 323.215 64.77) (xy 331.47 64.77))
+    (stroke (width 0) (type default) (color 0 0 0 0))
+  )
   (wire (pts (xy 320.04 148.59) (xy 304.8 148.59))
     (stroke (width 0) (type default) (color 0 0 0 0))
@@
     (effects (font (size 1.27 1.27)) (justify left bottom))
   )
-  (label "SND_A0" (at 276.225 118.11 0)
+  (label "SND_A0" (at 275.59 118.11 0)
     (effects (font (size 1.27 1.27)) (justify left bottom))
   )
@@
     (effects (font (size 1.27 1.27)) (justify right bottom))
   )
-  (label "SND_~{RD}" (at 276.225 120.65 0)
+  (label "SND_~{RD}" (at 275.59 120.65 0)
     (effects (font (size 1.27 1.27)) (justify left bottom))
   )
@@
     (effects (font (size 1.27 1.27)) (justify left bottom))
   )
-  (label "SND_~{NMI}" (at 27.94 149.86 0)
+  (label "SND_~{NMI}" (at 26.67 149.86 0)
     (effects (font (size 1.27 1.27)) (justify left bottom))
   )
@@
     (effects (font (size 1.27 1.27)) (justify left bottom))
   )
-  (label "SND_SELECT" (at 116.205 158.75 0)
+  (label "~{SND_SELECT} " (at 116.205 158.75 0)
     (effects (font (size 1.27 1.27)) (justify left bottom))
   )
@@
     (effects (font (size 1.27 1.27)) (justify left bottom))
   )
-  (label "~{RESET}" (at 276.225 128.27 0)
+  (label "~{SND_RST}" (at 275.59 128.27 0)
     (effects (font (size 1.27 1.27)) (justify left bottom))
   )
@@
     (effects (font (size 1.27 1.27)) (justify right bottom))
   )
-  (label "SND_SELECT" (at 116.84 123.19 0)
+  (label "~{SND_SELECT} " (at 116.84 123.19 0)
     (effects (font (size 1.27 1.27)) (justify left bottom))
   )
@@
     (effects (font (size 1.27 1.27)) (justify right bottom))
   )
-  (label "S_~{MREQ}" (at 33.655 182.88 0)
+  (label "S_~{MREQ}" (at 27.305 182.88 0)
     (effects (font (size 1.27 1.27)) (justify left bottom))
   )
@@
     (effects (font (size 1.27 1.27)) (justify left bottom))
   )
-  (label "SND_~{RFSH}" (at 27.94 162.56 0)
+  (label "SND_~{RFSH}" (at 26.67 162.56 0)
     (effects (font (size 1.27 1.27)) (justify left bottom))
   )
@@
     (effects (font (size 1.27 1.27)) (justify right bottom))
   )
-  (label "SND_~{WR}" (at 276.225 123.19 0)
+  (label "SND_~{WR}" (at 275.59 123.19 0)
     (effects (font (size 1.27 1.27)) (justify left bottom))
   )
@@
     (effects (font (size 1.27 1.27)) (justify left bottom))
   )
-  (label "SND_SELECT" (at 114.935 194.31 0)
+  (label "~{SND_SELECT} " (at 114.935 194.31 0)
     (effects (font (size 1.27 1.27)) (justify left bottom))
   )
@@
     (effects (font (size 1.27 1.27)) (justify left bottom))
   )
-  (label "~{RESET}" (at 324.739 64.77 0)
+  (label "~{SND_RST}" (at 323.215 64.77 0)
     (effects (font (size 1.27 1.27)) (justify left bottom))
   )
@@
     (effects (font (size 1.27 1.27)) (justify left bottom))
   )
-  (label "~{RESET}" (at 275.844 80.01 0)
+  (label "~{SND_RST}" (at 271.78 80.01 0)
     (effects (font (size 1.27 1.27)) (justify left bottom))
   )
@@
     (effects (font (size 1.27 1.27)) (justify left))
   )
-  (hierarchical_label "SND_SELECT" (shape input) (at 99.06 87.63 180)
+  (hierarchical_label "~{SND_SELECT} " (shape input) (at 99.06 87.63 180)
     (effects (font (size 1.27 1.27)) (justify right))
   )
@@
     (effects (font (size 1.27 1.27)) (justify right))
   )
-  (hierarchical_label "~{RESET}" (shape input) (at 36.83 134.62 180)
+  (hierarchical_label "~{SND_RST}" (shape input) (at 36.83 134.62 180)
     (effects (font (size 1.27 1.27)) (justify right))
   )
@@
     (pin "2")
   )
-  (symbol (lib_id "jt74:74LS08") (at 339.344 62.23 0) (mirror x) (unit 4) (convert 2)
+  (symbol (lib_id "jt74:74LS08") (at 339.09 62.23 0) (mirror x) (unit 4) (convert 2)
     (in_bom yes) (on_board yes)
-    (property "Reference" "B2" (id 0) (at 339.344 63.5 0))
-    (property "Value" "74LS08" (id 1) (at 339.344 60.96 0))
-    (property "Footprint" "" (id 2) (at 339.344 62.23 0)
+    (property "Reference" "B2" (id 0) (at 339.09 63.5 0))
+    (property "Value" "74LS08" (id 1) (at 339.09 60.96 0))
+    (property "Footprint" "" (id 2) (at 339.09 62.23 0)
       (effects (font (size 1.27 1.27)) hide)
     )
-    (property "Datasheet" "http://www.ti.com/lit/gpn/sn74LS08" (id 3) (at 339.344 62.23 0)
+    (property "Datasheet" "http://www.ti.com/lit/gpn/sn74LS08" (id 3) (at 339.09 62.23 0)
       (effects (font (size 1.27 1.27)) hide)
     )

Commit message: Extermination schematics updated (issue #33)
Changed lines of the file:
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@@
+    (stroke (width 0) (type default) (color 0 0 0 0))
+  )
+  (wire (pts (xy 370.84 148.59) (xy 370.84 140.97))
+    (stroke (width 0) (type default) (color 0 0 0 0))
+  )
+  (wire (pts (xy 36.83 134.62) (xy 40.64 134.62))
+    (stroke (width 0) (type default) (color 0 0 0 0))
+  )
+  (wire (pts (xy 275.59 128.27) (xy 284.48 128.27))
+    (stroke (width 0) (type default) (color 0 0 0 0))
+  )
+  (wire (pts (xy 110.49 170.18) (xy 127 170.18))
+    (stroke (width 0) (type default) (color 0 0 0 0))
+  )
+  (wire (pts (xy 287.02 204.47) (xy 299.72 204.47))
+    (stroke (width 0) (type default) (color 0 0 0 0))
+  )
+  (wire (pts (xy 337.185 133.35) (xy 337.185 135.89))
+    (stroke (width 0) (type default) (color 0 0 0 0))
+  )
+  (wire (pts (xy 332.74 228.6) (xy 332.74 231.14))
+    (stroke (width 0) (type default) (color 0 0 0 0))
+  )
+  (wire (pts (xy 275.59 123.19) (xy 284.48 123.19))
+    (stroke (width 0) (type default) (color 0 0 0 0))
+  )
+  (wire (pts (xy 388.62 165.1) (xy 373.38 165.1))
+    (stroke (width 0) (type default) (color 0 0 0 0))
+  )
+  (wire (pts (xy 337.185 105.41) (xy 337.185 107.95))
+    (stroke (width 0) (type default) (color 0 0 0 0))
+  )
+  (bus (pts (xy 107.95 38.1) (xy 107.95 66.04))
+    (stroke (width 0) (type default) (color 0 0 0 0))
+  )
+  (wire (pts (xy 110.49 106.68) (xy 127 106.68))
+    (stroke (width 0) (type default) (color 0 0 0 0))
+  )
+  (wire (pts (xy 252.73 146.05) (xy 279.4 146.05))
+    (stroke (width 0) (type default) (color 0 0 0 0))
+  )
+  (bus (pts (xy 90.17 182.88) (xy 90.17 185.42))
+    (stroke (width 0) (type default) (color 0 0 0 0))
+  )
+  (bus (pts (xy 114.3 81.28) (xy 114.3 83.82))
+    (stroke (width 0) (type default) (color 0 0 0 0))
+  )
+  (wire (pts (xy 304.8 123.19) (xy 316.865 123.19))
+    (stroke (width 0) (type default) (color 0 0 0 0))
+  )
+  (bus (pts (xy 165.1 218.44) (xy 165.1 220.98))
+    (stroke (width 0) (type default) (color 0 0 0 0))
+  )
+  (wire (pts (xy 284.48 97.79) (xy 271.78 97.79))
+    (stroke (width 0) (type default) (color 0 0 0 0))
+  )
+  (wire (pts (xy 110.49 71.12) (xy 127 71.12))
+    (stroke (width 0) (type default) (color 0 0 0 0))
+  )
+  (bus (pts (xy 114.3 154.94) (xy 114.3 157.48))
+    (stroke (width 0) (type default) (color 0 0 0 0))
+  )
+  (wire (pts (xy 252.73 168.91) (xy 252.73 175.26))
+    (stroke (width 0) (type default) (color 0 0 0 0))
+  )
+  (wire (pts (xy 298.45 168.91) (xy 298.45 170.18))
+    (stroke (width 0) (type default) (color 0 0 0 0))
+  )
+  (wire (pts (xy 116.84 76.2) (xy 127 76.2))
+    (stroke (width 0) (type default) (color 0 0 0 0))
+  )
+  (bus (pts (xy 213.36 118.11) (xy 220.98 118.11))
+    (stroke (width 0) (type default) (color 0 0 0 0))
+  )
+  (wire (pts (xy 363.22 195.58) (xy 363.22 198.12))
     (stroke (width 0) (type default) (color 0 0 0 0))
   )
@@
     (stroke (width 0) (type default) (color 0 0 0 0))
   )
-  (wire (pts (xy 370.84 148.59) (xy 370.84 140.97))
-    (stroke (width 0) (type default) (color 0 0 0 0))
-  )
-  (wire (pts (xy 36.83 134.62) (xy 40.64 134.62))
-    (stroke (width 0) (type default) (color 0 0 0 0))
-  )
-  (wire (pts (xy 275.59 128.27) (xy 284.48 128.27))
-    (stroke (width 0) (type default) (color 0 0 0 0))
-  )
-  (wire (pts (xy 110.49 170.18) (xy 127 170.18))
-    (stroke (width 0) (type default) (color 0 0 0 0))
-  )
-  (wire (pts (xy 287.02 204.47) (xy 299.72 204.47))
-    (stroke (width 0) (type default) (color 0 0 0 0))
-  )
-  (wire (pts (xy 337.185 133.35) (xy 337.185 135.89))
-    (stroke (width 0) (type default) (color 0 0 0 0))
-  )
-  (wire (pts (xy 332.74 228.6) (xy 332.74 231.14))
-    (stroke (width 0) (type default) (color 0 0 0 0))
-  )
-  (wire (pts (xy 275.59 123.19) (xy 284.48 123.19))
-    (stroke (width 0) (type default) (color 0 0 0 0))
-  )
-  (wire (pts (xy 388.62 165.1) (xy 373.38 165.1))
-    (stroke (width 0) (type default) (color 0 0 0 0))
-  )
-  (wire (pts (xy 337.185 105.41) (xy 337.185 107.95))
-    (stroke (width 0) (type default) (color 0 0 0 0))
-  )
-  (bus (pts (xy 107.95 38.1) (xy 107.95 66.04))
-    (stroke (width 0) (type default) (color 0 0 0 0))
-  )
-  (wire (pts (xy 110.49 106.68) (xy 127 106.68))
-    (stroke (width 0) (type default) (color 0 0 0 0))
-  )
-  (wire (pts (xy 252.73 146.05) (xy 279.4 146.05))
-    (stroke (width 0) (type default) (color 0 0 0 0))
-  )
-  (bus (pts (xy 90.17 182.88) (xy 90.17 185.42))
-    (stroke (width 0) (type default) (color 0 0 0 0))
-  )
-  (bus (pts (xy 114.3 81.28) (xy 114.3 83.82))
-    (stroke (width 0) (type default) (color 0 0 0 0))
-  )
-  (wire (pts (xy 304.8 123.19) (xy 316.865 123.19))
-    (stroke (width 0) (type default) (color 0 0 0 0))
-  )
-  (bus (pts (xy 165.1 218.44) (xy 165.1 220.98))
-    (stroke (width 0) (type default) (color 0 0 0 0))
-  )
-  (wire (pts (xy 284.48 97.79) (xy 271.78 97.79))
-    (stroke (width 0) (type default) (color 0 0 0 0))
-  )
-  (wire (pts (xy 110.49 71.12) (xy 127 71.12))
-    (stroke (width 0) (type default) (color 0 0 0 0))
-  )
-  (bus (pts (xy 114.3 154.94) (xy 114.3 157.48))
-    (stroke (width 0) (type default) (color 0 0 0 0))
-  )
-  (wire (pts (xy 252.73 168.91) (xy 252.73 175.26))
-    (stroke (width 0) (type default) (color 0 0 0 0))
-  )
-  (wire (pts (xy 298.45 168.91) (xy 298.45 170.18))
-    (stroke (width 0) (type default) (color 0 0 0 0))
-  )
-  (wire (pts (xy 116.84 76.2) (xy 127 76.2))
-    (stroke (width 0) (type default) (color 0 0 0 0))
-  )
-  (bus (pts (xy 213.36 118.11) (xy 215.9 118.11))
-    (stroke (width 0) (type default) (color 0 0 0 0))
-  )
-  (wire (pts (xy 363.22 195.58) (xy 363.22 198.12))
-    (stroke (width 0) (type default) (color 0 0 0 0))
-  )
   (bus (pts (xy 107.95 223.52) (xy 107.95 226.06))
     (stroke (width 0) (type default) (color 0 0 0 0))
@@
     (stroke (width 0) (type default) (color 0 0 0 0))
   )
-  (bus (pts (xy 102.87 27.94) (xy 107.95 27.94))
+  (bus (pts (xy 86.36 27.94) (xy 107.95 27.94))
     (stroke (width 0) (type default) (color 0 0 0 0))
   )
@@
     (effects (font (size 1.27 1.27)) (justify right bottom))
   )
-  (hierarchical_label "SND_~{RD}" (shape input) (at 35.56 177.8 180)
+  (hierarchical_label "SND_~{RD}" (shape output) (at 35.56 177.8 180)
     (effects (font (size 1.27 1.27)) (justify right))
   )
@@
     (effects (font (size 1.27 1.27)) (justify left))
   )
-  (hierarchical_label "SND_A[15..0]" (shape input) (at 102.87 27.94 180)
+  (hierarchical_label "SND_A[15..0]" (shape output) (at 86.36 27.94 180)
     (effects (font (size 1.27 1.27)) (justify right))
   )
@@
     (effects (font (size 1.27 1.27)) (justify right))
   )
-  (hierarchical_label "SND_D[7..0]" (shape bidirectional) (at 275.59 44.45 0)
+  (hierarchical_label "SND_D[7..0]" (shape tri_state) (at 275.59 44.45 0)
     (effects (font (size 1.27 1.27)) (justify left))
   )
@@
     (effects (font (size 1.27 1.27)) (justify right))
   )
-  (hierarchical_label "SHD[7..0]" (shape output) (at 215.9 118.11 0)
+  (hierarchical_label "SHD[7..0]" (shape bidirectional) (at 220.98 118.11 0)
     (effects (font (size 1.27 1.27)) (justify left))
   )
@@
     (effects (font (size 1.27 1.27)) (justify right))
   )
-  (hierarchical_label "SND_~{WR}" (shape input) (at 35.56 180.34 180)
+  (hierarchical_label "SND_~{WR}" (shape output) (at 35.56 180.34 180)
     (effects (font (size 1.27 1.27)) (justify right))
   )
