File: cores/kiwi/sch/exterm.kicad_sch (KiCad schematic)
At the start: 96 parts, among them J1 Conn_01x04_Male, J16 HA1388, J8 TL7705A, SW1 SW_DIP_x02, U5 74LS02

Commit message: Merged sch branch. Schematics moved from extem core to kiwi core. exterm core may never be independent from the kiwi core
Parts:
- removed 2.2Ω: R10, symbol Device:R_US
- removed 2.2Ω?: R11, symbol Device:R_US
- removed 6.2Ω: R8, symbol Device:R_US
- removed 8.2KΩ, R1KΩ: R7, symbol Device:R_US
- removed A10, A12, A13, A2, A4, A5, A7, A8, C11, C9, E4: 27C512, Package_DIP:DIP-28_W15.24mm, symbol Memory_EPROM:27C512
- removed A15, B5, E1: 74LS174, symbol jt74:74LS174
- removed A16: 74LS273, symbol jt74:74LS273
- removed A17: 12.000MHz, Oscillator:Oscillator_SMD_Abracon_ASDMB-4Pin_2.5x2.0mm, symbol Oscillator:ASDMB-xxxMHz
- removed B1, G13: 74LS04, symbol jt74:74LS04
- removed B11, B12, B8, B9: 74LS157, symbol jt74:74LS157
- removed B13, C4, C5, E11, E12: 74LS245, symbol jt74:74LS245
- removed B14, C14: 74LS367, symbol jt74:74LS367
- removed B15: YM3909, symbol yamaha:YM3909
- removed B17: YM3906, symbol yamaha:YM3906
- removed B2, B6: 74LS08, symbol jt74:74LS08
- removed B3, B4, B7: 74LS74, symbol jt74:74LS74
- removed C10, C6: C104, symbol Device:C
- removed C11, C14, C15, C16, C17, C18, C19, C2, C7: 4.7μF, symbol Device:CP1
- removed C13: 1μF, symbol Device:CP1
- removed C2, C3, D6, D8: PAL16L8, symbol Logic_Programmable:PAL16L8
- removed C2: 220μF, symbol Device:CP1
- removed C20: C1041, symbol Device:C
- removed C4: C101, symbol Device:C
- removed C6: 74LS32, symbol jt74:74LS32
- removed C8: MB8464A-10L-LL, symbol fujitsu:MB8464A-10L-LL
- removed C9: 10μF, symbol Device:CP1
- removed D3, E8: Z80CPU, symbol CPU:Z80CPU
- removed E13, E14, E16, E17: HM6116P-3, symbol arcade:HM6116P-3
- removed F13: MB7124E, symbol arcade:MB7124E
- removed F8: YM2203, Package_DIP:DIP-40_W15.24mm, symbol yamaha:YM2203
- removed G14: 74HC4024, Package_SO:SOIC-14_3.9x8.7mm_P1.27mm, symbol 74xx:74HC4024
- removed G4: INTEL8742, symbol Intel:INTEL8742
- removed H11: YM3014, Package_DIP:DIP-8_W7.62mm, symbol yamaha:YM3014
- removed H12: NJM4558, symbol Amplifier_Operational:NJM4558
- removed H5, U5: 74LS02, symbol jt74:74LS02
- removed J1: Conn_01x04_Male, symbol Connector:Conn_01x04_Male
- removed J16: HA1388, symbol hitachi:HA1388
- removed J8: TL7705A, symbol Power_Supervisor:TL7705A
- removed JP1: Jumper_2_Bridged, symbol Jumper:Jumper_2_Bridged
- removed R100Ω: R13, symbol Device:R_US
- removed R100Ω?: R14, symbol Device:R_US
- removed R150Ω, R330Ω (x2): R20, symbol Device:R_US
- removed R1KΩ: R16, symbol Device:R_US
- removed R1KΩ: R6, symbol Device:R_US
- removed R1KΩ: R1, symbol Device:R_US
- removed R330Ω: R19, symbol Device:R_US
- removed RV1: R_POT_US, symbol Device:R_POT_US
- removed SW1: SW_DIP_x02, symbol Switch:SW_DIP_x02
- removed SWA, SWB: SW_DIPS_08, symbol Mod_KC_Symbols:SW_DIPS_08
- removed ZD2: 18, Diode_SMD:D_SMF, symbol Diode:BZD27Cxx
- added J1: R_Pack08, symbol Device:R_Pack08
- added J2, J5: R_P, symbol Device:R_Pack08
- added ZD1: BZD27, Diode_SMD:D_SMF, symbol Diode:BZD27Cxx
Connections:
- net +12V: now also JM1.F (+12V)
- net -5V: now also JM1.E (-5V), ZD1.1 (K)
- net VCC: now also JM1.3 (VDDA), JM1.4 (+5V), JM1.C (+5V), JM1.D (+5V), J1.1 (R1.1), J1.8 (R8.1), J2.1 (R1.1), J2.8 (R8.1), J5.1 (R1.1), J5.8 (R8.1), ZD1.2 (A)
- net VSS: now also JM1.1 (GND), JM1.14 (VIDEO_GND), JM1.2 (VSSA), JM1.27 (GND), JM1.28 (GND), JM1.A (GND), JM1.B (GND), JM1.e (GND), JM1.f (GND), J1.16 (R1.2), J1.9 (R8.2), J2.16 (R1.2), J2.9 (R8.2), J5.16 (R1.2), J5.9 (R8.2)
- net N.C1: now reaches JM1.11 (NC)
- net RED: now reaches JM1.12 (RED)
- net BLUE: now reaches JM1.13 (BLUE)
- net COIN_1: now reaches JM1.16 (COIN_1)
- net 1P_START: now reaches JM1.17 (1P_START)
- net 1P_START: now also J5.2 (R2.1)
- net 1P_UP: now reaches JM1.18 (1P_UP)
- net 1P_UP: now also J2.5 (R5.1)
- net 1P_DOWN: now reaches JM1.19 (1P_DOWN)
- net 1P_DOWN: now also J2.4 (R4.1)
- net 1P_LEFT: now reaches JM1.20 (1P_LEFT)
- net 1P_LEFT: now also J1.7 (R7.1), J2.7 (R7.1)
- net 1P_RIGHT: now reaches JM1.21 (1P_RIGHT)
- net 1P_RIGHT: now also J1.6 (R6.1), J2.6 (R6.1)
- net 1P_BNT_1: now reaches JM1.22 (1P_BTN_1)
- net 1P_BNT_1: now also J5.3 (R3.1)
- net 1P_BNT_2: now reaches JM1.23 (1P_BTN_2)
- net 1P_BNT_2: now also J2.2 (R2.1)
- net 1P_BNT_3: now reaches JM1.24 (1P_BTN_3)
- net 1P_BNT_3: now also J2.3 (R3.1)
- net 1P_BNT_4: now reaches JM1.25 (1P_BTN_4)
- net 1P_SELECT: now reaches JM1.26 (1P_SELECT)
- net COIN_CNT_1: now reaches JM1.8 (COIN_CNT_1)
- net N.C0: now reaches JM1.9 (NC)
- net COIN_CNT_2: now reaches JM1.J (COIN_CNT_2)
- net GREEN: now reaches JM1.N (GREEN)
- net SYNC: now reaches JM1.P (SYNC)
- net SERVICE: now reaches JM1.R (SERVICE)
- net SERVICE: now also J5.4 (R4.1)
- net N.C4: now reaches JM1.S (NC)
- net N.C4: now also J5.5 (R5.1)
- net COIN_2: now reaches JM1.T (COIN_2)
- net 2P_START: now reaches JM1.U (2P_START)
- net 2P_START: now also J5.6 (R6.1)
- net 2P_UP: now reaches JM1.V (2P_UP)
- net 2P_UP: now also J1.5 (R5.1)
- net 2P_DOWN: now reaches JM1.W (2P_DOWN)
- net 2P_DOWN: now also J1.4 (R4.1)
- net 2P_LEFT: now reaches JM1.X (2P_LEFT)
- net 2P_RIGHT: now reaches JM1.Y (2P_RIGHT)
- net 2P_BNT_1: now reaches JM1.Z (2P_BTN_1)
- net 2P_BNT_1: now also J5.7 (R7.1)
- net 2P_BNT_2: now reaches JM1.a (2P_BTN_2)
- net 2P_BNT_2: now also J1.3 (R3.1)
- net 2P_BNT_3: now reaches JM1.b (2P_BTN_3)
- net 2P_BNT_3: now also J1.2 (R2.1)
- net 2P_BNT_4: now reaches JM1.c (2P_BTN_4)
- net 2P_SELECT: now reaches JM1.d (2P_SELECT)
- net N.C renamed N.C3
- new net C0: J5.15 (R2.2)
- new net C1: J2.14 (R3.2)
- new net C10: J1.14 (R3.2)
- new net C11: J5.10 (R7.2)
- new net C12: J1.13 (R4.2)
- new net C13: J1.12 (R5.2)
- new net C14: J1.11 (R6.2)
- new net C15: J1.10 (R7.2)
- new net C18: J5.12 (R5.2)
- new net C19: J5.13 (R4.2)
- new net C2: J2.15 (R2.2)
- new net C3: J5.14 (R3.2)
- new net C4: J2.13 (R4.2)
- new net C5: J2.12 (R5.2)
- new net C6: J2.11 (R6.2)
- new net C7: J2.10 (R7.2)
- new net C8: J5.11 (R6.2)
- new net C9: J1.15 (R2.2)
- no-connect marks 30 -> 0
Other:
- added sheet colmix (colmix.kicad_sch)
- added sheet gfx (gfx.kicad_sch)
- added sheet main (main.kicad_sch)
- added sheet mcu (mcu.kicad_sch)
- added sheet sound (sound.kicad_sch)
- added sheet watchdog (watchdog.kicad_sch)
- note added: "CABINET I/O"
- note added: "RC Filters"
- note removed: "?"
- note removed: "COLMIX"
- note removed: "CPU MAIN"
- note removed: "GXF"
- note removed: "MAIN"
- note removed: "NO MOUNTED"
- note removed: "NOT MOUNTED"
- note removed: "PIN16 G15"
- note removed: "PIN19SETA003"
- note removed: "PIN20SETA003"
- note removed: "PIN23PC050"
- note removed: "POSIBLEMENTE PXCLK"
- note removed: "REVISAR"
- note removed: "SOUND"
- note removed: "TRIESTADO?"
- moved on the sheet: JM1
