File: cores/kiwi/sch/insectx/cpu.kicad_sch (KiCad schematic)
At the start: 31 parts, among them U11 74LS04, U12 74LS08, U13 74LS74, U14 74LS74, U15 74LS174, U17 74LS74, U18 74LS157, U19 74LS157, U20 74LS157, U21 74LS157, U25 PAL16L8, U26 PAL16L8, U27 74LS245, U28 74LS245, U30 HM6264, U31 uPD43256BCZ-B, U32 27C010, U34 Z80CPU, U35 PAL16L8, U36 PAL16L8, U37 74LS174, U38 27512, U39 Z80CPU

Commit message: update_skutis
Other:
- note added: "falta"
Changed lines of the file:
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@@
     (company "Ulf Skutnabba, twitter: @skutis77")
   )
-  (bus_alias "SHRAM2" (members "~{SHRAMWR}" "~{SHRAMCS}" "~{MSHRAMEN}" "~{SSHRAMEN}"))
   (bus_alias "SHRAM" (members "~{OBJORVRAMEN}" "~{MSHRAMRQ}"))
   (bus_alias "OBJCODE" (members "~{OBJCODELO}" "~{OBJCODEHI}"))
+  (bus_alias "SHRAM2" (members "~{SHRAMWR}" "~{SHRAMCS}" "~{MSHRAMEN}" "~{SSHRAMEN}"))
   (junction (at 344.17 171.45) (diameter 0) (color 0 0 0 0)
   )
@@
     (effects (font (size 1.27 1.27)) (justify left bottom))
   )
+  (text "falta" (at 158.75 36.83 0)
+    (effects (font (size 1.27 1.27)) (justify left bottom))
+  )
