File: cores/kiwi/sch/insectx/cpu.kicad_sch (KiCad schematic)
At the start: 31 parts, among them U11 74LS04, U12 74LS08, U13 74LS74, U14 74LS74, U15 74LS174, U17 74LS74, U18 74LS157, U19 74LS157, U20 74LS157, U21 74LS157, U25 PAL16L8, U26 PAL16L8, U27 74LS245, U28 74LS245, U30 HM6264, U31 uPD43256BCZ-B, U32 27C010, U34 Z80CPU, U35 PAL16L8, U36 PAL16L8, U37 74LS174, U38 27512, U39 Z80CPU

Commit message: wip
Other:
- note added: "U26-B06-12 ~{SWAIT} = SBANK1 & ~i11 & ~~{SSHRAMEN} + ~{SSHRAMRQ} & SBANK1 & ~i11 ~{MWAIT} = ~{OBJORVRAMEN} & ~{SSHRAMEN} + i6 & ~{SSHRAMEN} ~{SSHRAMEN} = ~{SSHRAMRQ} + ~~{MSHRAMRQ} & ~{SSHRAMEN} ~{MSHRAMEN} = ~{MSHRAMRQ} + ~~{SSHRAMRQ} & ~{MSHRAMEN} ~{SHRAMCS} = ~{MSHRAMRQ} & ~{SSHRAMRQ} ~{SHRAMWR} = ~{MWR} & ~{SSHRAMEN} + ~{MSHRAMRQ} & ~{SSHRAMRQ} + ~{SWR} & ~{MSHRAMEN} ~{SSHRAMENB} = ~{SSHRAMEN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"
- note removed: "U26-B06-12 SWAIT = SBANK1 & /i11 & (/SSHRAMEN + SSHRAMRQ) MWAIT = (OBJORVRAMEN + i6) & SSHRAMEN SSHRAMEN = SSHRAMRQ + /MASHRAMRQ & SSHRAMEN MSHRAMEN = MASHRAMRQ + /SSHRAMRQ & MSHRAMEN SHRAMCS = MSHRAMRQ & SSHRAMRQ SHRAMWR = MWR & SSHRAMEN + MASHRAMRQ & SSHRAMRQ + SWR & MSHRAMEN SSHRAMENB = SSHRAMEN"
- note removed: "falta"
- moved on the sheet: R17
Changed lines of the file:
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@@
   (title_block
     (title "Insector X - P0-056A")
-    (date "2022-12-01")
+    (date "2022-12-02")
     (company "Ulf Skutnabba, twitter: @skutis77")
   )
@@
     (stroke (width 0) (type default) (color 0 0 0 0))
   )
-  (wire (pts (xy 25.4 222.25) (xy 34.29 222.25))
+  (wire (pts (xy 15.24 222.25) (xy 34.29 222.25))
     (stroke (width 0) (type default) (color 0 0 0 0))
   )
@@
     (stroke (width 0) (type default) (color 0 0 0 0))
   )
-  (wire (pts (xy 60.96 209.55) (xy 60.96 222.25))
-    (stroke (width 0) (type default) (color 0 0 0 0))
-  )
   (wire (pts (xy 293.37 198.12) (xy 299.72 198.12))
     (stroke (width 0) (type default) (color 0 0 0 0))
@@
     (stroke (width 0) (type default) (color 0 0 0 0))
   )
-  (wire (pts (xy 25.4 92.71) (xy 25.4 222.25))
+  (wire (pts (xy 15.24 92.71) (xy 15.24 222.25))
     (stroke (width 0) (type default) (color 0 0 0 0))
   )
@@
     (stroke (width 0) (type default) (color 0 0 0 0))
   )
-  (wire (pts (xy 38.1 92.71) (xy 25.4 92.71))
+  (wire (pts (xy 38.1 92.71) (xy 15.24 92.71))
     (stroke (width 0) (type default) (color 0 0 0 0))
   )
@@
     (effects (font (size 1.27 1.27)) (justify left bottom))
   )
-  (text "U26-B06-12\nSWAIT = SBANK1 & /i11 & (/SSHRAMEN + SSHRAMRQ)\nMWAIT = (OBJORVRAMEN + i6) & SSHRAMEN\nSSHRAMEN = SSHRAMRQ + /MASHRAMRQ & SSHRAMEN\nMSHRAMEN = MASHRAMRQ + /SSHRAMRQ & MSHRAMEN\nSHRAMCS = MSHRAMRQ & SSHRAMRQ\nSHRAMWR = MWR & SSHRAMEN + MASHRAMRQ & SSHRAMRQ + SWR & MSHRAMEN\nSSHRAMENB = SSHRAMEN"
-    (at 49.53 123.19 0)
-    (effects (font (size 1.27 1.27)) (justify left bottom))
-  )
-  (text "falta" (at 158.75 36.83 0)
+  (text "U26-B06-12\n\n~{SWAIT} = SBANK1 & ~i11 & ~~{SSHRAMEN} + ~{SSHRAMRQ} & SBANK1 & ~i11\n~{MWAIT} = ~{OBJORVRAMEN} & ~{SSHRAMEN} + i6 & ~{SSHRAMEN}\n~{SSHRAMEN} = ~{SSHRAMRQ} + ~~{MSHRAMRQ} & ~{SSHRAMEN}\n~{MSHRAMEN} = ~{MSHRAMRQ} + ~~{SSHRAMRQ} & ~{MSHRAMEN}\n~{SHRAMCS} = ~{MSHRAMRQ} & ~{SSHRAMRQ}\n~{SHRAMWR} = ~{MWR} & ~{SSHRAMEN} + ~{MSHRAMRQ} & ~{SSHRAMRQ} + ~{SWR} & ~{MSHRAMEN}\n~{SSHRAMENB} = ~{SSHRAMEN}\n\nInputs i7 and i8 have been set to logical 1 in the equations.\n-----------------------------------------------------------------------\nU36-B06-101\n\n~~{PALEN} = MA9 & MA10 & MA11 & MA12 & MA13 & ~~{MMREQ} & ~{MRFSH}\n~~{VRAMWR} = MA9 & MA10 & MA11 & MA12 & ~MA13 & ~MA14 & ~~{MMREQ} & ~{MRFSH}\n~~{BGTRNSP} = MA9 & MA10 & MA11 & MA12 & ~MA13 & MA14 & ~MA15 & ~~{MMREQ} & ~{MRFSH} & ~{MWR}\n~~{BNKSW} = MA9 & MA10 & MA11 & MA12 & ~MA13 & MA14 & MA15 & ~~{MMREQ} & ~{MRFSH} & ~~{MWR}\n~~{OBJCODELO} = MA9 & MA10 & ~MA11 & ~MA12 & ~~{MMREQ} & ~{MRFSH}\n~~{OBJCODEHI} = MA9 & MA10 & ~MA11 & MA12 & ~~{MMREQ} & ~{MRFSH}\n~~{MSHRAMRQ} = MA9 & MA10 & MA11 & ~MA12 & ~~{MMREQ} & ~{MRFSH}\n~~{OBJORVRAMEN} = MA9 & MA10 & MA11 & MA12 & ~MA13 & (~MA15 & ~~{MMREQ} & ~{MRFSH} + ~MA14 & ~~{MMREQ} & ~{MRFSH}) +\n                  MA9 & MA10 & ~MA11 & ~~{MMREQ} & ~{MRFSH}\n-----------------------------------------------------------------------\nU35-B53-12\n\n~{MRA16} = MA15 & MBSWD2\n~{MRA15} = MA15 & MBSWD1\n~~{MRA14} = MA15 & ~MBSWD0 + ~MA15 & ~MA14\n~~{MROMCS} = ~MA15 & MA14 & ~~{MMREQ} & ~{MRFSH} & ~MBSWD2 & MBSWD1 +\n       ~MA14 & ~~{MMREQ} & ~{MRFSH} & ~MBSWD2 & MBSWD1 +\n       ~MA15 & MA14 & ~~{MMREQ} & ~{MRFSH} & MBSWD2 +\n       ~MA15 & ~~{MMREQ} & ~{MRFSH} & ~MBSWD1 +\n       ~MA14 & ~~{MMREQ} & ~{MRFSH} & MBSWD2\n~~{MRAMCS} = MA15 & ~MA14 & ~~{MMREQ} & ~{MRFSH} & ~MBSWD2 & ~MBSWD1\no17 = ~{OBJCODELO} & ~H4B\no18 = ~{OBJCODEHI} & ~H4B\n~{OBJRAMCS} = ~{OBJCODELO} & ~{OBJCODEHI} & ~H4B\n-----------------------------------------------------------------------\nU25-B06-13\n~~{SROMCS} = ~SA14 & ~SA13 & ~~{SMREQ} & ~{SRFSH} + ~SA15 & SA14 & ~~{SMREQ} & ~{SRFSH} + ~SA15 & ~SA14 & ~~{SMREQ} & ~{SRFSH}\n~~{SSHRAMRQ} = SA15 & SA14 & SA13 & ~SA12 & ~~{SMREQ} & ~{SRFSH} + SA15 & SA14 & ~SA13 & SA12 & ~~{SMREQ} & ~{SRFSH}\n~~{SBNKSW} = SA15 & ~SA14 & SA13 & ~SA12 & ~~{SWR} & ~~{SMREQ} & ~{SRFSH}\n~~{YM2203CS} = SA15 & ~SA14 & SA13 & SA12 & ~~{SMREQ} & ~{SRFSH}\n~~{RDINPUTS} = SA15 & SA14 & ~SA13 & ~SA12 & ~~{SMREQ} & ~{SRFSH}\n~o17 = SA15 & SA14 & SA13 & SA12 & ~~{SMREQ} & ~{SRFSH}\nSRA13 = SA15 & SBANK0 + ~SA15 & SA13\nSRA14 = SA15 & SBANK1 + ~SA15 & SA14"
+    (at 17.78 193.04 0)
     (effects (font (size 1.27 1.27)) (justify left bottom))
   )
@@
     (pin "9")
   )
-  (symbol (lib_id "power:VCC") (at 60.96 201.93 0) (unit 1)
+  (symbol (lib_id "power:VCC") (at 60.96 214.63 0) (unit 1)
     (in_bom yes) (on_board yes) (fields_autoplaced)
-    (property "Reference" "#PWR0146" (id 0) (at 60.96 205.74 0)
+    (property "Reference" "#PWR0146" (id 0) (at 60.96 218.44 0)
       (effects (font (size 1.27 1.27)) hide)
     )
-    (property "Value" "VCC" (id 1) (at 60.96 196.85 0))
-    (property "Footprint" "" (id 2) (at 60.96 201.93 0)
+    (property "Value" "VCC" (id 1) (at 60.96 209.55 0))
+    (property "Footprint" "" (id 2) (at 60.96 214.63 0)
       (effects (font (size 1.27 1.27)) hide)
     )
-    (property "Datasheet" "" (id 3) (at 60.96 201.93 0)
+    (property "Datasheet" "" (id 3) (at 60.96 214.63 0)
       (effects (font (size 1.27 1.27)) hide)
     )
@@
     (pin "9")
   )
-  (symbol (lib_id "Device:R") (at 60.96 205.74 0) (unit 1)
+  (symbol (lib_id "Device:R") (at 60.96 218.44 0) (unit 1)
     (in_bom yes) (on_board yes) (fields_autoplaced)
-    (property "Reference" "R17" (id 0) (at 63.5 204.4699 0)
+    (property "Reference" "R17" (id 0) (at 63.5 217.1699 0)
       (effects (font (size 1.27 1.27)) (justify left))
     )
-    (property "Value" "1k" (id 1) (at 63.5 207.0099 0)
+    (property "Value" "1k" (id 1) (at 63.5 219.7099 0)
       (effects (font (size 1.27 1.27)) (justify left))
     )
-    (property "Footprint" "" (id 2) (at 59.182 205.74 90)
+    (property "Footprint" "" (id 2) (at 59.182 218.44 90)
       (effects (font (size 1.27 1.27)) hide)
     )
-    (property "Datasheet" "~" (id 3) (at 60.96 205.74 0)
+    (property "Datasheet" "~" (id 3) (at 60.96 218.44 0)
       (effects (font (size 1.27 1.27)) hide)
     )

Commit message: sch updated
Connections:
- net MA10: now also U36.6 (I6); no longer U36.2 (I2)
- net MA11: now also U36.5 (I5); no longer U36.3 (I3)
- net MA13: now also U36.3 (I3); no longer U36.5 (I5)
- net MA14: now also U36.2 (I2); no longer U36.6 (I6)
- net MA15: now also U36.1 (I1); no longer U36.7 (I7)
- net MA9: now also U36.7 (I7); no longer U36.1 (I1)
- net SBANK1: no longer U26.9 (I9)
- net at U13.4 (~{S}), U13.9 (Q): now also U26.9 (I9)
Other:
- note added: "U26-B06-12 ~{SWAIT} = i9 & ~i11 & (~~{SSHRAMEN} + ~{SSHRAMRQ}) ~{MWAIT} = ~{OBJORVRAMEN} & ~{SSHRAMEN} + i6 & ~{SSHRAMEN} ~{SSHRAMEN} = ~{SSHRAMRQ} + ~~{MSHRAMRQ} & ~{SSHRAMEN} ~{MSHRAMEN} = ~{MSHRAMRQ} + ~~{SSHRAMRQ} & ~{MSHRAMEN} ~{SHRAMCS} = ~{MSHRAMRQ} & ~{SSHRAMRQ} ~{SHRAMWR} = ~{MWR} & ~{SSHRAMEN} + ~{MSHRAMRQ} & ~{SSHRAMRQ} + ~{SWR} & ~{MSHRAMEN} ~{SSHRAMENB} = ~{SSHRAMEN} Inputs i7 and i8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"
- note removed: "U26-B06-12 ~{SWAIT} = SBANK1 & ~i11 & ~~{SSHRAMEN} + ~{SSHRAMRQ} & SBANK1 & ~i11 ~{MWAIT} = ~{OBJORVRAMEN} & ~{SSHRAMEN} + i6 & ~{SSHRAMEN} ~{SSHRAMEN} = ~{SSHRAMRQ} + ~~{MSHRAMRQ} & ~{SSHRAMEN} ~{MSHRAMEN} = ~{MSHRAMRQ} + ~~{SSHRAMRQ} & ~{MSHRAMEN} ~{SHRAMCS} = ~{MSHRAMRQ} & ~{SSHRAMRQ} ~{SHRAMWR} = ~{MWR} & ~{SSHRAMEN} + ~{MSHRAMRQ} & ~{SSHRAMRQ} + ~{SWR} & ~{MSHRAMEN} ~{SSHRAMENB} = ~{SSHRAMEN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"
