File: cores/kiwi/sch/insectx/sound.kicad_sch (KiCad schematic)
At the start: 38 parts, among them J16 HA1388

Commit message: Updated schematics according to: [insectx] schematic signals #22
Parts:
- removed B11, B12, B8, B9: 74LS157, symbol jt74:74LS157
- removed B2: 74LS08, symbol jt74:74LS08
- removed C2: PAL16L8, symbol Logic_Programmable:PAL16L8
- removed C20, CC21: C104J, symbol Device:C
- removed C8: MB8464A-10L-LL, symbol fujitsu:MB8464A-10L-LL
- removed CC10: C104, symbol Device:C
- removed CC11, CC14, CC15, CC16, CC17, CC18, CC19, CC9, CCC2: 4.7μF, symbol Device:C_Polarized_Small_US
- removed CC12: C103J, symbol Device:C
- removed CC13: 1μF, symbol Device:C_Polarized_Small_US
- removed D3: Z80CPU, symbol CPU:Z80CPU
- removed E1: 74LS174, symbol jt74:74LS174
- removed E4: 27C512, Package_DIP:DIP-28_W15.24mm, symbol Memory_EPROM:27C512
- removed H11: YM3014, Package_DIP:DIP-8_W7.62mm, symbol yamaha:YM3014
- removed H12: NJM4558, symbol Amplifier_Operational:NJM4558
- removed J16: HA1388, symbol hitachi:HA1388
- removed R10, R11: 2.2Ω, symbol Device:R_US
- removed R21: 1KΩ, symbol Device:R_US
- removed R6, R7: R1KΩ, symbol Device:R_US
- removed R8: 6.2Ω, symbol Device:R_US
- removed R9: 8.2KΩ, symbol Device:R_US
- removed RV1: R_P, symbol Device:R_Potentiometer_US
- removed SWA1, SWB2: SW_DIPS_08, symbol Mod_KC_Symbols:SW_DIPS_08
- removed YM_F8: YM2203, Package_DIP:DIP-40_W15.24mm, symbol yamaha:YM2203
- added C11, C12, C5: 100nF, symbol Device:C
- added C13: 2.2uF, symbol Device:C_Polarized
- added C14: 220uF, symbol Device:C_Polarized
- added C4: 10uF, symbol Device:C_Polarized
- added C6, C7: 10nF, symbol Device:C
- added C8, C9: 4.7uF, symbol Device:C_Polarized
- added R12, R14: 1k, symbol Device:R
- added R15: 8.2k, symbol Device:R
- added R19, R21: 4.7R, symbol Device:R
- added R20: 6.2k, symbol Device:R
- added SW2, SW3: SW_DIP_x08, symbol Switch:SW_DIP_x08
- added U44: NJM4558, symbol Device:Opamp_Dual
- added U47: YM2203, Package_DIP:DIP-40_W15.24mm, symbol yamaha:YM2203
- added U53: YM3014, Package_DIP:DIP-8_W7.62mm, symbol yamaha:YM3014
- added U55: MB3730, symbol fujitsu:MB3730
- added VR1: 890R, symbol Device:R_Potentiometer
Connections:
- net VCC: now also U44.8 (V+), U47.21 (VCC), U53.1 (VCC)
- net VSS: now also U53.6 (VSS)
- new net: C4.1, U44.5 (+), U53.7 (RB)
- new net: C7.1, C9.1, U55.1
- new net: C13.1, U55.2
- new net: C14.1, U55.3
- new net: C5.1, R15.1
- new net: C6.1, R14.1, R15.2, R20.1, VR1.1
- new net: C8.1, U44.1, U44.2 (-)
- new net: U44.3 (+), U53.2 (BUFF)
- new net: C5.2, R12.1, U47.18 (CHC), U47.19 (CHB), U47.20 (CHA)
- new net: C11.2, R21.2
- new net: C8.2, R20.2
- new net: SW2.7, U47.10 (IOA6)
- new net: SW2.6, U47.11 (IOA5)
- new net: SW2.5, U47.12 (IOA4)
- new net: SW2.4, U47.13 (IOA3)
- new net: SW2.3, U47.14 (IOA2)
- new net: SW2.2, U47.15 (IOA1)
- new net: SW2.1, U47.16 (IOA0)
- new net: U47.22 (SH), U53.3 (LOAD)
- new net: U47.23 (OPO), U53.4 (SD)
- new net: SW3.1, U47.26 (IOB0)
- new net: SW3.2, U47.27 (IOB1)
- new net: SW3.3, U47.28 (IOB2)
- new net: SW3.4, U47.29 (IOB3)
- new net: SW3.5, U47.30 (IOB4)
- new net: SW3.6, U47.31 (IOB5)
- new net: SW3.7, U47.32 (IOB6)
- new net: SW3.8, U47.33 (IOB7)
- new net: U47.39 (PHS), U53.5 (PH1)
- new net: SW2.8, U47.9 (IOA7)
- new net: U44.6 (-), U44.7, U53.8 (MP)
- new net: C12.2, R19.2
- new net: C9.2, VR1.2
- new net +12V: U55.7
- new net GND: C11.1, C12.1, C13.2, C14.2, C4.2, C6.2, C7.2, R12.2, R14.2, SW2.10, SW2.11, SW2.12, SW2.13, SW2.14, SW2.15, SW2.16, SW2.9, SW3.10, SW3.11, SW3.12, SW3.13, SW3.14, SW3.15, SW3.16, SW3.9, U44.4 (V-), U47.1 (VSS), U55.4 (VSS), VR1.3
- new net H2B: U47.38 (PHM)
- new net SA0: U47.37 (A0)
- new net SD0: U47.40 (D0)
- new net SD1: U47.2 (D1)
- new net SD2: U47.3 (D2)
- new net SD3: U47.4 (D3)
- new net SD4: U47.5 (D4)
- new net SD5: U47.6 (D5)
- new net SD6: U47.7 (D6)
- new net SD7: U47.8 (D7)
- new net SPEAKER+: R21.1, U55.6
- new net SPEAKER-: R19.1, U55.5
- new net ~{SRD}: U47.36 (~{RD})
- new net ~{SRST}: U47.24 (~{IC})
- new net ~{SWR}: U47.35 (~{WR})
- new net ~{YM2203CS}: U47.34 (~{CS})
- new net ~{YMIRQ}: U47.25 (~{IRQ})
- no-connect marks 14 -> 0
Other:
- note removed: "Shared RAM"
- company: JOTEGO -> Ulf Skutnabba, twitter: @skutis77
- title: EXTERMINATION -> Insector X - P0-056A
