File: cores/kiwi/sch/exterm/gfx_ram.kicad_sch (KiCad schematic)
At the start: 6 parts

Commit message: issue#46
Connections:
- net H3B renamed H3_BUF
Changed lines of the file:
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@@
     (stroke (width 0) (type default) (color 0 0 0 0))
   )
-  (wire (pts (xy 53.975 125.73) (xy 64.135 125.73))
+  (wire (pts (xy 50.8 125.73) (xy 64.135 125.73))
     (stroke (width 0) (type default) (color 0 0 0 0))
   )
@@
     (stroke (width 0) (type default) (color 0 0 0 0))
   )
-  (wire (pts (xy 60.325 86.36) (xy 64.135 86.36))
+  (wire (pts (xy 59.69 86.36) (xy 64.135 86.36))
     (stroke (width 0) (type default) (color 0 0 0 0))
   )
@@
     (effects (font (size 1.27 1.27)) (justify right bottom))
   )
-  (label "H3B" (at 53.975 125.73 0)
+  (label "H3_BUF" (at 50.8 125.73 0)
     (effects (font (size 1.27 1.27)) (justify left bottom))
   )
@@
     (effects (font (size 1.27 1.27)) (justify right))
   )
-  (hierarchical_label "H3B" (shape input) (at 60.325 86.36 180)
+  (hierarchical_label "H3_BUF" (shape input) (at 59.69 86.36 180)
     (effects (font (size 1.27 1.27)) (justify right))
   )
