File: cores/kiwi/sch/exterm/main.kicad_sch (KiCad schematic)
At the start: 23 parts

Commit message: issue#46
Parts:
- removed B3, B7: 74LS74, symbol jt74:74LS74
- removed C4, C5: 74LS245, symbol jt74:74LS245
- removed C6: 74LS32, symbol jt74:74LS32
Connections:
- net GFX_~{CE}: now reaches B6.6
- net CLK_MAIN: no longer names the net of B13.17 (B1), B4.11 (C), E8.6 (~{CLK}), R19.2
- net CLK_SND renamed H0_BUF
- net H1B renamed H1_BUF
- net H3B renamed H3_BUF
- net H4B renamed H4_BUF
- net M_~{IORQ}: no longer names the net of B4.1 (~{R}), E8.20 (~{IORQ})
- net M_~{MREQ} renamed ~{MREQ}
- net M_~{RFSH} renamed ~{RFSH}
- net PHM renamed H2_BUF
- net PULL DOWN: no longer names the net of B13.16 (B2), RR15.2
- net QH: no longer names the net of B4.9 (Q), C3.6 (I6)
- net SB_~{CE} renamed ~{SBNKSWR}
- net ~{MAIN_A11} renamed ~{WDOGCLR}
- net ~{MAIN_A13} renamed ~{OBJCODEHI}
- net ~{MAIN_WR} renamed ~{OBJCODELO}
- net ~{SB_CE}: no longer names the net of C3.5 (I5), D8.19 (IO1)
- net ~{SND_WR} renamed ~{SBNKMWR}
- net ~{VBLK} renamed VBLK
- net ~{WATCHDOG} renamed WATCHDOG
- no-connect marks 15 -> 13
Other:
- note added: "LOW PASS FILTER"
- moved on the sheet: B13, B1A, B2B, B2C, B4A, B4B, B6B, C3, CC4, D8, R1, R19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
